Commit message: add mirrors

File: orne_box_description/urdf/orne_box_tilted_lidar.gazebo.xacro (robot description, xacro)
@@ -46,5 +46,5 @@
     <sensor type="ray" name="head_hokuyo_sensor">
       <pose>0 0 0 0 0 0</pose>
-      <visualize>$(arg laser_visual)</visualize>
+      <visualize>false</visualize>
       <update_rate>40</update_rate>
       <ray>
@@ -113,3 +113,73 @@
     </sensor>
   </gazebo>
+  <gazebo reference="hokuyo_tilted_left_link">
+    <sensor type="ray" name="hokuyo_tilted_left_sensor">
+      <pose>0 0 0 0 0 0</pose>
+      <visualize>$(arg laser_visual)</visualize>
+      <update_rate>10</update_rate>
+      <ray>
+        <scan>
+          <horizontal>
+            <samples>682</samples>
+            <resolution>1</resolution>
+            <min_angle>${PI/180*60}</min_angle>
+            <max_angle>${PI/180*120}</max_angle>
+          </horizontal>
+        </scan>
+        <range>
+          <min>0.10</min>
+          <max>5.60</max>
+          <resolution>0.01</resolution>
+        </range>
+        <noise>
+          <type>gaussian</type>
+          <!-- Noise parameters based on published spec for Hokuyo laser
+               achieving "+-30mm" accuracy at range < 10m.  A mean of 0.0m and
+               stddev of 0.01m will put 99.7% of samples within 0.03m of the true
+               reading. -->
+          <mean>0.0</mean>
+          <stddev>0.01</stddev>
+        </noise>
+      </ray>
+      <plugin name="gazebo_ros_head_hokuyo_controller" filename="libgazebo_ros_laser.so">
+        <topicName>/tilted_scan_left</topicName>
+        <frameName>hokuyo_tilted_left_link</frameName>
+      </plugin>
+    </sensor>
+  </gazebo>
+  <gazebo reference="hokuyo_tilted_right_link">
+    <sensor type="ray" name="hokuyo_tilted_right_sensor">
+      <pose>0 0 0 0 0 0</pose>
+      <visualize>$(arg laser_visual)</visualize>
+      <update_rate>10</update_rate>
+      <ray>
+        <scan>
+          <horizontal>
+            <samples>682</samples>
+            <resolution>1</resolution>
+            <min_angle>${-PI/180*120}</min_angle>
+            <max_angle>${-PI/180*60}</max_angle>
+          </horizontal>
+        </scan>
+        <range>
+          <min>0.10</min>
+          <max>5.60</max>
+          <resolution>0.01</resolution>
+        </range>
+        <noise>
+          <type>gaussian</type>
+          <!-- Noise parameters based on published spec for Hokuyo laser
+               achieving "+-30mm" accuracy at range < 10m.  A mean of 0.0m and
+               stddev of 0.01m will put 99.7% of samples within 0.03m of the true
+               reading. -->
+          <mean>0.0</mean>
+          <stddev>0.01</stddev>
+        </noise>
+      </ray>
+      <plugin name="gazebo_ros_head_hokuyo_controller" filename="libgazebo_ros_laser.so">
+        <topicName>/tilted_scan_right</topicName>
+        <frameName>hokuyo_tilted_right_link</frameName>
+      </plugin>
+    </sensor>
+  </gazebo>
 </robot>

File: orne_box_description/urdf/orne_box_tilted_lidar.urdf.xacro (robot description, xacro)
@@ -185,7 +185,20 @@
     <origin xyz="0.374295 0 0.2185" rpy="${-PI} 0 0"/>
   </xacro:sensor_hokuyo>
+  <xacro:property name="pitch" value="${PI/9}" />
+  <xacro:property name="roll" value="${PI*3/8}" />
+  <xacro:property name="len" value="0.1" />
+  <xacro:property name="front" value="1.00" />
+  <xacro:property name="height" value="0.30" />
   <xacro:include filename="$(find icart_mini_description)/urdf/sensors/hokuyo.urdf.xacro"/>
   <xacro:sensor_hokuyo name="hokuyo_tilted" parent="base_link">
-    <origin xyz="0.47 0 0.30" rpy="0 ${PI/9} 0"/>
+    <origin xyz="${front} 0 ${height}" rpy="0 ${pitch} 0"/>
+  </xacro:sensor_hokuyo>
+  <xacro:include filename="$(find icart_mini_description)/urdf/sensors/hokuyo.urdf.xacro"/>
+  <xacro:sensor_hokuyo name="hokuyo_tilted_left" parent="base_link">
+    <origin xyz="${front+len*sin(roll)*sin(pitch)} ${len*(-cos(roll)+1)} ${height+len*sin(roll)*cos(pitch)}" rpy="${-roll} ${pitch} 0"/>
+  </xacro:sensor_hokuyo>
+  <xacro:include filename="$(find icart_mini_description)/urdf/sensors/hokuyo.urdf.xacro"/>
+  <xacro:sensor_hokuyo name="hokuyo_tilted_right" parent="base_link">
+    <origin xyz="${front+len*sin(roll)*sin(pitch)} ${len*(cos(roll)-1)} ${height+len*sin(roll)*cos(pitch)}" rpy="${roll} ${pitch} 0"/>
   </xacro:sensor_hokuyo>
   <transmission name="tran1">

Commit message: make experimental setup

File: orne_box_description/urdf/orne_box_tilted_lidar.gazebo.xacro (robot description, xacro)
@@ -4,7 +4,14 @@
   <xacro:arg name="laser_visual" default="true"/>
   <xacro:arg name="imu_visual"   default="false"/>
+<!--
   <gazebo>
     <plugin name="gazebo_ros_control" filename="libgazebo_ros_control.so">
       <robotSimType>icart_mini_gazebo/ICartMiniHWSim</robotSimType>
+    </plugin>
+  </gazebo>
+-->
+  <gazebo>
+    <plugin name="gazebo_ros_control" filename="libgazebo_ros_control.so">
+      <robotSimType>gazebo_ros_control/DefaultRobotHWSim</robotSimType>
     </plugin>
   </gazebo>

File: orne_box_description/urdf/orne_box_tilted_lidar.urdf.xacro (robot description, xacro)
@@ -185,20 +185,88 @@
     <origin xyz="0.374295 0 0.2185" rpy="${-PI} 0 0"/>
   </xacro:sensor_hokuyo>
-  <xacro:property name="pitch" value="${PI/9}" />
-  <xacro:property name="roll" value="${PI*3/8}" />
+  <joint name="hokuyo_tilted_prismatic_joint" type="prismatic">
+    <parent link="base_link"/>
+    <child link="hokuyo_tilted_prismatic_link"/>
+    <origin xyz="1.0 0 1.0" rpy="0 0 0"/>
+    <axis xyz="0 0 1"/>
+    <limit effort="100" velocity="100.0" lower="-1" upper="1" />
+  </joint>
+  <link name="hokuyo_tilted_prismatic_link">
+    <inertial>
+      <origin xyz="0 0 0" />
+      <mass value="0.2" />
+      <inertia ixx="0.1" ixy="0.0" ixz="0.0" iyy="0.1" iyz="0.0" izz="0.1" />
+    </inertial>
+  </link>
+  <joint name="hokuyo_tilted_pitch_joint" type="revolute">
+    <parent link="hokuyo_tilted_prismatic_link"/>
+    <child link="hokuyo_tilted_pitch_link"/>
+    <origin xyz="0 0 0" rpy="0 0 0"/>
+    <axis xyz="0 1 0"/>
+    <limit effort="100" velocity="100.0" lower="${-PI}" upper="${PI}" />
+  </joint>
+  <link name="hokuyo_tilted_pitch_link">
+    <inertial>
+      <origin xyz="0 0 0" />
+      <mass value="0.2" />
+      <inertia ixx="0.1" ixy="0.0" ixz="0.0" iyy="0.1" iyz="0.0" izz="0.1" />
+    </inertial>
+  </link>
+  <joint name="hokuyo_tilted_roll_joint" type="revolute">
+    <parent link="hokuyo_tilted_pitch_link"/>
+    <child link="hokuyo_tilted_roll_link"/>
+    <origin xyz="0 0 0" rpy="0 0 0"/>
+    <axis xyz="1 0 0"/>
+    <limit effort="100" velocity="100.0" lower="${-PI}" upper="${PI}" />
+  </joint>
+  <link name="hokuyo_tilted_roll_link">
+    <inertial>
+      <origin xyz="0 0 0" />
+      <mass value="0.2" />
+      <inertia ixx="0.1" ixy="0.0" ixz="0.0" iyy="0.1" iyz="0.0" izz="0.1" />
+    </inertial>
+  </link>
   <xacro:property name="len" value="0.1" />
-  <xacro:property name="front" value="1.00" />
-  <xacro:property name="height" value="0.30" />
+  <xacro:property name="front" value="0" />
+  <xacro:property name="height" value="0" />
   <xacro:include filename="$(find icart_mini_description)/urdf/sensors/hokuyo.urdf.xacro"/>
-  <xacro:sensor_hokuyo name="hokuyo_tilted_center" parent="base_link">
-    <origin xyz="${front} 0 ${height}" rpy="0 ${pitch} 0"/>
+  <xacro:sensor_hokuyo name="hokuyo_tilted_center" parent="hokuyo_tilted_roll_link">
+    <origin xyz="${front} 0 ${height}" rpy="0 0 0"/>
   </xacro:sensor_hokuyo>
+  <joint name="hokuyo_mirror_roll1_joint" type="revolute">
+    <parent link="hokuyo_tilted_center_link"/>
+    <child link="hokuyo_mirror_roll1_link"/>
+    <origin xyz="0 ${len} 0" rpy="0 0 0"/>
+    <axis xyz="-1 0 0"/>
+    <limit effort="100" velocity="100.0" lower="${-PI}" upper="${PI}" />
+  </joint>
+  <link name="hokuyo_mirror_roll1_link">
+    <inertial>
+      <origin xyz="0 0 0" />
+      <mass value="0.2" />
+      <inertia ixx="0.1" ixy="0.0" ixz="0.0" iyy="0.1" iyz="0.0" izz="0.1" />
+    </inertial>
+  </link>
   <xacro:include filename="$(find icart_mini_description)/urdf/sensors/hokuyo.urdf.xacro"/>
-  <xacro:sensor_hokuyo name="hokuyo_tilted_left" parent="base_link">
-    <origin xyz="${front+len*sin(roll)*sin(pitch)} ${len*(-cos(roll)+1)} ${height+len*sin(roll)*cos(pitch)}" rpy="${-roll} ${pitch} 0"/>
+  <xacro:sensor_hokuyo name="hokuyo_tilted_left" parent="hokuyo_mirror_roll1_link">
+    <origin xyz="0 ${-len} 0" rpy="0 0 0"/>
   </xacro:sensor_hokuyo>
+  <joint name="hokuyo_mirror_roll2_joint" type="revolute">
+    <parent link="hokuyo_tilted_center_link"/>
+    <child link="hokuyo_mirror_roll2_link"/>
+    <origin xyz="0 ${-len} 0" rpy="0 0 0"/>
+    <axis xyz="1 0 0"/>
+    <limit effort="100" velocity="100.0" lower="${-PI}" upper="${PI}" />
+  </joint>
+  <link name="hokuyo_mirror_roll2_link">
+    <inertial>
+      <origin xyz="0 0 0" />
+      <mass value="0.2" />
+      <inertia ixx="0.1" ixy="0.0" ixz="0.0" iyy="0.1" iyz="0.0" izz="0.1" />
+    </inertial>
+  </link>
   <xacro:include filename="$(find icart_mini_description)/urdf/sensors/hokuyo.urdf.xacro"/>
-  <xacro:sensor_hokuyo name="hokuyo_tilted_right" parent="base_link">
-    <origin xyz="${front+len*sin(roll)*sin(pitch)} ${len*(cos(roll)-1)} ${height+len*sin(roll)*cos(pitch)}" rpy="${roll} ${pitch} 0"/>
+  <xacro:sensor_hokuyo name="hokuyo_tilted_right" parent="hokuyo_mirror_roll2_link">
+    <origin xyz="0 ${len} 0" rpy="0 0 0"/>
   </xacro:sensor_hokuyo>
   <transmission name="tran1">
@@ -222,3 +290,53 @@
     </actuator>
   </transmission>
+  <transmission name="tran3">
+    <type>transmission_interface/SimpleTransmission</type>
+    <joint name="hokuyo_tilted_pitch_joint">
+      <hardwareInterface>PositionJointInterface</hardwareInterface>
+    </joint>
+  <actuator name="hokuyo_tilted_pitch_motor">
+      <hardwareInterface>PositionJointInterface</hardwareInterface>
+      <mechanicalReduction>1</mechanicalReduction>
+    </actuator>
+  </transmission>
+  <transmission name="tran4">
+    <type>transmission_interface/SimpleTransmission</type>
+    <joint name="hokuyo_tilted_roll_joint">
+      <hardwareInterface>PositionJointInterface</hardwareInterface>
+    </joint>
+  <actuator name="hokuyo_tilted_roll_motor">
+      <hardwareInterface>PositionJointInterface</hardwareInterface>
+      <mechanicalReduction>1</mechanicalReduction>
+    </actuator>
+  </transmission>
+  <transmission name="tran5">
+    <type>transmission_interface/SimpleTransmission</type>
+    <joint name="hokuyo_mirror_roll1_joint">
+      <hardwareInterface>PositionJointInterface</hardwareInterface>
+    </joint>
+  <actuator name="hokuyo_mirror_roll1_motor">
+      <hardwareInterface>PositionJointInterface</hardwareInterface>
+      <mechanicalReduction>1</mechanicalReduction>
+    </actuator>
+  </transmission>
+  <transmission name="tran6">
+    <type>transmission_interface/SimpleTransmission</type>
+    <joint name="hokuyo_mirror_roll2_joint">
+      <hardwareInterface>PositionJointInterface</hardwareInterface>
+    </joint>
+  <actuator name="hokuyo_mirror_roll2_motor">
+      <hardwareInterface>PositionJointInterface</hardwareInterface>
+      <mechanicalReduction>1</mechanicalReduction>
+    </actuator>
+  </transmission>
+  <transmission name="tran7">
+    <type>transmission_interface/SimpleTransmission</type>
+    <joint name="hokuyo_tilted_prismatic_joint">
+      <hardwareInterface>PositionJointInterface</hardwareInterface>
+    </joint>
+  <actuator name="hokuyo_tilted_prismatic_joint">
+      <hardwareInterface>PositionJointInterface</hardwareInterface>
+      <mechanicalReduction>1</mechanicalReduction>
+    </actuator>
+  </transmission>
 </robot>
