Commit message: add mcl_3dl launch file

File: orne_box_description/urdf/orne_box_3d_lidar.urdf.xacro (robot description, xacro)
@@ -179,5 +179,5 @@
   <!-- Setting for imu -->
   <xacro:sensor_imu name="imu" parent="base_link" size="0.05 0.05 0.05">
-    <origin xyz="0.3 0 0.2445" rpy="0 0 ${-PI/2}"/>
+    <origin xyz="0.3 0 0.2445" rpy="${-PI} 0 ${-PI/2}"/>
   </xacro:sensor_imu>
   <xacro:include filename="$(find icart_mini_description)/urdf/sensors/hokuyo.urdf.xacro"/>

Commit message: add 3d lidar bringup launch file

File: orne_box_description/urdf/orne_box_3d_lidar.urdf.xacro (robot description, xacro)
@@ -179,5 +179,5 @@
   <!-- Setting for imu -->
   <xacro:sensor_imu name="imu" parent="base_link" size="0.05 0.05 0.05">
-    <origin xyz="0.3 0 0.2445" rpy="${-PI} 0 ${-PI/2}"/>
+    <origin xyz="0.374295 0.12 0.270" rpy="${-PI} 0 ${PI/2}"/>
   </xacro:sensor_imu>
   <xacro:include filename="$(find icart_mini_description)/urdf/sensors/hokuyo.urdf.xacro"/>
@@ -186,6 +186,6 @@
   </xacro:sensor_hokuyo>
   <xacro:include filename="$(find velodyne_description)/urdf/VLP-16.urdf.xacro"/>
-  <xacro:VLP-16 parent="base_link" name="velodyne" topic="/velodyne_points" organize_cloud="false" hz="10" samples="440" gpu="false">
-    <origin xyz="0 0 0.4" rpy="0 0 0" />
+  <xacro:VLP-16 parent="base_link" name="surestar" topic="/rfans_points" organize_cloud="false" hz="10" samples="440" gpu="false">
+    <origin xyz="0.23 0 0.40" rpy="0 0 0" />
   </xacro:VLP-16>
   <transmission name="tran1">

Commit message: changes orne_box_3d_lidar.urdf.xacro

File: orne_box_description/urdf/orne_box_3d_lidar.urdf.xacro (robot description, xacro)
@@ -1,211 +1,19 @@
 <?xml version="1.0" ?>
 <robot name="orne_box" xmlns:xacro="http://www.ros.org/wiki/xacro">
-  <xacro:property name="PI" value="3.1415926535897931"/>
-  <xacro:include filename="$(find icart_mini_description)/urdf/materials.xacro" />
-  <xacro:include filename="$(find orne_box_description)/urdf/orne_box.gazebo.xacro"/>
-  <link name="base_link">
-<!--
-    <visual>
-      <origin xyz="0 0 -0.154" rpy="0 0 0"/>
-      <geometry>
-        <mesh filename="package://orne_box_description/meshes/bases/orne_box_base.stl" scale="1 1 1"/>
-      </geometry>
-      <material name="orange"/>
-    </visual>
--->
-    <visual>
-      <origin xyz="0.090 0 0.1715" rpy="0 0 0"/>
-      <geometry>
-        <box size="0.400 0.404 0.202"/>
-      </geometry>
-      <material name="orange"/>
-    </visual>
-    <visual>
-      <origin xyz="0.36125 0 0.2625" rpy="0 0 0"/>
-      <geometry>
-        <box size="0.1425 0.404 0.020"/>
-      </geometry>
-      <material name="orange"/>
-    </visual>
-    <visual>
-      <origin xyz="0.35625 0 0.156" rpy="0 0 0"/>
-      <geometry>
-        <box size="0.1325 0.404 0.020"/>
-      </geometry>
-      <material name="orange"/>
-    </visual>
-    <visual>
-      <origin xyz="-0.120 0 0.4815" rpy="0 0 0"/>
-      <geometry>
-        <box size="0.020 0.404 0.822"/>
-      </geometry>
-      <material name="orange"/>
-    </visual>
-    <collision>
-      <origin xyz="0.090 0 0.1715" rpy="0 0 0"/>
-      <geometry>
-        <box size="0.400 0.404 0.202"/>
-      </geometry>
-    </collision>
-    <collision>
-      <origin xyz="0.36125 0 0.2625" rpy="0 0 0"/>
-      <geometry>
-        <box size="0.1425 0.404 0.020"/>
-      </geometry>
-    </collision>
-    <collision>
-      <origin xyz="0.35625 0 0.156" rpy="0 0 0"/>
-      <geometry>
-        <box size="0.1325 0.404 0.020"/>
-      </geometry>
-    </collision>
-    <collision>
-      <origin xyz="-0.120 0 0.4815" rpy="0 0 0"/>
-      <geometry>
-        <box size="0.020 0.404 0.822"/>
-      </geometry>
-    </collision>
-    <inertial>
-      <origin xyz="0.090 0 0.1715" rpy="0 0 0"/>
-      <mass value="25.0"/>
-      <inertia ixx="1.0" ixy="0.0" ixz="0.0" iyy="1.0" iyz="0.0" izz="1.0" />
-    </inertial>
-  </link>
-  <joint name="left_wheel_hinge" type="revolute">
-    <parent link="base_link"/>
-    <child link="wheel_left_link"/>
-    <origin xyz="0.0 0.23075 0.152" rpy="${-PI/2} 0 0"/>
-    <axis xyz="0 0 1"/>
-    <limit effort="100" velocity="100.0"  lower="-5000" upper="5000" />
-  </joint>
-  <link name="wheel_left_link">
-    <visual>
-      <origin xyz="0 0 0" rpy="0 0 0"/>
-      <geometry>
-        <mesh filename="package://orne_box_description/meshes/wheels/tire.stl" scale="1 1 1"/>
-      </geometry>
-<!--
-      <origin xyz="0 0 0" rpy="0 0 0"/>
-      <geometry>
-        <cylinder length="0.045" radius="0.152"/>
-      </geometry>
--->
-      <material name="white"/>
-    </visual>
-    <collision>
-      <origin xyz="0 0 0" rpy="0 0 0"/>
-      <geometry>
-        <cylinder length="0.045" radius="0.152"/>
-      </geometry>
-    </collision>
-    <inertial>
-      <origin xyz="0 0 0" />
-      <mass value="0.2" />
-      <inertia ixx="0.1" ixy="0.0" ixz="0.0" iyy="0.1" iyz="0.0" izz="0.1" />
-    </inertial>
-  </link>
-  <joint name="right_wheel_hinge" type="revolute">
-    <parent link="base_link"/>
-    <child link="wheel_right_link"/>
-    <origin xyz="0.0 -0.23075 0.152" rpy="${-PI/2} 0 0"/>
-    <axis xyz="0 0 1"/>
-    <limit effort="100" velocity="100.0"  lower="-5000" upper="5000" />
-  </joint>
-  <link name="wheel_right_link">
-    <visual>
-      <origin xyz="0 0 0" rpy="0 0 0"/>
-      <geometry>
-        <mesh filename="package://orne_box_description/meshes/wheels/tire.stl" scale="1 1 1"/>
-      </geometry>
-<!--
-      <origin xyz="0 0 0" rpy="0 0 0"/>
-      <geometry>
-        <cylinder length="0.045" radius="0.152"/>
-      </geometry>
--->
-      <material name="white"/>
-    </visual>
-    <collision>
-      <origin xyz="0 0 0" rpy="0 0 0"/>
-      <geometry>
-        <cylinder length="0.045" radius="0.152"/>
-      </geometry>
-    </collision>
-    <inertial>
-      <origin xyz="0 0 0" />
-      <mass value="0.2" />
-      <inertia ixx="0.1" ixy="0.0" ixz="0.0" iyy="0.1" iyz="0.0" izz="0.1" />
-    </inertial>
-  </link>
-  <joint name="caster_front_joint" type="fixed">
-    <parent link="base_link"/>
-    <child link="caster_front_link"/>
-    <origin xyz="0.362 0 0.050" rpy="0 0 0"/>
-  </joint>
-  <link name="caster_front_link">
-    <visual>
-      <origin xyz="0 0.150 0" rpy="${PI/2} 0 0"/>
-      <geometry>
-        <cylinder length="0.025" radius="0.050"/>
-      </geometry>
-      <material name="red"/>
-    </visual>
-    <visual>
-      <origin xyz="0 -0.150 0" rpy="${PI/2} 0 0"/>
-      <geometry>
-        <cylinder length="0.025" radius="0.050"/>
-      </geometry>
-      <material name="red"/>
-    </visual>
-    <collision>
-      <origin xyz="0 0.150 0" rpy="${PI/2} 0 0"/>
-      <geometry>
-        <cylinder length="0.025" radius="0.050"/>
-      </geometry>
-    </collision>
-    <collision>
-      <origin xyz="0 -0.150 0" rpy="${PI/2} 0 0"/>
-      <geometry>
-        <cylinder length="0.025" radius="0.050"/>
-      </geometry>
-    </collision>
-    <inertial>
-      <origin xyz="0 0 0" />
-      <mass value="0.2" />
-      <inertia ixx="0.1" ixy="0.0" ixz="0.0" iyy="0.1" iyz="0.0" izz="0.1" />
-    </inertial>
-  </link>
-  <xacro:include filename="$(find icart_mini_description)/urdf/sensors/imu.urdf.xacro"/>
-  <!-- Setting for imu -->
-  <xacro:sensor_imu name="imu" parent="base_link" size="0.05 0.05 0.05">
-    <origin xyz="0.374295 0.12 0.270" rpy="${-PI} 0 ${PI/2}"/>
-  </xacro:sensor_imu>
-  <xacro:include filename="$(find icart_mini_description)/urdf/sensors/hokuyo.urdf.xacro"/>
-  <xacro:sensor_hokuyo name="hokuyo" parent="base_link">
-    <origin xyz="0.374295 0 0.2185" rpy="${-PI} 0 0"/>
-  </xacro:sensor_hokuyo>
+  <xacro:include filename="$(find orne_box_description)/urdf/orne_box.urdf.xacro"/>
   <xacro:include filename="$(find velodyne_description)/urdf/VLP-16.urdf.xacro"/>
+  <xacro:include filename="$(find orne_box_description)/urdf/sensors/gnss.urdf.xacro"/>
+  <xacro:include filename="$(find orne_box_description)/urdf/sensors/camera.urdf.xacro"/>
+  <!-- Setting for 3D-LiDAR -->
   <xacro:VLP-16 parent="base_link" name="surestar" topic="/rfans_points" organize_cloud="false" hz="10" samples="440" gpu="false">
     <origin xyz="0.23 0 0.40" rpy="0 0 0" />
   </xacro:VLP-16>
-  <transmission name="tran1">
-    <type>transmission_interface/SimpleTransmission</type>
-    <joint name="left_wheel_hinge">
-      <hardwareInterface>VelocityJointInterface</hardwareInterface>
-    </joint>
-  <actuator name="left_motor">
-      <hardwareInterface>VelocityJointInterface</hardwareInterface>
-      <mechanicalReduction>1</mechanicalReduction>
-    </actuator>
-  </transmission>
-  <transmission name="tran2">
-    <type>transmission_interface/SimpleTransmission</type>
-    <joint name="right_wheel_hinge">
-      <hardwareInterface>VelocityJointInterface</hardwareInterface>
-    </joint>
-  <actuator name="right_motor">
-      <hardwareInterface>VelocityJointInterface</hardwareInterface>
-      <mechanicalReduction>1</mechanicalReduction>
-    </actuator>
-  </transmission>
+  <!-- Setting for GNSS -->
+  <xacro:sensor_gnss name="gnss" parent="base_link">
+    <origin xyz="-0.12 0.12 0.9" rpy="0 0 0"/>
+  </xacro:sensor_gnss>
+  <!-- Setting for Camera -->
+  <xacro:sensor_camera name="camera" parent="base_link">
+    <origin xyz="-0.08 0.0 0.8" rpy="0 0.38 0"/>
+  </xacro:sensor_camera>
 </robot>

Commit message: disabled VLP16 urdf for ignition gazebo

File: orne_box_description/urdf/orne_box_3d_lidar.urdf.xacro (robot description, xacro)
@@ -1,12 +1,16 @@
 <?xml version="1.0" ?>
 <robot name="orne_box" xmlns:xacro="http://www.ros.org/wiki/xacro">
+  <xacro:arg name="ignition_gazebo" default="false"/>
   <xacro:include filename="$(find orne_box_description)/urdf/orne_box.urdf.xacro"/>
-  <xacro:include filename="$(find velodyne_description)/urdf/VLP-16.urdf.xacro"/>
+  <!-- @TODO More clear boolean operation -->
+  <xacro:if value="${'$(arg ignition_gazebo)' == 'false'}">
+    <xacro:include filename="$(find velodyne_description)/urdf/VLP-16.urdf.xacro"/>
+    <!-- Setting for 3D-LiDAR -->
+    <xacro:VLP-16 parent="base_link" name="surestar" topic="/rfans_points" organize_cloud="false" hz="10" samples="440" gpu="false">
+      <origin xyz="0.23 0 0.40" rpy="0 0 0" />
+    </xacro:VLP-16>
+  </xacro:if>
   <xacro:include filename="$(find orne_box_description)/urdf/sensors/gnss.urdf.xacro"/>
   <xacro:include filename="$(find orne_box_description)/urdf/sensors/camera.urdf.xacro"/>
-  <!-- Setting for 3D-LiDAR -->
-  <xacro:VLP-16 parent="base_link" name="surestar" topic="/rfans_points" organize_cloud="false" hz="10" samples="440" gpu="false">
-    <origin xyz="0.23 0 0.40" rpy="0 0 0" />
-  </xacro:VLP-16>
   <!-- Setting for GNSS -->
   <xacro:sensor_gnss name="gnss" parent="base_link">
