Commit message: move base_link

File: orne_box_description/urdf/orne_box.urdf.xacro (robot description, xacro)
@@ -15,5 +15,5 @@
 -->
     <visual>
-      <origin xyz="0.090 0 0.0195" rpy="0 0 0"/>
+      <origin xyz="0.090 0 0.1715" rpy="0 0 0"/>
       <geometry>
         <box size="0.400 0.404 0.202"/>
@@ -22,5 +22,5 @@
     </visual>
     <visual>
-      <origin xyz="0.36125 0 0.1105" rpy="0 0 0"/>
+      <origin xyz="0.36125 0 0.2625" rpy="0 0 0"/>
       <geometry>
         <box size="0.1425 0.404 0.020"/>
@@ -29,5 +29,5 @@
     </visual>
     <visual>
-      <origin xyz="0.35625 0 0.004" rpy="0 0 0"/>
+      <origin xyz="0.35625 0 0.156" rpy="0 0 0"/>
       <geometry>
         <box size="0.1325 0.404 0.020"/>
@@ -36,5 +36,5 @@
     </visual>
     <visual>
-      <origin xyz="-0.120 0 0.3295" rpy="0 0 0"/>
+      <origin xyz="-0.120 0 0.4815" rpy="0 0 0"/>
       <geometry>
         <box size="0.020 0.404 0.822"/>
@@ -43,5 +43,5 @@
     </visual>
     <collision>
-      <origin xyz="0.090 0 0.0195" rpy="0 0 0"/>
+      <origin xyz="0.090 0 0.1715" rpy="0 0 0"/>
       <geometry>
         <box size="0.400 0.404 0.202"/>
@@ -49,5 +49,5 @@
     </collision>
     <collision>
-      <origin xyz="0.36125 0 0.1105" rpy="0 0 0"/>
+      <origin xyz="0.36125 0 0.2625" rpy="0 0 0"/>
       <geometry>
         <box size="0.1425 0.404 0.020"/>
@@ -55,5 +55,5 @@
     </collision>
     <collision>
-      <origin xyz="0.35625 0 0.004" rpy="0 0 0"/>
+      <origin xyz="0.35625 0 0.156" rpy="0 0 0"/>
       <geometry>
         <box size="0.1325 0.404 0.020"/>
@@ -61,5 +61,5 @@
     </collision>
     <collision>
-      <origin xyz="-0.120 0 0.3295" rpy="0 0 0"/>
+      <origin xyz="-0.120 0 0.4815" rpy="0 0 0"/>
       <geometry>
         <box size="0.020 0.404 0.822"/>
@@ -67,5 +67,5 @@
     </collision>
     <inertial>
-      <origin xyz="0.090 0 0.0195" rpy="0 0 0"/>
+      <origin xyz="0.090 0 0.1715" rpy="0 0 0"/>
       <mass value="25.0"/>
       <inertia ixx="1.0" ixy="0.0" ixz="0.0" iyy="1.0" iyz="0.0" izz="1.0" />
@@ -75,5 +75,5 @@
     <parent link="base_link"/>
     <child link="wheel_left_link"/>
-    <origin xyz="0.0 0.23075 0.0" rpy="${-PI/2} 0 0"/>
+    <origin xyz="0.0 0.23075 0.152" rpy="${-PI/2} 0 0"/>
     <axis xyz="0 0 1"/>
     <limit effort="100" velocity="100.0"  lower="-5000" upper="5000" />
@@ -108,5 +108,5 @@
     <parent link="base_link"/>
     <child link="wheel_right_link"/>
-    <origin xyz="0.0 -0.23075 0.0" rpy="${-PI/2} 0 0"/>
+    <origin xyz="0.0 -0.23075 0.152" rpy="${-PI/2} 0 0"/>
     <axis xyz="0 0 1"/>
     <limit effort="100" velocity="100.0"  lower="-5000" upper="5000" />
@@ -141,5 +141,5 @@
     <parent link="base_link"/>
     <child link="caster_front_link"/>
-    <origin xyz="0.362 0 -0.102" rpy="0 0 0"/>
+    <origin xyz="0.362 0 0.050" rpy="0 0 0"/>
   </joint>
   <link name="caster_front_link">
@@ -179,9 +179,9 @@
   <!-- Setting for imu -->
   <xacro:sensor_imu name="imu" parent="base_link" size="0.05 0.05 0.05">
-    <origin xyz="0.3 0 0.0925" rpy="0 0 ${-PI/2}"/>
+    <origin xyz="0.3 0 0.2445" rpy="0 0 ${-PI/2}"/>
   </xacro:sensor_imu>
   <xacro:include filename="$(find icart_mini_description)/urdf/sensors/hokuyo.urdf.xacro"/>
   <xacro:sensor_hokuyo name="hokuyo" parent="base_link">
-    <origin xyz="0.374295 0 0.0665" rpy="${-PI} 0 0"/>
+    <origin xyz="0.374295 0 0.2185" rpy="${-PI} 0 0"/>
   </xacro:sensor_hokuyo>
   <transmission name="tran1">

Commit message: test

File: orne_box_description/urdf/orne_box.urdf.xacro (robot description, xacro)
@@ -61,5 +61,5 @@
   <link name="lidar_with_mirror_prismatic_link">
     <inertial>
-      <origin xyz="0 0 0" />
+      <origin xyz="0 0 0"/>
       <mass value="0.2" />
       <inertia ixx="0.1" ixy="0.0" ixz="0.0" iyy="0.1" iyz="0.0" izz="0.1" />
@@ -69,5 +69,5 @@
     <parent link="lidar_with_mirror_prismatic_link"/>
     <child link="lidar_with_mirror_pitch_link"/>
-    <origin xyz="0 0 0" rpy="0 ${PI/9} 0"/>
+    <origin xyz="0 0 0" rpy="0 ${PI/12} 0"/>
     <axis xyz="0 1 0"/>
     <limit effort="100" velocity="100.0" lower="${-PI}" upper="${PI}" />

Commit message: fix

File: orne_box_description/urdf/orne_box.urdf.xacro (robot description, xacro)
@@ -98,5 +98,5 @@
   <xacro:property name="height" value="0" />
   <xacro:sensor_hokuyo name="lidar_with_mirror_center" parent="lidar_with_mirror_roll_link" size="0.05 0.05 0.05">
-    <origin xyz="${front} 0 ${height}" rpy="0 0 0"/>
+    <origin xyz="${front} 0 ${height}" rpy="${PI} 0 0"/>
   </xacro:sensor_hokuyo>
   <joint name="lidar_with_mirror_mirror1_roll_joint" type="fixed">

Commit message: changes orne_box.urdf.xacro

File: orne_box_description/urdf/orne_box.urdf.xacro (robot description, xacro)
@@ -2,206 +2,43 @@
 <robot name="orne_box" xmlns:xacro="http://www.ros.org/wiki/xacro">
   <xacro:property name="PI" value="3.1415926535897931"/>
-  <xacro:include filename="$(find icart_mini_description)/urdf/materials.xacro" />
+  <xacro:include filename="$(find orne_box_description)/urdf/material_colors.xacro" />
   <xacro:include filename="$(find orne_box_description)/urdf/orne_box.gazebo.xacro"/>
-  <link name="base_link">
-<!--
-    <visual>
-      <origin xyz="0 0 -0.154" rpy="0 0 0"/>
-      <geometry>
-        <mesh filename="package://orne_box_description/meshes/bases/orne_box_base.stl" scale="1 1 1"/>
-      </geometry>
-      <material name="orange"/>
-    </visual>
--->
-    <visual>
-      <origin xyz="0.090 0 0.1715" rpy="0 0 0"/>
-      <geometry>
-        <box size="0.400 0.404 0.202"/>
-      </geometry>
-      <material name="orange"/>
-    </visual>
-    <visual>
-      <origin xyz="0.36125 0 0.2625" rpy="0 0 0"/>
-      <geometry>
-        <box size="0.1425 0.404 0.020"/>
-      </geometry>
-      <material name="orange"/>
-    </visual>
-    <visual>
-      <origin xyz="0.35625 0 0.156" rpy="0 0 0"/>
-      <geometry>
-        <box size="0.1325 0.404 0.020"/>
-      </geometry>
-      <material name="orange"/>
-    </visual>
-    <visual>
-      <origin xyz="-0.120 0 0.4815" rpy="0 0 0"/>
-      <geometry>
-        <box size="0.020 0.404 0.822"/>
-      </geometry>
-      <material name="orange"/>
-    </visual>
-    <collision>
-      <origin xyz="0.090 0 0.1715" rpy="0 0 0"/>
-      <geometry>
-        <box size="0.400 0.404 0.202"/>
-      </geometry>
-    </collision>
-    <collision>
-      <origin xyz="0.36125 0 0.2625" rpy="0 0 0"/>
-      <geometry>
-        <box size="0.1425 0.404 0.020"/>
-      </geometry>
-    </collision>
-    <collision>
-      <origin xyz="0.35625 0 0.156" rpy="0 0 0"/>
-      <geometry>
-        <box size="0.1325 0.404 0.020"/>
-      </geometry>
-    </collision>
-    <collision>
-      <origin xyz="-0.120 0 0.4815" rpy="0 0 0"/>
-      <geometry>
-        <box size="0.020 0.404 0.822"/>
-      </geometry>
-    </collision>
-    <inertial>
-      <origin xyz="0.090 0 0.1715" rpy="0 0 0"/>
-      <mass value="25.0"/>
-      <inertia ixx="1.0" ixy="0.0" ixz="0.0" iyy="1.0" iyz="0.0" izz="1.0" />
-    </inertial>
-  </link>
-  <joint name="left_wheel_hinge" type="revolute">
-    <parent link="base_link"/>
-    <child link="wheel_left_link"/>
+  <xacro:include filename="$(find orne_box_description)/urdf/links/base_link.urdf.xacro"/>
+  <xacro:include filename="$(find orne_box_description)/urdf/links/caster_link.urdf.xacro"/>
+  <xacro:include filename="$(find orne_box_description)/urdf/links/wheel_link.urdf.xacro"/>
+  <xacro:include filename="$(find orne_box_description)/urdf/joints/caster_joint.urdf.xacro"/>
+  <xacro:include filename="$(find orne_box_description)/urdf/joints/wheel_joint.urdf.xacro"/>
+  <xacro:include filename="$(find orne_box_description)/urdf/sensors/imu.urdf.xacro"/>
+  <xacro:include filename="$(find orne_box_description)/urdf/sensors/hokuyo.urdf.xacro"/>
+  <!-- Setting for base -->
+	<xacro:base_link/>
+  <!-- Setting for caster -->
+  <xacro:caster_joint parent="base_link">
+    <origin xyz="0.362 0.0 0.050" rpy="0 0 0"/>
+  </xacro:caster_joint>
+	<xacro:caster_link/>
+  <!-- Setting for left wheel -->
+  <xacro:wheel_joint prefix="left" parent="base_link">
     <origin xyz="0.0 0.23075 0.152" rpy="${-PI/2} 0 0"/>
     <axis xyz="0 0 1"/>
-    <limit effort="100" velocity="100.0"  lower="-5000" upper="5000" />
-  </joint>
-  <link name="wheel_left_link">
-    <visual>
-      <origin xyz="0 0 0" rpy="0 0 0"/>
-      <geometry>
-        <mesh filename="package://orne_box_description/meshes/wheels/tire.stl" scale="1 1 1"/>
-      </geometry>
-<!--
-      <origin xyz="0 0 0" rpy="0 0 0"/>
-      <geometry>
-        <cylinder length="0.045" radius="0.152"/>
-      </geometry>
--->
-      <material name="white"/>
-    </visual>
-    <collision>
-      <origin xyz="0 0 0" rpy="0 0 0"/>
-      <geometry>
-        <cylinder length="0.045" radius="0.152"/>
-      </geometry>
-    </collision>
-    <inertial>
-      <origin xyz="0 0 0" />
-      <mass value="0.2" />
-      <inertia ixx="0.1" ixy="0.0" ixz="0.0" iyy="0.1" iyz="0.0" izz="0.1" />
-    </inertial>
-  </link>
-  <joint name="right_wheel_hinge" type="revolute">
-    <parent link="base_link"/>
-    <child link="wheel_right_link"/>
+  </xacro:wheel_joint>
+  <xacro:wheel_link prefix="left" width="0.045" radius="0.152">
+    <origin xyz="0.0 0.0 0.0" rpy="0 0 0"/>
+  </xacro:wheel_link>
+  <!-- Setting for right wheel -->
+  <xacro:wheel_joint prefix="right" parent="base_link">
     <origin xyz="0.0 -0.23075 0.152" rpy="${-PI/2} 0 0"/>
     <axis xyz="0 0 1"/>
-    <limit effort="100" velocity="100.0"  lower="-5000" upper="5000" />
-  </joint>
-  <link name="wheel_right_link">
-    <visual>
-      <origin xyz="0 0 0" rpy="0 0 0"/>
-      <geometry>
-        <mesh filename="package://orne_box_description/meshes/wheels/tire.stl" scale="1 1 1"/>
-      </geometry>
-<!--
-      <origin xyz="0 0 0" rpy="0 0 0"/>
-      <geometry>
-        <cylinder length="0.045" radius="0.152"/>
-      </geometry>
--->
-      <material name="white"/>
-    </visual>
-    <collision>
-      <origin xyz="0 0 0" rpy="0 0 0"/>
-      <geometry>
-        <cylinder length="0.045" radius="0.152"/>
-      </geometry>
-    </collision>
-    <inertial>
-      <origin xyz="0 0 0" />
-      <mass value="0.2" />
-      <inertia ixx="0.1" ixy="0.0" ixz="0.0" iyy="0.1" iyz="0.0" izz="0.1" />
-    </inertial>
-  </link>
-  <joint name="caster_front_joint" type="fixed">
-    <parent link="base_link"/>
-    <child link="caster_front_link"/>
-    <origin xyz="0.362 0 0.050" rpy="0 0 0"/>
-  </joint>
-  <link name="caster_front_link">
-    <visual>
-      <origin xyz="0 0.150 0" rpy="${PI/2} 0 0"/>
-      <geometry>
-        <cylinder length="0.025" radius="0.050"/>
-      </geometry>
-      <material name="red"/>
-    </visual>
-    <visual>
-      <origin xyz="0 -0.150 0" rpy="${PI/2} 0 0"/>
-      <geometry>
-        <cylinder length="0.025" radius="0.050"/>
-      </geometry>
-      <material name="red"/>
-    </visual>
-    <collision>
-      <origin xyz="0 0.150 0" rpy="${PI/2} 0 0"/>
-      <geometry>
-        <cylinder length="0.025" radius="0.050"/>
-      </geometry>
-    </collision>
-    <collision>
-      <origin xyz="0 -0.150 0" rpy="${PI/2} 0 0"/>
-      <geometry>
-        <cylinder length="0.025" radius="0.050"/>
-      </geometry>
-    </collision>
-    <inertial>
-      <origin xyz="0 0 0" />
-      <mass value="0.2" />
-      <inertia ixx="0.1" ixy="0.0" ixz="0.0" iyy="0.1" iyz="0.0" izz="0.1" />
-    </inertial>
-  </link>
-  <xacro:include filename="$(find icart_mini_description)/urdf/sensors/imu.urdf.xacro"/>
-  <!-- Setting for imu -->
+  </xacro:wheel_joint>
+  <xacro:wheel_link prefix="right" width="0.045" radius="0.152">
+    <origin xyz="0.0 0.0 0.0" rpy="0 0 0"/>
+  </xacro:wheel_link>
+  <!-- Setting for IMU -->
   <xacro:sensor_imu name="imu" parent="base_link" size="0.05 0.05 0.05">
-    <origin xyz="0.3 0 0.2445" rpy="0 0 ${-PI/2}"/>
+    <origin xyz="0.23 0.0 0.270" rpy="${-PI} 0 ${PI/2}"/>
   </xacro:sensor_imu>
-  <xacro:include filename="$(find icart_mini_description)/urdf/sensors/hokuyo.urdf.xacro"/>
-  <xacro:sensor_hokuyo name="hokuyo" parent="base_link">
+  <!-- Setting for 2D-LiDAR -->
+  <xacro:sensor_hokuyo name="hokuyo" parent="base_link" size="0.05 0.05 0.05">
     <origin xyz="0.374295 0 0.2185" rpy="${-PI} 0 0"/>
   </xacro:sensor_hokuyo>
-  <transmission name="tran1">
-    <type>transmission_interface/SimpleTransmission</type>
-    <joint name="left_wheel_hinge">
-      <hardwareInterface>VelocityJointInterface</hardwareInterface>
-    </joint>
-  <actuator name="left_motor">
-      <hardwareInterface>VelocityJointInterface</hardwareInterface>
-      <mechanicalReduction>1</mechanicalReduction>
-    </actuator>
-  </transmission>
-  <transmission name="tran2">
-    <type>transmission_interface/SimpleTransmission</type>
-    <joint name="right_wheel_hinge">
-      <hardwareInterface>VelocityJointInterface</hardwareInterface>
-    </joint>
-  <actuator name="right_motor">
-      <hardwareInterface>VelocityJointInterface</hardwareInterface>
-      <mechanicalReduction>1</mechanicalReduction>
-    </actuator>
-  </transmission>
 </robot>

Commit message: 実験走行11_04

File: orne_box_description/urdf/orne_box.urdf.xacro (robot description, xacro)
@@ -55,5 +55,4 @@
   <xacro:sensor_hokuyo name="low_hokuyo" parent="base_link" size="0.05 0.05 0.05">
     <origin xyz="0.374295 0 0.2185" rpy="${-PI} 0 0"/>
-    <!--origin xyz="0.23 0 0.4" rpy="0 0 0"/-->
   </xacro:sensor_hokuyo>
 </robot>

File: orne_box_description/urdf/orne_box_3d_lidar.urdf.xacro (robot description, xacro)
@@ -75,4 +75,6 @@
   <xacro:include filename="$(find orne_box_description)/urdf/sensors/gnss.urdf.xacro"/>
   <xacro:include filename="$(find orne_box_description)/urdf/sensors/camera.urdf.xacro"/>
+  <!--xacro:include filename="$(find orne_box_description)/urdf/sensors/hokuyo.urdf.xacro"/-->
+  <!--xacro:include filename="$(find orne_box_description)/urdf/sensors/imu.urdf.xacro"/-->
   <!-- Setting for GNSS -->
   <xacro:sensor_gnss name="gnss" parent="base_link">
@@ -83,3 +85,9 @@
     <origin xyz="-0.08 0.0 0.8" rpy="0 0.38 0"/>
   </xacro:sensor_camera>
+  <!--xacro:sensor_hokuyo name="low_hokuyo" parent="base_link" size="0.05 0.05 0.05">
+    <origin xyz="0.374295 0 0.2185" rpy="${-PI} 0 0"/>
+  </xacro:sensor_hokuyo-->
+ <!--xacro:sensor_imu name="imu" parent="base_link" size="0.05 0.05 0.05">
+    <origin xyz="0.23 0.0 0.270" rpy="${-PI} 0 ${PI/2}"/>
+  </xacro:sensor_imu-->
 </robot>

Commit message: update front caster

File: orne_box_description/urdf/orne_box.urdf.xacro (robot description, xacro)
@@ -6,6 +6,10 @@
   <xacro:include filename="$(find orne_box_description)/urdf/links/base_link.urdf.xacro"/>
   <xacro:include filename="$(find orne_box_description)/urdf/links/caster_link.urdf.xacro"/>
+  <xacro:include filename="$(find orne_box_description)/urdf/links/caster_wheel_link.urdf.xacro"/>
+  <xacro:include filename="$(find orne_box_description)/urdf/links/caster_swivel_link.urdf.xacro"/>
   <xacro:include filename="$(find orne_box_description)/urdf/links/wheel_link.urdf.xacro"/>
   <xacro:include filename="$(find orne_box_description)/urdf/joints/caster_joint.urdf.xacro"/>
+  <xacro:include filename="$(find orne_box_description)/urdf/joints/caster_wheel_joint.urdf.xacro"/>
+  <xacro:include filename="$(find orne_box_description)/urdf/joints/caster_swivel_joint.urdf.xacro"/>
   <xacro:include filename="$(find orne_box_description)/urdf/joints/wheel_joint.urdf.xacro"/>
   <xacro:include filename="$(find orne_box_description)/urdf/sensors/imu.urdf.xacro"/>
@@ -14,8 +18,22 @@
   <xacro:base_link/>
   <!-- Setting for caster -->
+  <!--
   <xacro:caster_joint parent="base_link">
     <origin xyz="0.362 0.0 0.050" rpy="0 0 0"/>
   </xacro:caster_joint>
   <xacro:caster_link/>
+  -->
+  <xacro:caster_wheel_link prefix="left"/>
+  <xacro:caster_swivel_link prefix="left"/>
+  <xacro:caster_wheel_joint prefix="left"/>
+  <xacro:caster_swivel_joint prefix="left" parent="base_link">
+    <origin xyz="0.362 0.150 0.12" rpy="0 0 0"/>
+  </xacro:caster_swivel_joint>
+  <xacro:caster_wheel_link prefix="right"/>
+  <xacro:caster_swivel_link prefix="right"/>
+  <xacro:caster_wheel_joint prefix="right"/>
+  <xacro:caster_swivel_joint prefix="right" parent="base_link">
+    <origin xyz="0.362 -0.150 0.12" rpy="0 0 0"/>
+  </xacro:caster_swivel_joint>
   <!-- Setting for left wheel -->
   <xacro:wheel_joint prefix="left" parent="base_link">

Commit message: 実験走行パラメータ

File: orne_box_description/urdf/orne_box.urdf.xacro (robot description, xacro)
@@ -52,3 +52,6 @@
     <origin xyz="0.374295 0 0.2185" rpy="${-PI} 0 0"/>
   </xacro:sensor_hokuyo>
+  <xacro:sensor_hokuyo name="mirror_lidar" parent="base_link" size="0.05 0.05 0.05">
+    <origin xyz="-0.08 0.0 0.7" rpy="${-PI} 0.175 0"/>
+  </xacro:sensor_hokuyo>
 </robot>

Commit message: fixed mirror lidar link

File: orne_box_description/urdf/orne_box.urdf.xacro (robot description, xacro)
@@ -52,8 +52,8 @@
     <origin xyz="0.374295 0 0.2185" rpy="${-PI} 0 0"/>
   </xacro:sensor_hokuyo>
-  <joint name="lidar_with_mirror_prismatic_joint" type="prismatic">
+  <joint name="lidar_with_mirror_prismatic_joint" type="fixed">
     <parent link="base_link"/>
     <child link="lidar_with_mirror_prismatic_link"/>
-    <origin xyz="1.0 0 0.3" rpy="0 0 0"/>
+    <origin xyz="-0.15 0 0.56" rpy="0 0 0"/>
     <axis xyz="0 0 1"/>
     <limit effort="100" velocity="100.0" lower="-0.3" upper="1" />
@@ -66,5 +66,5 @@
     </inertial>
   </link>
-  <joint name="lidar_with_mirror_pitch_joint" type="revolute">
+  <joint name="lidar_with_mirror_pitch_joint" type="fixed">
     <parent link="lidar_with_mirror_prismatic_link"/>
     <child link="lidar_with_mirror_pitch_link"/>
@@ -80,5 +80,5 @@
     </inertial>
   </link>
-  <joint name="lidar_with_mirror_roll_joint" type="revolute">
+  <joint name="lidar_with_mirror_roll_joint" type="fixed">
     <parent link="lidar_with_mirror_pitch_link"/>
     <child link="lidar_with_mirror_roll_link"/>
@@ -100,5 +100,5 @@
     <origin xyz="${front} 0 ${height}" rpy="0 0 0"/>
   </xacro:sensor_hokuyo>
-  <joint name="lidar_with_mirror_mirror1_roll_joint" type="revolute">
+  <joint name="lidar_with_mirror_mirror1_roll_joint" type="fixed">
     <parent link="lidar_with_mirror_center_link"/>
     <child link="lidar_with_mirror_mirror1_roll_link"/>
@@ -117,5 +117,5 @@
     <origin xyz="0 ${-len} 0" rpy="0 0 0"/>
   </xacro:sensor_hokuyo>
-  <joint name="lidar_with_mirror_mirror2_roll_joint" type="revolute">
+  <joint name="lidar_with_mirror_mirror2_roll_joint" type="fixed">
     <parent link="lidar_with_mirror_center_link"/>
     <child link="lidar_with_mirror_mirror2_roll_link"/>
