Commit message: fix urdf

File: orne_box_description/urdf/orne_box.urdf.xacro (robot description, xacro)
@@ -13,4 +13,5 @@
   <xacro:include filename="$(find orne_box_description)/urdf/sensors/imu.urdf.xacro"/>
   <xacro:include filename="$(find orne_box_description)/urdf/sensors/hokuyo.urdf.xacro"/>
+  <xacro:include filename="$(find orne_box_description)/urdf/sensors/lidar_with_mirror.urdf.xacro" />
   <!-- Setting for base -->
   <xacro:base_link/>
@@ -52,85 +53,7 @@
     <origin xyz="0.374295 0 0.2185" rpy="${-PI} 0 0"/>
   </xacro:sensor_hokuyo>
-  <joint name="lidar_with_mirror_prismatic_joint" type="fixed">
-    <parent link="base_link"/>
-    <child link="lidar_with_mirror_prismatic_link"/>
+  <!-- Setting for mirror_lidar -->
+  <xacro:lidar_with_mirror name="lidar_with_mirror" parent="base_link" left_roll_rad="0.769999299112962" left_pitch_rad="-0.05" left_distance_m="0.073124500184212" right_roll_rad="0.787426157712581" right_pitch_rad="-0.05" right_distance_m="0.072588298861567">
     <origin xyz="-0.15 0 0.56" rpy="0 0 0"/>
-    <axis xyz="0 0 1"/>
-    <limit effort="100" velocity="100.0" lower="-0.3" upper="1" />
-  </joint>
-  <link name="lidar_with_mirror_prismatic_link">
-    <inertial>
-      <origin xyz="0 0 0"/>
-      <mass value="0.2" />
-      <inertia ixx="0.1" ixy="0.0" ixz="0.0" iyy="0.1" iyz="0.0" izz="0.1" />
-    </inertial>
-  </link>
-  <joint name="lidar_with_mirror_pitch_joint" type="fixed">
-    <parent link="lidar_with_mirror_prismatic_link"/>
-    <child link="lidar_with_mirror_pitch_link"/>
-    <origin xyz="0 0 0" rpy="0 ${PI/12} 0"/>
-    <axis xyz="0 1 0"/>
-    <limit effort="100" velocity="100.0" lower="${-PI}" upper="${PI}" />
-  </joint>
-  <link name="lidar_with_mirror_pitch_link">
-    <inertial>
-      <origin xyz="0 0 0" />
-      <mass value="0.2" />
-      <inertia ixx="0.1" ixy="0.0" ixz="0.0" iyy="0.1" iyz="0.0" izz="0.1" />
-    </inertial>
-  </link>
-  <joint name="lidar_with_mirror_roll_joint" type="fixed">
-    <parent link="lidar_with_mirror_pitch_link"/>
-    <child link="lidar_with_mirror_roll_link"/>
-    <origin xyz="0 0 0" rpy="0 0 0"/>
-    <axis xyz="1 0 0"/>
-    <limit effort="100" velocity="100.0" lower="${-PI}" upper="${PI}" />
-  </joint>
-  <link name="lidar_with_mirror_roll_link">
-    <inertial>
-      <origin xyz="0 0 0" />
-      <mass value="0.2" />
-      <inertia ixx="0.1" ixy="0.0" ixz="0.0" iyy="0.1" iyz="0.0" izz="0.1" />
-    </inertial>
-  </link>
-  <xacro:property name="len" value="0.1" />
-  <xacro:property name="front" value="0" />
-  <xacro:property name="height" value="0" />
-  <xacro:sensor_hokuyo name="lidar_with_mirror_center" parent="lidar_with_mirror_roll_link" size="0.05 0.05 0.05">
-    <origin xyz="${front} 0 ${height}" rpy="${PI} 0 0"/>
-  </xacro:sensor_hokuyo>
-  <joint name="lidar_with_mirror_mirror1_roll_joint" type="fixed">
-    <parent link="lidar_with_mirror_center_link"/>
-    <child link="lidar_with_mirror_mirror1_roll_link"/>
-    <origin xyz="0 ${len} 0" rpy="${-PI/4} 0 0"/>
-    <axis xyz="-1 0 0"/>
-    <limit effort="100" velocity="100.0" lower="${-PI}" upper="${PI}" />
-  </joint>
-  <link name="lidar_with_mirror_mirror1_roll_link">
-    <inertial>
-      <origin xyz="0 0 0" />
-      <mass value="0.2" />
-      <inertia ixx="0.1" ixy="0.0" ixz="0.0" iyy="0.1" iyz="0.0" izz="0.1" />
-    </inertial>
-  </link>
-  <xacro:sensor_hokuyo name="lidar_with_mirror_left" parent="lidar_with_mirror_mirror1_roll_link" size="0.05 0.05 0.05">
-    <origin xyz="0 ${-len} 0" rpy="0 0 0"/>
-  </xacro:sensor_hokuyo>
-  <joint name="lidar_with_mirror_mirror2_roll_joint" type="fixed">
-    <parent link="lidar_with_mirror_center_link"/>
-    <child link="lidar_with_mirror_mirror2_roll_link"/>
-    <origin xyz="0 ${-len} 0" rpy="${PI/4} 0 0"/>
-    <axis xyz="1 0 0"/>
-    <limit effort="100" velocity="100.0" lower="${-PI}" upper="${PI}" />
-  </joint>
-  <link name="lidar_with_mirror_mirror2_roll_link">
-    <inertial>
-      <origin xyz="0 0 0" />
-      <mass value="0.2" />
-      <inertia ixx="0.1" ixy="0.0" ixz="0.0" iyy="0.1" iyz="0.0" izz="0.1" />
-    </inertial>
-  </link>
-  <xacro:sensor_hokuyo name="lidar_with_mirror_right" parent="lidar_with_mirror_mirror2_roll_link" size="0.05 0.05 0.05">
-    <origin xyz="0 ${len} 0" rpy="0 0 0"/>
-  </xacro:sensor_hokuyo>
+  </xacro:lidar_with_mirror>
 </robot>

File: orne_box_description/urdf/sensors/hokuyo.urdf.xacro (robot description, xacro)
@@ -4,5 +4,5 @@
     <joint name="${name}_joint" type="fixed">
       <axis xyz="1 0 0"/>
-      <xacro:insert_block name="origin"/>
+      <xacro:insert_block name="origin">
       <parent link="${parent}"/>
       <child link="${name}_link"/>

Commit message: experimental params

File: orne_box_description/urdf/orne_box.urdf.xacro (robot description, xacro)
@@ -55,5 +55,5 @@
   <!-- Setting for mirror_lidar -->
   <xacro:lidar_with_mirror name="lidar_with_mirror" parent="base_link" left_roll_rad="0.769999299112962" left_pitch_rad="-0.05" left_distance_m="0.073124500184212" right_roll_rad="0.787426157712581" right_pitch_rad="-0.05" right_distance_m="0.072588298861567">
-    <origin xyz="-0.15 0 0.56" rpy="0 0 0"/>
+    <origin xyz="-0.15 0 0.56" rpy="0 ${PI/12} 0"/>
   </xacro:lidar_with_mirror>
 </robot>

Commit message: 上の2D-LiDARの追加

File: orne_box_description/urdf/orne_box.urdf.xacro (robot description, xacro)
@@ -50,5 +50,6 @@
   <!-- Setting for 2D-LiDAR -->
   <xacro:sensor_hokuyo name="hokuyo" parent="base_link" size="0.05 0.05 0.05">
-    <origin xyz="0.374295 0 0.2185" rpy="${-PI} 0 0"/>
+    <!--origin xyz="0.374295 0 0.2185" rpy="${-PI} 0 0"/-->
+    <origin xyz="0.23 0 0.4" rpy="0 0 0"/>
   </xacro:sensor_hokuyo>
   <xacro:sensor_hokuyo name="mirror_lidar" parent="base_link" size="0.05 0.05 0.05">

Commit message: 競合点の修正

File: orne_box_description/urdf/orne_box.urdf.xacro (robot description, xacro)
@@ -50,9 +50,6 @@
   <!-- Setting for 2D-LiDAR -->
   <xacro:sensor_hokuyo name="hokuyo" parent="base_link" size="0.05 0.05 0.05">
-    <!--origin xyz="0.374295 0 0.2185" rpy="${-PI} 0 0"/-->
-    <origin xyz="0.23 0 0.4" rpy="0 0 0"/>
-  </xacro:sensor_hokuyo>
-  <xacro:sensor_hokuyo name="mirror_lidar" parent="base_link" size="0.05 0.05 0.05">
-    <origin xyz="-0.08 0.0 0.7" rpy="${-PI} 0.175 0"/>
+    <origin xyz="0.374295 0 0.2185" rpy="${-PI} 0 0"/>
+    <!--origin xyz="0.23 0 0.4" rpy="0 0 0"/-->
   </xacro:sensor_hokuyo>
 </robot>

Commit message: LiDAR追加

File: orne_box_description/urdf/orne_box.urdf.xacro (robot description, xacro)
@@ -50,4 +50,8 @@
   <!-- Setting for 2D-LiDAR -->
   <xacro:sensor_hokuyo name="hokuyo" parent="base_link" size="0.05 0.05 0.05">
+    <origin xyz="0.23 0 0.35" rpy="0 0 0"/>
+    <!--origin xyz="0.23 0 0.4" rpy="0 0 0"/-->
+  </xacro:sensor_hokuyo>
+  <xacro:sensor_hokuyo name="low_hokuyo" parent="base_link" size="0.05 0.05 0.05">
     <origin xyz="0.374295 0 0.2185" rpy="${-PI} 0 0"/>
     <!--origin xyz="0.23 0 0.4" rpy="0 0 0"/-->

Commit message: fix imu rpy for box3

File: orne_box_description/urdf/orne_box.urdf.xacro (robot description, xacro)
@@ -45,6 +45,10 @@
   </xacro:wheel_link>
   <!-- Setting for IMU -->
+  <!-- <xacro:sensor_imu name="imu" parent="base_link" size="0.05 0.05 0.05">
+    <origin xyz="0.23 0.0 0.270" rpy="${-PI} 0 ${PI/2}"/>
+  </xacro:sensor_imu> -->
   <xacro:sensor_imu name="imu" parent="base_link" size="0.05 0.05 0.05">
-    <origin xyz="0.23 0.0 0.270" rpy="${-PI} 0 ${PI/2}"/>
+    <origin xyz="0.23 0.0 0.270" rpy="0 0 0"/>
+    <origin_child xyz="0.0 0.0 0.0" rpy="0 0 0"/>
   </xacro:sensor_imu>
   <!-- Setting for 2D-LiDAR -->

File: orne_box_description/urdf/sensors/imu.urdf.xacro (robot description, xacro)
@@ -1,5 +1,5 @@
 <?xml version="1.0"?>
 <robot xmlns:xacro="http://ros.org/wiki/xacro" xmlns:controller="http://playerstage.sourceforge.net/gazebo/xmlschema/#controller" xmlns:interface="http://playerstage.sourceforge.net/gazebo/xmlschema/#interface" name="sensor_imu">
-  <xacro:macro name="sensor_imu" params="name parent *origin size">
+  <xacro:macro name="sensor_imu" params="name parent *origin *origin_child size">
     <joint name="${name}_joint" type="fixed">
       <axis xyz="1 0 0"/>
@@ -16,14 +16,14 @@
       </inertial>
       <visual>
-        <origin rpy="0 0 0" xyz="0 0 0"/>
+        <!-- <origin rpy="0 0 0" xyz="0 0 0"/>
         <geometry>
           <box size="${size}"/>
         </geometry>
-        <material name="green"/>
+        <material name="green"/> -->
       </visual>
     </link>
     <joint name="${name}_base_joint" type="fixed">
       <axis xyz="1 0 0"/>
-      <xacro:insert_block name="origin"/>
+      <xacro:insert_block name="origin_child"/>
       <parent link="${name}_link"/>
       <child link="${name}"/>

Commit message: add mirror lidar.launch.py

File: orne_box_description/urdf/orne_box.urdf.xacro (robot description, xacro)
@@ -57,5 +57,5 @@
   </xacro:sensor_hokuyo>
   <xacro:sensor_hokuyo name="mirror_lidar" parent="base_link" size="0.05 0.05 0.05">
-    <origin xyz="-0.08 0.0 0.7" rpy="${-PI} 0.175 0"/>
+    <origin xyz="0.43 0.0 0.34" rpy="0 0.314 0"/>
   </xacro:sensor_hokuyo>
 </robot>

Commit message: temp

File: orne_box_description/urdf/orne_box.urdf.xacro (robot description, xacro)
@@ -1,54 +1,207 @@
-<?xml version="1.0"?>
-<robot xmlns:xacro="http://www.ros.org/wiki/xacro" name="orne_box">
+<?xml version="1.0" ?>
+<robot name="orne_box" xmlns:xacro="http://www.ros.org/wiki/xacro">
   <xacro:property name="PI" value="3.1415926535897931"/>
-  <xacro:include filename="$(find orne_box_description)/urdf/material_colors.xacro"/>
+  <xacro:include filename="$(find icart_mini_description)/urdf/materials.xacro" />
   <xacro:include filename="$(find orne_box_description)/urdf/orne_box.gazebo.xacro"/>
-  <xacro:include filename="$(find orne_box_description)/urdf/links/base_link.urdf.xacro"/>
-  <xacro:include filename="$(find orne_box_description)/urdf/links/caster_wheel_link.urdf.xacro"/>
-  <xacro:include filename="$(find orne_box_description)/urdf/links/caster_swivel_link.urdf.xacro"/>
-  <xacro:include filename="$(find orne_box_description)/urdf/links/wheel_link.urdf.xacro"/>
-  <xacro:include filename="$(find orne_box_description)/urdf/joints/caster_wheel_joint.urdf.xacro"/>
-  <xacro:include filename="$(find orne_box_description)/urdf/joints/caster_swivel_joint.urdf.xacro"/>
-  <xacro:include filename="$(find orne_box_description)/urdf/joints/wheel_joint.urdf.xacro"/>
-  <xacro:include filename="$(find orne_box_description)/urdf/sensors/imu.urdf.xacro"/>
-  <xacro:include filename="$(find orne_box_description)/urdf/sensors/hokuyo.urdf.xacro"/>
-  <!-- Setting for base -->
-  <xacro:base_link/>
-  <!-- Setting for caster -->
-  <xacro:caster_wheel_link prefix="left"/>
-  <xacro:caster_swivel_link prefix="left"/>
-  <xacro:caster_wheel_joint prefix="left"/>
-  <xacro:caster_swivel_joint prefix="left" parent="base_link">
-    <origin xyz="0.362 0.150 0.115" rpy="0 0 0"/>
-  </xacro:caster_swivel_joint>
-  <xacro:caster_wheel_link prefix="right"/>
-  <xacro:caster_swivel_link prefix="right"/>
-  <xacro:caster_wheel_joint prefix="right"/>
-  <xacro:caster_swivel_joint prefix="right" parent="base_link">
-    <origin xyz="0.362 -0.150 0.115" rpy="0 0 0"/>
-  </xacro:caster_swivel_joint>
-  <!-- Setting for left wheel -->
-  <xacro:wheel_joint prefix="left" parent="base_link">
+  <link name="base_link">
+<!--
+    <visual>
+      <origin xyz="0 0 -0.154" rpy="0 0 0"/>
+      <geometry>
+        <mesh filename="package://orne_box_description/meshes/bases/orne_box_base.stl" scale="1 1 1"/>
+      </geometry>
+      <material name="orange"/>
+    </visual>
+-->
+    <visual>
+      <origin xyz="0.090 0 0.1715" rpy="0 0 0"/>
+      <geometry>
+        <box size="0.400 0.404 0.202"/>
+      </geometry>
+      <material name="orange"/>
+    </visual>
+    <visual>
+      <origin xyz="0.36125 0 0.2625" rpy="0 0 0"/>
+      <geometry>
+        <box size="0.1425 0.404 0.020"/>
+      </geometry>
+      <material name="orange"/>
+    </visual>
+    <visual>
+      <origin xyz="0.35625 0 0.156" rpy="0 0 0"/>
+      <geometry>
+        <box size="0.1325 0.404 0.020"/>
+      </geometry>
+      <material name="orange"/>
+    </visual>
+    <visual>
+      <origin xyz="-0.120 0 0.4815" rpy="0 0 0"/>
+      <geometry>
+        <box size="0.020 0.404 0.822"/>
+      </geometry>
+      <material name="orange"/>
+    </visual>
+    <collision>
+      <origin xyz="0.090 0 0.1715" rpy="0 0 0"/>
+      <geometry>
+        <box size="0.400 0.404 0.202"/>
+      </geometry>
+    </collision>
+    <collision>
+      <origin xyz="0.36125 0 0.2625" rpy="0 0 0"/>
+      <geometry>
+        <box size="0.1425 0.404 0.020"/>
+      </geometry>
+    </collision>
+    <collision>
+      <origin xyz="0.35625 0 0.156" rpy="0 0 0"/>
+      <geometry>
+        <box size="0.1325 0.404 0.020"/>
+      </geometry>
+    </collision>
+    <collision>
+      <origin xyz="-0.120 0 0.4815" rpy="0 0 0"/>
+      <geometry>
+        <box size="0.020 0.404 0.822"/>
+      </geometry>
+    </collision>
+    <inertial>
+      <origin xyz="0.090 0 0.1715" rpy="0 0 0"/>
+      <mass value="25.0"/>
+      <inertia ixx="1.0" ixy="0.0" ixz="0.0" iyy="1.0" iyz="0.0" izz="1.0" />
+    </inertial>
+  </link>
+  <joint name="left_wheel_hinge" type="revolute">
+    <parent link="base_link"/>
+    <child link="wheel_left_link"/>
     <origin xyz="0.0 0.23075 0.152" rpy="${-PI/2} 0 0"/>
     <axis xyz="0 0 1"/>
-  </xacro:wheel_joint>
-  <xacro:wheel_link prefix="left" width="0.045" radius="0.152">
-    <origin xyz="0.0 0.0 0.0" rpy="0 0 0"/>
-  </xacro:wheel_link>
-  <!-- Setting for right wheel -->
-  <xacro:wheel_joint prefix="right" parent="base_link">
+    <limit effort="100" velocity="100.0"  lower="-5000" upper="5000" />
+  </joint>
+  <link name="wheel_left_link">
+    <visual>
+      <origin xyz="0 0 0" rpy="0 0 0"/>
+      <geometry>
+        <mesh filename="package://orne_box_description/meshes/wheels/tire.stl" scale="1 1 1"/>
+      </geometry>
+<!--
+      <origin xyz="0 0 0" rpy="0 0 0"/>
+      <geometry>
+        <cylinder length="0.045" radius="0.152"/>
+      </geometry>
+-->
+      <material name="white"/>
+    </visual>
+    <collision>
+      <origin xyz="0 0 0" rpy="0 0 0"/>
+      <geometry>
+        <cylinder length="0.045" radius="0.152"/>
+      </geometry>
+    </collision>
+    <inertial>
+      <origin xyz="0 0 0" />
+      <mass value="0.2" />
+      <inertia ixx="0.1" ixy="0.0" ixz="0.0" iyy="0.1" iyz="0.0" izz="0.1" />
+    </inertial>
+  </link>
+  <joint name="right_wheel_hinge" type="revolute">
+    <parent link="base_link"/>
+    <child link="wheel_right_link"/>
     <origin xyz="0.0 -0.23075 0.152" rpy="${-PI/2} 0 0"/>
     <axis xyz="0 0 1"/>
-  </xacro:wheel_joint>
-  <xacro:wheel_link prefix="right" width="0.045" radius="0.152">
-    <origin xyz="0.0 0.0 0.0" rpy="0 0 0"/>
-  </xacro:wheel_link>
-  <!-- Setting for IMU -->
+    <limit effort="100" velocity="100.0"  lower="-5000" upper="5000" />
+  </joint>
+  <link name="wheel_right_link">
+    <visual>
+      <origin xyz="0 0 0" rpy="0 0 0"/>
+      <geometry>
+        <mesh filename="package://orne_box_description/meshes/wheels/tire.stl" scale="1 1 1"/>
+      </geometry>
+<!--
+      <origin xyz="0 0 0" rpy="0 0 0"/>
+      <geometry>
+        <cylinder length="0.045" radius="0.152"/>
+      </geometry>
+-->
+      <material name="white"/>
+    </visual>
+    <collision>
+      <origin xyz="0 0 0" rpy="0 0 0"/>
+      <geometry>
+        <cylinder length="0.045" radius="0.152"/>
+      </geometry>
+    </collision>
+    <inertial>
+      <origin xyz="0 0 0" />
+      <mass value="0.2" />
+      <inertia ixx="0.1" ixy="0.0" ixz="0.0" iyy="0.1" iyz="0.0" izz="0.1" />
+    </inertial>
+  </link>
+  <joint name="caster_front_joint" type="fixed">
+    <parent link="base_link"/>
+    <child link="caster_front_link"/>
+    <origin xyz="0.362 0 0.050" rpy="0 0 0"/>
+  </joint>
+  <link name="caster_front_link">
+    <visual>
+      <origin xyz="0 0.150 0" rpy="${PI/2} 0 0"/>
+      <geometry>
+        <cylinder length="0.025" radius="0.050"/>
+      </geometry>
+      <material name="red"/>
+    </visual>
+    <visual>
+      <origin xyz="0 -0.150 0" rpy="${PI/2} 0 0"/>
+      <geometry>
+        <cylinder length="0.025" radius="0.050"/>
+      </geometry>
+      <material name="red"/>
+    </visual>
+    <collision>
+      <origin xyz="0 0.150 0" rpy="${PI/2} 0 0"/>
+      <geometry>
+        <cylinder length="0.025" radius="0.050"/>
+      </geometry>
+    </collision>
+    <collision>
+      <origin xyz="0 -0.150 0" rpy="${PI/2} 0 0"/>
+      <geometry>
+        <cylinder length="0.025" radius="0.050"/>
+      </geometry>
+    </collision>
+    <inertial>
+      <origin xyz="0 0 0" />
+      <mass value="0.2" />
+      <inertia ixx="0.1" ixy="0.0" ixz="0.0" iyy="0.1" iyz="0.0" izz="0.1" />
+    </inertial>
+  </link>
+  <xacro:include filename="$(find icart_mini_description)/urdf/sensors/imu.urdf.xacro"/>
+  <!-- Setting for imu -->
   <xacro:sensor_imu name="imu" parent="base_link" size="0.05 0.05 0.05">
-    <origin xyz="0.23 0.0 0.270" rpy="${-PI} 0 ${PI/2}"/>
+    <origin xyz="0.3 0 0.2445" rpy="0 0 ${-PI/2}"/>
   </xacro:sensor_imu>
-  <!-- Setting for 2D-LiDAR -->
-  <xacro:sensor_hokuyo name="hokuyo" parent="base_link" size="0.05 0.05 0.05">
+  <xacro:include filename="$(find icart_mini_description)/urdf/sensors/hokuyo.urdf.xacro"/>
+  <xacro:sensor_hokuyo name="hokuyo" parent="base_link">
     <origin xyz="0.374295 0 0.2185" rpy="${-PI} 0 0"/>
   </xacro:sensor_hokuyo>
+  <transmission name="tran1">
+    <type>transmission_interface/SimpleTransmission</type>
+    <joint name="left_wheel_hinge">
+      <hardwareInterface>VelocityJointInterface</hardwareInterface>
+    </joint>
+  <actuator name="left_motor">
+      <hardwareInterface>VelocityJointInterface</hardwareInterface>
+      <mechanicalReduction>1</mechanicalReduction>
+    </actuator>
+  </transmission>
+  <transmission name="tran2">
+    <type>transmission_interface/SimpleTransmission</type>
+    <joint name="right_wheel_hinge">
+      <hardwareInterface>VelocityJointInterface</hardwareInterface>
+    </joint>
+  <actuator name="right_motor">
+      <hardwareInterface>VelocityJointInterface</hardwareInterface>
+      <mechanicalReduction>1</mechanicalReduction>
+    </actuator>
+  </transmission>
 </robot>

Commit message: fix for box

File: orne_box_description/urdf/orne_box.urdf.xacro (robot description, xacro)
@@ -11,5 +11,5 @@
   <xacro:include filename="$(find orne_box_description)/urdf/joints/caster_swivel_joint.urdf.xacro"/>
   <xacro:include filename="$(find orne_box_description)/urdf/joints/wheel_joint.urdf.xacro"/>
-  <xacro:include filename="$(find orne_box_description)/urdf/sensors/imu.urdf.xacro"/>
+  <!-- <xacro:include filename="$(find orne_box_description)/urdf/sensors/imu.urdf.xacro"/> -->
   <xacro:include filename="$(find orne_box_description)/urdf/sensors/hokuyo.urdf.xacro"/>
   <!-- Setting for base -->
@@ -45,13 +45,13 @@
   </xacro:wheel_link>
   <!-- Setting for IMU -->
-  <xacro:sensor_imu name="imu" parent="base_link" size="0.05 0.05 0.05">
+  <!-- <xacro:sensor_imu name="imu" parent="base_link" size="0.05 0.05 0.05">
     <origin xyz="0.23 0.0 0.270" rpy="${-PI} 0 ${PI/2}"/>
-  </xacro:sensor_imu>
+  </xacro:sensor_imu> -->
   <!-- Setting for 2D-LiDAR -->
+  <!-- <xacro:sensor_hokuyo name="hokuyo" parent="base_link" size="0.05 0.05 0.05">
+    <origin xyz="0.23 0 0.35" rpy="0 0 0"/> -->
+    <!--origin xyz="0.23 0 0.4" rpy="0 0 0"/-->
+  <!-- </xacro:sensor_hokuyo> -->
   <xacro:sensor_hokuyo name="hokuyo" parent="base_link" size="0.05 0.05 0.05">
-    <origin xyz="0.23 0 0.35" rpy="0 0 0"/>
-    <!--origin xyz="0.23 0 0.4" rpy="0 0 0"/-->
-  </xacro:sensor_hokuyo>
-  <xacro:sensor_hokuyo name="low_hokuyo" parent="base_link" size="0.05 0.05 0.05">
     <origin xyz="0.374295 0 0.2185" rpy="${-PI} 0 0"/>
   </xacro:sensor_hokuyo>

Commit message: 動作確認

File: orne_box_description/urdf/orne_box.urdf.xacro (robot description, xacro)
@@ -54,5 +54,5 @@
   <!-- </xacro:sensor_hokuyo> -->
   <xacro:sensor_hokuyo name="hokuyo" parent="base_link" size="0.05 0.05 0.05">
-    <origin xyz="0.374295 0 0.2185" rpy="${-PI} 0 0"/>
+    <origin xyz="0.374295 0 0.2185" rpy="0 0 0"/>
   </xacro:sensor_hokuyo>
 </robot>
