Commit message: add mid360 TF

File: orne_box_description/urdf/orne_box.urdf.xacro (robot description, xacro)
@@ -12,4 +12,5 @@
   <xacro:include filename="$(find orne_box_description)/urdf/joints/wheel_joint.urdf.xacro"/>
   <xacro:include filename="$(find orne_box_description)/urdf/sensors/imu.urdf.xacro"/>
+  <xacro:include filename="$(find orne_box_description)/urdf/sensors/mid360.urdf.xacro"/>
        <!--<xacro:include filename="$(find orne_box_description)/urdf/sensors/hokuyo.urdf.xacro"/>-->
   <!-- Setting for base -->
@@ -52,4 +53,7 @@
     <origin_child xyz="0.0 0.0 0.0" rpy="0 0 0"/>
   </xacro:sensor_imu>
+  <xacro:sensor_mid360 name="livox_frame" parent="base_link">
+    <origin xyz="0.424 0.0 0.343" rpy="0 0 0"/>
+  </xacro:sensor_mid360>
   <!-- Setting for 2D-LiDAR -->
   <!--<xacro:sensor_hokuyo name="hokuyo" parent="base_link" size="0.05 0.05 0.05">

Commit message: change upside down MID360

File: orne_box_description/urdf/orne_box.urdf.xacro (robot description, xacro)
@@ -54,5 +54,5 @@
   </xacro:sensor_imu>
   <xacro:sensor_mid360 name="livox_frame" parent="base_link">
-    <origin xyz="0.424 0.0 0.343" rpy="0 0 0"/>
+    <origin xyz="0.424 0.0 0.203" rpy="0 3.14159 0"/>
   </xacro:sensor_mid360>
   <!-- Setting for 2D-LiDAR -->

Commit message: change urdf

File: orne_box_description/urdf/orne_box.urdf.xacro (robot description, xacro)
@@ -54,5 +54,5 @@
   </xacro:sensor_imu>
   <xacro:sensor_mid360 name="livox_frame" parent="base_link">
-    <origin xyz="0.424 0.0 0.203" rpy="0 3.14159 0"/>
+	  <origin xyz="0.424 0.0 0.203" rpy="0 3.14159 ${PI/2}"/>
   </xacro:sensor_mid360>
   <!-- Setting for 2D-LiDAR -->

Commit message: diff orne_box.urdf.xacro and mid360.urdf.xacro

File: orne_box_description/urdf/orne_box.urdf.xacro (robot description, xacro)
@@ -12,4 +12,5 @@
   <xacro:include filename="$(find orne_box_description)/urdf/joints/wheel_joint.urdf.xacro"/>
   <xacro:include filename="$(find orne_box_description)/urdf/sensors/imu.urdf.xacro"/>
+  <xacro:include filename="$(find orne_box_description)/urdf/sensors/mid360.urdf.xacro"/>
        <!--<xacro:include filename="$(find orne_box_description)/urdf/sensors/hokuyo.urdf.xacro"/>-->
   <!-- Setting for base -->
@@ -52,4 +53,7 @@
     <origin_child xyz="0.0 0.0 0.0" rpy="0 0 0"/>
   </xacro:sensor_imu>
+  <xacro:sensor_mid360 name="livox_frame" parent="base_link">
+	  <origin xyz="0.424 0.0 0.203" rpy="0 3.14159 ${PI/2}"/>
+  </xacro:sensor_mid360>
   <!-- Setting for 2D-LiDAR -->
   <!--<xacro:sensor_hokuyo name="hokuyo" parent="base_link" size="0.05 0.05 0.05">
