Commit message: execute on gazebo

File: orne_box_description/urdf/orne_box.gazebo.xacro (robot description, xacro)
@@ -7,6 +7,6 @@
   </gazebo>
   <gazebo reference="wheel_left_link">
-    <mu1>0.1</mu1>
-    <mu2>0.1</mu2>
+    <mu1>1.0</mu1>
+    <mu2>1.0</mu2>
     <kp>500000.0</kp>
     <kd>10.0</kd>
@@ -17,6 +17,6 @@
   </gazebo>
   <gazebo reference="wheel_right_link">
-    <mu1>0.1</mu1>
-    <mu2>0.1</mu2>
+    <mu1>1.0</mu1>
+    <mu2>1.0</mu2>
     <kp>500000.0</kp>
     <kd>10.0</kd>
@@ -27,6 +27,6 @@
   </gazebo>
   <gazebo reference="caster_front_link">
-    <mu1>0.1</mu1>
-    <mu2>0.1</mu2>
+    <mu1>0.01</mu1>
+    <mu2>0.01</mu2>
     <kp>1000000.0</kp>
     <kd>100.0</kd>

File: orne_box_description/urdf/orne_box.urdf.xacro (robot description, xacro)
@@ -3,22 +3,17 @@
   <xacro:include filename="$(find orne_box_description)/urdf/common_properties.xacro"/>
   <xacro:include filename="$(find orne_box_description)/urdf/orne_box.gazebo.xacro"/>
-  <link name="base_footprint"/>
-  <joint name="base_joint" type="fixed">
-    <parent link="base_footprint"/>
-    <child link="base_link"/>
-    <origin xyz="0.0 0.0 0.152" rpy="0 0 0"/>
-  </joint>
   <link name="base_link">
     <visual>
-      <origin xyz="0.0 0 -0.152" rpy="0 0 0"/>
+      <origin xyz="0 0 -0.154" rpy="0 0 0"/>
       <geometry>
         <mesh filename="package://orne_box_description/meshes/bases/orne_box_base.stl" scale="1 1 1"/>
+        <box size="0.540 0.404 0.202"/>
       </geometry>
       <material name="light_black"/>
     </visual>
     <collision>
-      <origin xyz="0.158 0 0" rpy="0 0 0"/>
+      <origin xyz="0.160 0 0.0195" rpy="0 0 0"/>
       <geometry>
-        <box size="0.540 0.40 0.02"/>
+        <box size="0.540 0.404 0.202"/>
       </geometry>
     </collision>
@@ -48,5 +43,5 @@
       <origin xyz="0 0 0" rpy="0 0 0"/>
       <geometry>
-        <cylinder length="0.0225" radius="0.152"/>
+        <cylinder length="0.045" radius="0.152"/>
       </geometry>
     </collision>
@@ -76,5 +71,5 @@
       <origin xyz="0 0 0" rpy="0 0 0"/>
       <geometry>
-        <cylinder length="0.0225" radius="0.152"/>
+        <cylinder length="0.045" radius="0.152"/>
       </geometry>
     </collision>
@@ -90,11 +85,17 @@
     <parent link="base_link"/>
     <child link="caster_front_link"/>
-    <origin xyz="0.374295 0 0.015" rpy="-3.14 0 0"/>
+    <origin xyz="0.362 0 -0.102" rpy="0 0 0"/>
   </joint>
   <link name="caster_front_link">
     <collision>
-      <origin xyz="0 0.0 0.0835" rpy="0 0 0"/>
+      <origin xyz="0 0.150 0" rpy="1.57 0 0"/>
       <geometry>
-        <box size="0.10 0.4 0.167"/>
+        <cylinder length="0.025" radius="0.050"/>
+      </geometry>
+    </collision>
+    <collision>
+      <origin xyz="0 -0.150 0" rpy="1.57 0 0"/>
+      <geometry>
+        <cylinder length="0.025" radius="0.050"/>
       </geometry>
     </collision>
@@ -110,13 +111,13 @@
     <parent link="base_link"/>
     <child link="imu_link"/>
-    <origin xyz="0 0 0" rpy="0 0 0"/>
+    <origin xyz="0.3 0 0.1225" rpy="0 0 -1.57"/>
   </joint>
   <link name="imu_link"/>
   <joint name="scan_joint" type="fixed">
     <parent link="base_link"/>
-    <child link="base_scan"/>
+    <child link="hokuyo_link"/>
     <origin xyz="0.374295 0 0.1225" rpy="-3.14 0 0"/>
   </joint>
-  <link name="base_scan">
+  <link name="hokuyo_link">
     <inertial>
       <mass value="0.08" />

Commit message: change inertia

File: orne_box_description/urdf/orne_box.gazebo.xacro (robot description, xacro)
@@ -3,6 +3,11 @@
   <xacro:arg name="laser_visual" default="false"/>
   <xacro:arg name="imu_visual"   default="false"/>
+  <gazebo>
+    <plugin name="gazebo_ros_control" filename="libgazebo_ros_control.so">
+      <robotSimType>icart_mini_gazebo/ICartMiniHWSim</robotSimType>
+    </plugin>
+  </gazebo>
   <gazebo reference="base_link">
-    <material>Gazebo/DarkGrey</material>
+    <material>Gazebo/Orange</material>
   </gazebo>
   <gazebo reference="wheel_left_link">
@@ -14,5 +19,5 @@
     <maxVel>1.0</maxVel>
     <fdir1>1 0 0</fdir1>
-    <material>Gazebo/FlatBlack</material>
+    <material>Gazebo/White</material>
   </gazebo>
   <gazebo reference="wheel_right_link">
@@ -24,5 +29,5 @@
     <maxVel>1.0</maxVel>
     <fdir1>1 0 0</fdir1>
-    <material>Gazebo/FlatBlack</material>
+    <material>Gazebo/White</material>
   </gazebo>
   <gazebo reference="caster_front_link">
@@ -33,5 +38,5 @@
     <minDepth>0.001</minDepth>
     <maxVel>1.0</maxVel>
-    <material>Gazebo/FlatBlack</material>
+    <material>Gazebo/Red</material>
   </gazebo>
   <gazebo reference="imu_link">
@@ -42,4 +47,5 @@
     <material>Gazebo/FlatBlack</material>
   </gazebo>
+<!--
   <gazebo>
     <plugin name="orne_box_controller" filename="libgazebo_ros_diff_drive.so">
@@ -64,4 +70,5 @@
     </plugin>
   </gazebo>
+-->
   <gazebo>
     <plugin name="imu_plugin" filename="libgazebo_ros_imu.so">

File: orne_box_description/urdf/orne_box.urdf.xacro (robot description, xacro)
@@ -1,8 +1,9 @@
 <?xml version="1.0" ?>
-<robot name="orne_box" xmlns:xacro="http://ros.org/wiki/xacro">
-  <xacro:include filename="$(find orne_box_description)/urdf/common_properties.xacro"/>
+<robot name="orne_box" xmlns:xacro="http://www.ros.org/wiki/xacro">
+  <xacro:include filename="$(find icart_mini_description)/urdf/materials.xacro" />
   <xacro:include filename="$(find orne_box_description)/urdf/orne_box.gazebo.xacro"/>
   <link name="base_link">
     <visual>
+<!--
       <origin xyz="0 0 -0.154" rpy="0 0 0"/>
       <geometry>
@@ -10,10 +11,54 @@
         <box size="0.540 0.404 0.202"/>
       </geometry>
-      <material name="light_black"/>
-    </visual>
-    <collision>
-      <origin xyz="0.160 0 0.0195" rpy="0 0 0"/>
-      <geometry>
-        <box size="0.540 0.404 0.202"/>
+-->
+      <origin xyz="0.090 0 0.0195" rpy="0 0 0"/>
+      <geometry>
+        <box size="0.400 0.404 0.202"/>
+      </geometry>
+      <material name="orange"/>
+    </visual>
+    <visual>
+      <origin xyz="0.36125 0 0.1105" rpy="0 0 0"/>
+      <geometry>
+        <box size="0.1425 0.404 0.020"/>
+      </geometry>
+      <material name="orange"/>
+    </visual>
+    <visual>
+      <origin xyz="0.35625 0 0.004" rpy="0 0 0"/>
+      <geometry>
+        <box size="0.1325 0.404 0.020"/>
+      </geometry>
+      <material name="orange"/>
+    </visual>
+    <visual>
+      <origin xyz="-0.120 0 0.3295" rpy="0 0 0"/>
+      <geometry>
+        <box size="0.020 0.404 0.822"/>
+      </geometry>
+      <material name="orange"/>
+    </visual>
+    <collision>
+      <origin xyz="0.090 0 0.0195" rpy="0 0 0"/>
+      <geometry>
+        <box size="0.400 0.404 0.202"/>
+      </geometry>
+    </collision>
+    <collision>
+      <origin xyz="0.36125 0 0.1105" rpy="0 0 0"/>
+      <geometry>
+        <box size="0.1425 0.404 0.020"/>
+      </geometry>
+    </collision>
+    <collision>
+      <origin xyz="0.35625 0 0.004" rpy="0 0 0"/>
+      <geometry>
+        <box size="0.1325 0.404 0.020"/>
+      </geometry>
+    </collision>
+    <collision>
+      <origin xyz="-0.120 0 0.3295" rpy="0 0 0"/>
+      <geometry>
+        <box size="0.020 0.404 0.822"/>
       </geometry>
     </collision>
@@ -21,22 +66,27 @@
       <origin xyz="0 0.07 -0.05" rpy="0 0 0"/>
       <mass value="25.0"/>
-      <inertia ixx="0.1" ixy="0.0" ixz="0.0"
-               iyy="0.1" iyz="0.0"
-               izz="0.1" />
-    </inertial>
-  </link>
-  <joint name="wheel_left_joint" type="continuous">
+      <inertia ixx="1.0" ixy="0.0" ixz="0.0" iyy="1.0" iyz="0.0" izz="1.0" />
+    </inertial>
+  </link>
+  <joint name="left_wheel_hinge" type="revolute">
     <parent link="base_link"/>
     <child link="wheel_left_link"/>
     <origin xyz="0.0 0.23075 0.0" rpy="-1.57 0 0"/>
     <axis xyz="0 0 1"/>
+    <limit effort="100" velocity="100.0"  lower="-5000" upper="5000" />
   </joint>
   <link name="wheel_left_link">
     <visual>
+<!--
       <origin xyz="0 0 0" rpy="0 0 0"/>
       <geometry>
         <mesh filename="package://orne_box_description/meshes/wheels/tire.stl" scale="1 1 1"/>
       </geometry>
-      <material name="dark"/>
+-->
+      <origin xyz="0 0 0" rpy="0 0 0"/>
+      <geometry>
+        <cylinder length="0.045" radius="0.152"/>
+      </geometry>
+      <material name="white"/>
     </visual>
     <collision>
@@ -49,36 +99,49 @@
       <origin xyz="0 0 0" />
       <mass value="0.2" />
+      <inertia ixx="0.1" ixy="0.0" ixz="0.0" iyy="0.1" iyz="0.0" izz="0.1" />
+<!--
       <inertia ixx="1.1175580e-05" ixy="-4.2369783e-11" ixz="-5.9381719e-09"
                iyy="1.1192413e-05" iyz="-1.4400107e-11"
                izz="2.0712558e-05" />
-    </inertial>
-  </link>
-  <joint name="wheel_right_joint" type="continuous">
+-->
+    </inertial>
+  </link>
+  <joint name="right_wheel_hinge" type="revolute">
     <parent link="base_link"/>
     <child link="wheel_right_link"/>
     <origin xyz="0.0 -0.23075 0.0" rpy="-1.57 0 0"/>
     <axis xyz="0 0 1"/>
+    <limit effort="100" velocity="100.0"  lower="-5000" upper="5000" />
   </joint>
   <link name="wheel_right_link">
     <visual>
+<!--
       <origin xyz="0 0 0" rpy="0 0 0"/>
       <geometry>
         <mesh filename="package://orne_box_description/meshes/wheels/tire.stl" scale="1 1 1"/>
       </geometry>
-      <material name="dark"/>
-    </visual>
-    <collision>
-      <origin xyz="0 0 0" rpy="0 0 0"/>
-      <geometry>
-        <cylinder length="0.045" radius="0.152"/>
-      </geometry>
-    </collision>
-      <inertial>
-        <origin xyz="0 0 0" />
-        <mass value="0.2" />
-        <inertia ixx="1.1175580e-05" ixy="-4.2369783e-11" ixz="-5.9381719e-09"
-               iyy="1.1192413e-05" iyz="-1.4400107e-11"
-               izz="2.0712558e-05" />
-      </inertial>
+-->
+      <origin xyz="0 0 0" rpy="0 0 0"/>
+      <geometry>
+        <cylinder length="0.045" radius="0.152"/>
+      </geometry>
+      <material name="white"/>
+    </visual>
+    <collision>
+      <origin xyz="0 0 0" rpy="0 0 0"/>
+      <geometry>
+        <cylinder length="0.045" radius="0.152"/>
+      </geometry>
+    </collision>
+    <inertial>
+      <origin xyz="0 0 0" />
+      <mass value="0.2" />
+      <inertia ixx="0.1" ixy="0.0" ixz="0.0" iyy="0.1" iyz="0.0" izz="0.1" />
+<!--
+      <inertia ixx="1.1175580e-05" ixy="-4.2369783e-11" ixz="-5.9381719e-09"
+             iyy="1.1192413e-05" iyz="-1.4400107e-11"
+             izz="2.0712558e-05" />
+-->
+    </inertial>
   </link>
   <joint name="caster_front_joint" type="fixed">
@@ -88,22 +151,34 @@
   </joint>
   <link name="caster_front_link">
-    <collision>
+    <visual>
       <origin xyz="0 0.150 0" rpy="1.57 0 0"/>
       <geometry>
         <cylinder length="0.025" radius="0.050"/>
       </geometry>
-    </collision>
-    <collision>
+      <material name="red"/>
+    </visual>
+    <visual>
       <origin xyz="0 -0.150 0" rpy="1.57 0 0"/>
       <geometry>
         <cylinder length="0.025" radius="0.050"/>
       </geometry>
+      <material name="red"/>
+    </visual>
+    <collision>
+      <origin xyz="0 0.150 0" rpy="1.57 0 0"/>
+      <geometry>
+        <cylinder length="0.025" radius="0.050"/>
+      </geometry>
+    </collision>
+    <collision>
+      <origin xyz="0 -0.150 0" rpy="1.57 0 0"/>
+      <geometry>
+        <cylinder length="0.025" radius="0.050"/>
+      </geometry>
     </collision>
     <inertial>
       <origin xyz="0 0 0" />
       <mass value="0.2" />
-      <inertia ixx="0.001" ixy="0.0" ixz="0.0"
-               iyy="0.001" iyz="0.0"
-               izz="0.001" />
+      <inertia ixx="0.1" ixy="0.0" ixz="0.0" iyy="0.1" iyz="0.0" izz="0.1" />
     </inertial>
   </link>
@@ -123,8 +198,26 @@
       <mass value="0.08" />
       <origin xyz="0 0 0" />
-      <inertia ixx="0.001" ixy="0.0" ixz="0.0"
-               iyy="0.001" iyz="0.0"
-               izz="0.001" />
-    </inertial>
-  </link>
+      <inertia ixx="0.1" ixy="0.0" ixz="0.0" iyy="0.1" iyz="0.0" izz="0.1" />
+    </inertial>
+  </link>
+  <transmission name="tran1">
+    <type>transmission_interface/SimpleTransmission</type>
+    <joint name="left_wheel_hinge">
+      <hardwareInterface>VelocityJointInterface</hardwareInterface>
+    </joint>
+  <actuator name="left_motor">
+      <hardwareInterface>VelocityJointInterface</hardwareInterface>
+      <mechanicalReduction>1</mechanicalReduction>
+    </actuator>
+  </transmission>
+  <transmission name="tran2">
+    <type>transmission_interface/SimpleTransmission</type>
+    <joint name="right_wheel_hinge">
+      <hardwareInterface>VelocityJointInterface</hardwareInterface>
+    </joint>
+  <actuator name="right_motor">
+      <hardwareInterface>VelocityJointInterface</hardwareInterface>
+      <mechanicalReduction>1</mechanicalReduction>
+    </actuator>
+  </transmission>
 </robot>

Commit message: add LiDAR

File: orne_box_description/urdf/orne_box.gazebo.xacro (robot description, xacro)
@@ -1,5 +1,5 @@
 <?xml version="1.0"?>
 <robot name="orne_box" xmlns:xacro="http://ros.org/wiki/xacro">
-  <xacro:arg name="laser_visual" default="false"/>
+  <xacro:arg name="laser_visual" default="true"/>
   <xacro:arg name="imu_visual"   default="false"/>
   <gazebo>
@@ -14,9 +14,8 @@
     <mu1>1.0</mu1>
     <mu2>1.0</mu2>
-    <kp>500000.0</kp>
-    <kd>10.0</kd>
+    <kp>1000000.0</kp>
+    <kd>100.0</kd>
     <minDepth>0.001</minDepth>
     <maxVel>1.0</maxVel>
-    <fdir1>1 0 0</fdir1>
     <material>Gazebo/White</material>
   </gazebo>
@@ -24,18 +23,13 @@
     <mu1>1.0</mu1>
     <mu2>1.0</mu2>
-    <kp>500000.0</kp>
-    <kd>10.0</kd>
-    <minDepth>0.001</minDepth>
-    <maxVel>1.0</maxVel>
-    <fdir1>1 0 0</fdir1>
-    <material>Gazebo/White</material>
-  </gazebo>
-  <gazebo reference="caster_front_link">
-    <mu1>0.01</mu1>
-    <mu2>0.01</mu2>
     <kp>1000000.0</kp>
     <kd>100.0</kd>
     <minDepth>0.001</minDepth>
     <maxVel>1.0</maxVel>
+    <material>Gazebo/White</material>
+  </gazebo>
+  <gazebo reference="caster_front_link">
+    <mu1>0.0</mu1>
+    <mu2>0.0</mu2>
     <material>Gazebo/Red</material>
   </gazebo>
@@ -47,63 +41,10 @@
     <material>Gazebo/FlatBlack</material>
   </gazebo>
-<!--
-  <gazebo>
-    <plugin name="orne_box_controller" filename="libgazebo_ros_diff_drive.so">
-      <commandTopic>cmd_vel</commandTopic>
-      <odometryTopic>odom</odometryTopic>
-      <odometryFrame>odom</odometryFrame>
-      <odometrySource>world</odometrySource>
-      <publishOdomTF>true</publishOdomTF>
-      <robotBaseFrame>base_footprint</robotBaseFrame>
-      <publishWheelTF>false</publishWheelTF>
-      <publishTf>true</publishTf>
-      <publishWheelJointState>true</publishWheelJointState>
-      <legacyMode>false</legacyMode>
-      <updateRate>30</updateRate>
-      <leftJoint>wheel_left_joint</leftJoint>
-      <rightJoint>wheel_right_joint</rightJoint>
-      <wheelSeparation>0.4615</wheelSeparation>
-      <wheelDiameter>0.304</wheelDiameter>
-      <wheelAcceleration>1</wheelAcceleration>
-      <wheelTorque>10</wheelTorque>
-      <rosDebugLevel>na</rosDebugLevel>
-    </plugin>
-  </gazebo>
--->
-  <gazebo>
-    <plugin name="imu_plugin" filename="libgazebo_ros_imu.so">
-      <alwaysOn>true</alwaysOn>
-      <bodyName>imu_link</bodyName>
-      <frameName>imu_link</frameName>
-      <topicName>imu</topicName>
-      <serviceName>imu_service</serviceName>
-      <gaussianNoise>0.0</gaussianNoise>
-      <updateRate>200</updateRate>
-      <imu>
-        <noise>
-          <type>gaussian</type>
-          <rate>
-            <mean>0.0</mean>
-            <stddev>2e-4</stddev>
-            <bias_mean>0.0000075</bias_mean>
-            <bias_stddev>0.0000008</bias_stddev>
-          </rate>
-          <accel>
-            <mean>0.0</mean>
-            <stddev>1.7e-2</stddev>
-            <bias_mean>0.1</bias_mean>
-            <bias_stddev>0.001</bias_stddev>
-          </accel>
-        </noise>
-      </imu>
-    </plugin>
-  </gazebo>
-  <!--UTM-30-LX specifications-->
-  <gazebo reference="base_scan">
-    <material>Gazebo/FlatBlack</material>
-    <sensor type="ray" name="lds_lfcd_sensor">
+  <!-- hokuyo -->
+  <gazebo reference="hokuyo_link">
+    <sensor type="ray" name="head_hokuyo_sensor">
       <pose>0 0 0 0 0 0</pose>
       <visualize>$(arg laser_visual)</visualize>
-      <update_rate>5</update_rate>
+      <update_rate>40</update_rate>
       <ray>
         <scan>
@@ -116,17 +57,21 @@
         </scan>
         <range>
-          <min>0.1</min>
+          <min>0.10</min>
           <max>30.0</max>
-          <resolution>0.05</resolution>
+          <resolution>0.01</resolution>
         </range>
         <noise>
           <type>gaussian</type>
+          <!-- Noise parameters based on published spec for Hokuyo laser
+               achieving "+-30mm" accuracy at range < 10m.  A mean of 0.0m and
+               stddev of 0.01m will put 99.7% of samples within 0.03m of the true
+               reading. -->
           <mean>0.0</mean>
           <stddev>0.01</stddev>
         </noise>
       </ray>
-      <plugin name="gazebo_ros_lds_lfcd_controller" filename="libgazebo_ros_laser.so">
-        <topicName>scan</topicName>
-        <frameName>base_scan</frameName>
+      <plugin name="gazebo_ros_head_hokuyo_controller" filename="libgazebo_ros_laser.so">
+        <topicName>/scan</topicName>
+        <frameName>hokuyo_link</frameName>
       </plugin>
     </sensor>

File: orne_box_description/urdf/orne_box.urdf.xacro (robot description, xacro)
@@ -1,15 +1,18 @@
 <?xml version="1.0" ?>
 <robot name="orne_box" xmlns:xacro="http://www.ros.org/wiki/xacro">
+  <xacro:property name="PI" value="3.1415926535897931"/>
   <xacro:include filename="$(find icart_mini_description)/urdf/materials.xacro" />
   <xacro:include filename="$(find orne_box_description)/urdf/orne_box.gazebo.xacro"/>
   <link name="base_link">
-    <visual>
 <!--
+    <visual>
       <origin xyz="0 0 -0.154" rpy="0 0 0"/>
       <geometry>
         <mesh filename="package://orne_box_description/meshes/bases/orne_box_base.stl" scale="1 1 1"/>
-        <box size="0.540 0.404 0.202"/>
-      </geometry>
+      </geometry>
+      <material name="orange"/>
+    </visual>
 -->
+    <visual>
       <origin xyz="0.090 0 0.0195" rpy="0 0 0"/>
       <geometry>
@@ -64,5 +67,5 @@
     </collision>
     <inertial>
-      <origin xyz="0 0.07 -0.05" rpy="0 0 0"/>
+      <origin xyz="0.090 0 0.0195" rpy="0 0 0"/>
       <mass value="25.0"/>
       <inertia ixx="1.0" ixy="0.0" ixz="0.0" iyy="1.0" iyz="0.0" izz="1.0" />
@@ -72,5 +75,5 @@
     <parent link="base_link"/>
     <child link="wheel_left_link"/>
-    <origin xyz="0.0 0.23075 0.0" rpy="-1.57 0 0"/>
+    <origin xyz="0.0 0.23075 0.0" rpy="1.57 0 0"/>
     <axis xyz="0 0 1"/>
     <limit effort="100" velocity="100.0"  lower="-5000" upper="5000" />
@@ -78,14 +81,14 @@
   <link name="wheel_left_link">
     <visual>
+      <origin xyz="0 0 0" rpy="0 0 0"/>
+      <geometry>
+        <mesh filename="package://orne_box_description/meshes/wheels/tire.stl" scale="1 1 1"/>
+      </geometry>
 <!--
       <origin xyz="0 0 0" rpy="0 0 0"/>
       <geometry>
-        <mesh filename="package://orne_box_description/meshes/wheels/tire.stl" scale="1 1 1"/>
+        <cylinder length="0.045" radius="0.152"/>
       </geometry>
 -->
-      <origin xyz="0 0 0" rpy="0 0 0"/>
-      <geometry>
-        <cylinder length="0.045" radius="0.152"/>
-      </geometry>
       <material name="white"/>
     </visual>
@@ -100,9 +103,4 @@
       <mass value="0.2" />
       <inertia ixx="0.1" ixy="0.0" ixz="0.0" iyy="0.1" iyz="0.0" izz="0.1" />
-<!--
-      <inertia ixx="1.1175580e-05" ixy="-4.2369783e-11" ixz="-5.9381719e-09"
-               iyy="1.1192413e-05" iyz="-1.4400107e-11"
-               izz="2.0712558e-05" />
--->
     </inertial>
   </link>
@@ -116,14 +114,14 @@
   <link name="wheel_right_link">
     <visual>
+      <origin xyz="0 0 0" rpy="0 0 0"/>
+      <geometry>
+        <mesh filename="package://orne_box_description/meshes/wheels/tire.stl" scale="1 1 1"/>
+      </geometry>
 <!--
       <origin xyz="0 0 0" rpy="0 0 0"/>
       <geometry>
-        <mesh filename="package://orne_box_description/meshes/wheels/tire.stl" scale="1 1 1"/>
+        <cylinder length="0.045" radius="0.152"/>
       </geometry>
 -->
-      <origin xyz="0 0 0" rpy="0 0 0"/>
-      <geometry>
-        <cylinder length="0.045" radius="0.152"/>
-      </geometry>
       <material name="white"/>
     </visual>
@@ -138,9 +136,4 @@
       <mass value="0.2" />
       <inertia ixx="0.1" ixy="0.0" ixz="0.0" iyy="0.1" iyz="0.0" izz="0.1" />
-<!--
-      <inertia ixx="1.1175580e-05" ixy="-4.2369783e-11" ixz="-5.9381719e-09"
-             iyy="1.1192413e-05" iyz="-1.4400107e-11"
-             izz="2.0712558e-05" />
--->
     </inertial>
   </link>
@@ -183,22 +176,13 @@
     </inertial>
   </link>
-  <joint name="imu_joint" type="fixed">
-    <parent link="base_link"/>
-    <child link="imu_link"/>
-    <origin xyz="0.3 0 0.1225" rpy="0 0 -1.57"/>
-  </joint>
-  <link name="imu_link"/>
-  <joint name="scan_joint" type="fixed">
-    <parent link="base_link"/>
-    <child link="hokuyo_link"/>
-    <origin xyz="0.374295 0 0.1225" rpy="-3.14 0 0"/>
-  </joint>
-  <link name="hokuyo_link">
-    <inertial>
-      <mass value="0.08" />
-      <origin xyz="0 0 0" />
-      <inertia ixx="0.1" ixy="0.0" ixz="0.0" iyy="0.1" iyz="0.0" izz="0.1" />
-    </inertial>
-  </link>
+  <xacro:include filename="$(find icart_mini_description)/urdf/sensors/imu.urdf.xacro"/>
+  <!-- Setting for imu -->
+  <xacro:sensor_imu name="imu" parent="base_link" size="0.05 0.05 0.05">
+    <origin xyz="0.3 0 0.0925" rpy="0 0 -1.57"/>
+  </xacro:sensor_imu>
+  <xacro:include filename="$(find icart_mini_description)/urdf/sensors/hokuyo.urdf.xacro"/>
+  <xacro:sensor_hokuyo name="hokuyo" parent="base_link">
+    <origin xyz="0.374295 0 0.0665" rpy="-3.14 0 0"/>
+  </xacro:sensor_hokuyo>
   <transmission name="tran1">
     <type>transmission_interface/SimpleTransmission</type>
