Commit message: use PI

File: orne_box_description/urdf/orne_box.gazebo.xacro (robot description, xacro)
@@ -1,4 +1,5 @@
 <?xml version="1.0"?>
 <robot name="orne_box" xmlns:xacro="http://ros.org/wiki/xacro">
+  <xacro:property name="PI" value="3.1415926535897931"/>
   <xacro:arg name="laser_visual" default="true"/>
   <xacro:arg name="imu_visual"   default="false"/>
@@ -50,8 +51,8 @@
         <scan>
           <horizontal>
-            <samples>720</samples>
+            <samples>880</samples>
             <resolution>0.25</resolution>
-            <min_angle>-1.570796</min_angle>
-            <max_angle>1.570796</max_angle>
+            <min_angle>${-PI/180*110}</min_angle>
+            <max_angle>${ PI/180*110}</max_angle>
           </horizontal>
         </scan>

File: orne_box_description/urdf/orne_box.urdf.xacro (robot description, xacro)
@@ -75,5 +75,5 @@
     <parent link="base_link"/>
     <child link="wheel_left_link"/>
-    <origin xyz="0.0 0.23075 0.0" rpy="1.57 0 0"/>
+    <origin xyz="0.0 0.23075 0.0" rpy="${-PI/2} 0 0"/>
     <axis xyz="0 0 1"/>
     <limit effort="100" velocity="100.0"  lower="-5000" upper="5000" />
@@ -108,5 +108,5 @@
     <parent link="base_link"/>
     <child link="wheel_right_link"/>
-    <origin xyz="0.0 -0.23075 0.0" rpy="-1.57 0 0"/>
+    <origin xyz="0.0 -0.23075 0.0" rpy="${-PI/2} 0 0"/>
     <axis xyz="0 0 1"/>
     <limit effort="100" velocity="100.0"  lower="-5000" upper="5000" />
@@ -145,5 +145,5 @@
   <link name="caster_front_link">
     <visual>
-      <origin xyz="0 0.150 0" rpy="1.57 0 0"/>
+      <origin xyz="0 0.150 0" rpy="${PI/2} 0 0"/>
       <geometry>
         <cylinder length="0.025" radius="0.050"/>
@@ -152,5 +152,5 @@
     </visual>
     <visual>
-      <origin xyz="0 -0.150 0" rpy="1.57 0 0"/>
+      <origin xyz="0 -0.150 0" rpy="${PI/2} 0 0"/>
       <geometry>
         <cylinder length="0.025" radius="0.050"/>
@@ -159,11 +159,11 @@
     </visual>
     <collision>
-      <origin xyz="0 0.150 0" rpy="1.57 0 0"/>
-      <geometry>
-        <cylinder length="0.025" radius="0.050"/>
-      </geometry>
-    </collision>
-    <collision>
-      <origin xyz="0 -0.150 0" rpy="1.57 0 0"/>
+      <origin xyz="0 0.150 0" rpy="${PI/2} 0 0"/>
+      <geometry>
+        <cylinder length="0.025" radius="0.050"/>
+      </geometry>
+    </collision>
+    <collision>
+      <origin xyz="0 -0.150 0" rpy="${PI/2} 0 0"/>
       <geometry>
         <cylinder length="0.025" radius="0.050"/>
@@ -179,9 +179,9 @@
   <!-- Setting for imu -->
   <xacro:sensor_imu name="imu" parent="base_link" size="0.05 0.05 0.05">
-    <origin xyz="0.3 0 0.0925" rpy="0 0 -1.57"/>
+    <origin xyz="0.3 0 0.0925" rpy="0 0 ${-PI/2}"/>
   </xacro:sensor_imu>
   <xacro:include filename="$(find icart_mini_description)/urdf/sensors/hokuyo.urdf.xacro"/>
   <xacro:sensor_hokuyo name="hokuyo" parent="base_link">
-    <origin xyz="0.374295 0 0.0665" rpy="-3.14 0 0"/>
+    <origin xyz="0.374295 0 0.0665" rpy="${-PI} 0 0"/>
   </xacro:sensor_hokuyo>
   <transmission name="tran1">

Commit message: changes orne_box.gazebo.xacro

File: orne_box_description/urdf/orne_box.gazebo.xacro (robot description, xacro)
@@ -6,5 +6,6 @@
   <gazebo>
     <plugin name="gazebo_ros_control" filename="libgazebo_ros_control.so">
-      <robotSimType>icart_mini_gazebo/ICartMiniHWSim</robotSimType>
+      <robotNamespace>/orne-box</robotNamespace>
+      <robotSimType>gazebo_ros_control/DefaultRobotHWSim</robotSimType>
     </plugin>
   </gazebo>
@@ -40,5 +41,5 @@
       <visualize>$(arg imu_visual)</visualize>
     </sensor>
-    <material>Gazebo/FlatBlack</material>
+    <material>Gazebo/Green</material>
   </gazebo>
   <!-- hokuyo -->
@@ -77,4 +78,5 @@
       </plugin>
     </sensor>
+    <material>Gazebo/Black</material>
   </gazebo>
 </robot>

Commit message: add argument ignition_gazebo

File: orne_box_description/urdf/orne_box.gazebo.xacro (robot description, xacro)
@@ -4,79 +4,83 @@
   <xacro:arg name="laser_visual" default="true"/>
   <xacro:arg name="imu_visual"   default="false"/>
-  <gazebo>
-    <plugin name="gazebo_ros_control" filename="libgazebo_ros_control.so">
-      <robotNamespace>orne_box</robotNamespace>
-      <robotSimType>gazebo_ros_control/DefaultRobotHWSim</robotSimType>
-    </plugin>
-  </gazebo>
-  <gazebo reference="base_link">
-    <material>Gazebo/Orange</material>
-  </gazebo>
-  <gazebo reference="left_wheel">
-    <mu1>1.0</mu1>
-    <mu2>1.0</mu2>
-    <kp>1000000.0</kp>
-    <kd>100.0</kd>
-    <minDepth>0.001</minDepth>
-    <maxVel>1.0</maxVel>
-    <material>Gazebo/White</material>
-  </gazebo>
-  <gazebo reference="right_wheel">
-    <mu1>1.0</mu1>
-    <mu2>1.0</mu2>
-    <kp>1000000.0</kp>
-    <kd>100.0</kd>
-    <minDepth>0.001</minDepth>
-    <maxVel>1.0</maxVel>
-    <material>Gazebo/White</material>
-  </gazebo>
-  <gazebo reference="caster_front_link">
-    <mu1>0.0</mu1>
-    <mu2>0.0</mu2>
-    <material>Gazebo/Red</material>
-  </gazebo>
-  <gazebo reference="imu_link">
-    <sensor type="imu" name="imu">
-      <always_on>true</always_on>
-      <visualize>$(arg imu_visual)</visualize>
-    </sensor>
-    <material>Gazebo/Green</material>
-  </gazebo>
-  <!-- hokuyo -->
-  <gazebo reference="hokuyo_link">
-    <sensor type="ray" name="head_hokuyo_sensor">
-      <pose>0 0 0 0 0 0</pose>
-      <visualize>$(arg laser_visual)</visualize>
-      <update_rate>40</update_rate>
-      <ray>
-        <scan>
-          <horizontal>
-            <samples>880</samples>
-            <resolution>0.25</resolution>
-            <min_angle>${-PI/180*110}</min_angle>
-            <max_angle>${ PI/180*110}</max_angle>
-          </horizontal>
-        </scan>
-        <range>
-          <min>0.10</min>
-          <max>30.0</max>
-          <resolution>0.01</resolution>
-        </range>
-        <noise>
-          <type>gaussian</type>
-          <!-- Noise parameters based on published spec for Hokuyo laser
-               achieving "+-30mm" accuracy at range < 10m.  A mean of 0.0m and
-               stddev of 0.01m will put 99.7% of samples within 0.03m of the true
-               reading. -->
-          <mean>0.0</mean>
-          <stddev>0.01</stddev>
-        </noise>
-      </ray>
-      <plugin name="gazebo_ros_head_hokuyo_controller" filename="libgazebo_ros_laser.so">
-        <topicName>/scan</topicName>
-        <frameName>hokuyo_link</frameName>
+  <xacro:arg name="ignition_gazebo" default="false"/>
+  <!-- @TODO More clear boolean operation -->
+  <xacro:if value="${'$(arg ignition_gazebo)' == 'false'}">
+    <gazebo>
+      <plugin name="gazebo_ros_control" filename="libgazebo_ros_control.so">
+        <robotNamespace>orne_box</robotNamespace>
+        <robotSimType>gazebo_ros_control/DefaultRobotHWSim</robotSimType>
       </plugin>
-    </sensor>
-    <material>Gazebo/Black</material>
-  </gazebo>
+    </gazebo>
+    <gazebo reference="base_link">
+      <material>Gazebo/Orange</material>
+    </gazebo>
+    <gazebo reference="left_wheel">
+      <mu1>1.0</mu1>
+      <mu2>1.0</mu2>
+      <kp>1000000.0</kp>
+      <kd>100.0</kd>
+      <minDepth>0.001</minDepth>
+      <maxVel>1.0</maxVel>
+      <material>Gazebo/White</material>
+    </gazebo>
+    <gazebo reference="right_wheel">
+      <mu1>1.0</mu1>
+      <mu2>1.0</mu2>
+      <kp>1000000.0</kp>
+      <kd>100.0</kd>
+      <minDepth>0.001</minDepth>
+      <maxVel>1.0</maxVel>
+      <material>Gazebo/White</material>
+    </gazebo>
+    <gazebo reference="caster_front_link">
+      <mu1>0.0</mu1>
+      <mu2>0.0</mu2>
+      <material>Gazebo/Red</material>
+    </gazebo>
+    <gazebo reference="imu_link">
+      <sensor type="imu" name="imu">
+        <always_on>true</always_on>
+        <visualize>$(arg imu_visual)</visualize>
+      </sensor>
+      <material>Gazebo/Green</material>
+    </gazebo>
+    <!-- hokuyo -->
+    <gazebo reference="hokuyo_link">
+      <sensor type="ray" name="head_hokuyo_sensor">
+        <pose>0 0 0 0 0 0</pose>
+        <visualize>$(arg laser_visual)</visualize>
+        <update_rate>40</update_rate>
+        <ray>
+          <scan>
+            <horizontal>
+              <samples>880</samples>
+              <resolution>0.25</resolution>
+              <min_angle>${-PI/180*110}</min_angle>
+              <max_angle>${ PI/180*110}</max_angle>
+            </horizontal>
+          </scan>
+          <range>
+            <min>0.10</min>
+            <max>30.0</max>
+            <resolution>0.01</resolution>
+          </range>
+          <noise>
+            <type>gaussian</type>
+            <!-- Noise parameters based on published spec for Hokuyo laser
+                 achieving "+-30mm" accuracy at range < 10m.  A mean of 0.0m and
+                 stddev of 0.01m will put 99.7% of samples within 0.03m of the true
+                 reading. -->
+            <mean>0.0</mean>
+            <stddev>0.01</stddev>
+          </noise>
+        </ray>
+        <plugin name="gazebo_ros_head_hokuyo_controller" filename="libgazebo_ros_laser.so">
+          <topicName>/scan</topicName>
+          <frameName>hokuyo_link</frameName>
+        </plugin>
+      </sensor>
+      <material>Gazebo/Black</material>
+    </gazebo>
+  </xacro:if>
 </robot>

File: orne_box_description/urdf/sensors/imu.urdf.xacro (robot description, xacro)
@@ -3,4 +3,5 @@
                          xmlns:controller="http://playerstage.sourceforge.net/gazebo/xmlschema/#controller"
                          xmlns:interface="http://playerstage.sourceforge.net/gazebo/xmlschema/#interface">
+  <xacro:arg name="ignition_gazebo" default="false"/>
   <xacro:macro name="sensor_imu" params="name parent *origin size">
     <joint name="${name}_joint" type="fixed">
@@ -19,13 +20,16 @@
       </visual>
     </link>
-    <gazebo>
-      <plugin name="ros_imu" filename="libgazebo_ros_imu.so">
-        <bodyName>imu_link</bodyName> <!-- bodyName always set base_link by URDF parser -->
-        <topicName>imu_data</topicName>
-        <serviceName>imu_service</serviceName>
-        <gaussianNoise>0.005</gaussianNoise>
-        <updateRate>100.0</updateRate>
-      </plugin>
-    </gazebo>
+    <!-- @TODO More clear boolean operation -->
+    <xacro:if value="${'$(arg ignition_gazebo)' == 'false'}">
+      <gazebo>
+        <plugin name="ros_imu" filename="libgazebo_ros_imu.so">
+          <bodyName>imu_link</bodyName> <!-- bodyName always set base_link by URDF parser -->
+          <topicName>imu_data</topicName>
+          <serviceName>imu_service</serviceName>
+          <gaussianNoise>0.005</gaussianNoise>
+          <updateRate>100.0</updateRate>
+        </plugin>
+      </gazebo>
+    </xacro:if>
   </xacro:macro>
 </robot>

Commit message: add sensor plugin for ign gazebo

File: orne_box_description/urdf/orne_box.gazebo.xacro (robot description, xacro)
@@ -84,3 +84,110 @@
     </gazebo>
   </xacro:if>
+  <xacro:if value="$(arg ignition_gazebo)">
+    <gazebo>
+      <plugin filename="ignition-gazebo-joint-state-publisher-system" name="ignition::gazebo::systems::JointStatePublisher">
+        <topic>model/orne_box/joint_states</topic>
+      </plugin>
+      <plugin filename="ignition-gazebo-pose-publisher-system" name="ignition::gazebo::systems::PosePublisher">
+        <publish_link_pose>true</publish_link_pose>
+        <publish_collision_pose>true</publish_collision_pose>
+        <publish_visual_pose>false</publish_visual_pose>
+        <publish_nested_model_pose>false</publish_nested_model_pose>
+      </plugin>
+      <plugin filename="ignition-gazebo-diff-drive-system" name="ignition::gazebo::systems::DiffDrive">
+        <left_joint>left_wheel_joint</left_joint>
+        <right_joint>right_wheel_joint</right_joint>
+        <wheel_separation>1.25</wheel_separation>
+        <wheel_radius>0.3</wheel_radius>
+        <odom_publish_frequency>10</odom_publish_frequency>
+        <max_linear_acceleration>1</max_linear_acceleration>
+        <min_linear_acceleration>-1</min_linear_acceleration>
+        <max_angular_acceleration>2</max_angular_acceleration>
+        <min_angular_acceleration>-2</min_angular_acceleration>
+        <max_linear_velocity>0.5</max_linear_velocity>
+        <min_linear_velocity>-0.5</min_linear_velocity>
+        <max_angular_velocity>1</max_angular_velocity>
+        <min_angular_velocity>-1</min_angular_velocity>
+        <topic>cmd_vel</topic>
+      </plugin>
+    </gazebo>
+    <gazebo reference="hokuyo_link">
+      <sensor type="gpu_lidar" name="head_hokuyo_sensor">
+        <pose>0 0 0 0 0 0</pose>
+        <visualize>$(arg laser_visual)</visualize>
+        <update_rate>40</update_rate>
+        <topic>model/orne_box/hokuyo_scan</topic>
+        <lidar>
+          <scan>
+            <horizontal>
+              <samples>361</samples>
+              <resolution>0.25</resolution>
+              <min_angle>${-PI/180*110}</min_angle>
+              <max_angle>${ PI/180*110}</max_angle>
+            </horizontal>
+          </scan>
+          <range>
+            <min>0.10</min>
+            <max>30.0</max>
+            <resolution>0.01</resolution>
+          </range>
+          <noise>
+            <type>gaussian</type>
+            <mean>0.0</mean>
+            <stddev>0.01</stddev>
+          </noise>
+        </lidar>
+      </sensor>
+    </gazebo>
+    <gazebo reference="imu_link">
+      <sensor name="imu_link" type="imu">
+        <always_on>1</always_on>
+        <update_rate>200</update_rate>
+        <visualize>false</visualize>
+        <topic>model/orne_box/imu</topic>
+        <imu>
+          <angular_velocity>
+            <x>
+              <noise type="gaussian">
+                <mean>0.0</mean>
+                <stddev>0.1</stddev>
+              </noise>
+            </x>
+            <y>
+              <noise type="gaussian">
+                <mean>0.0</mean>
+                <stddev>0.1</stddev>
+              </noise>
+            </y>
+            <z>
+              <noise type="gaussian">
+                <mean>0.0</mean>
+                <stddev>0.2</stddev>
+              </noise>
+            </z>
+          </angular_velocity>
+          <linear_acceleration>
+            <x>
+              <noise type="gaussian">
+                <mean>0.0</mean>
+                <stddev>0.1</stddev>
+              </noise>
+            </x>
+            <y>
+              <noise type="gaussian">
+                <mean>0.0</mean>
+                <stddev>0.1</stddev>
+              </noise>
+            </y>
+            <z>
+              <noise type="gaussian">
+                <mean>0.0</mean>
+                <stddev>0.2</stddev>
+              </noise>
+            </z>
+          </linear_acceleration>
+        </imu>
+      </sensor>
+    </gazebo>
+  </xacro:if>
 </robot>

File: orne_box_description/urdf/orne_box_3d_lidar.urdf.xacro (robot description, xacro)
@@ -11,4 +11,67 @@
     </xacro:VLP-16>
   </xacro:if>
+  <xacro:if value="$(arg ignition_gazebo)">
+    <link name="surestar">
+      <inertial>
+        <origin xyz="0.0 0.0 0.0" rpy="0.0 0.0 0.0"/>
+        <mass value="0.3"/>
+        <inertia ixx="0.0" ixy="0.0" ixz="0.0" iyy="0.0" iyz="0.0" izz="0.0"/>
+      </inertial>
+      <visual name="">
+        <origin xyz="0.0 0.0 0.0" rpy="0.0 0.0 0.0"/>
+        <geometry>
+          <cylinder radius="0.06" length="0.1"/>
+        </geometry>
+        <material name="">
+          <color rgba="0.0 1.0 0.0 1.0"/>
+        </material>
+      </visual>
+      <collision>
+        <origin xyz="0.0 0.0 0.0" rpy="0.0 0.0 0.0"/>
+        <geometry>
+          <cylinder radius="0.06" length="0.13"/>
+        </geometry>
+      </collision>
+    </link>
+    <joint name="surestar_joint" type="fixed">
+      <origin xyz="0.23 0.0 0.4" rpy="0.0 0.0 0.0"/>
+      <parent link="base_link"/>
+      <child link="surestar"/>
+    </joint>
+    <gazebo reference="surestar">
+      <sensor name="surestar" type="gpu_lidar">
+        <alwaysOn>1</alwaysOn>
+        <update_rate>10</update_rate>
+        <visualize>true</visualize>
+        <lidar>
+          <scan>
+            <horizontal>
+              <!-- Correct points of 1875 -->
+              <samples>722</samples>
+              <resolution>1</resolution>
+              <min_angle>-3.141592</min_angle>
+              <max_angle>3.141592</max_angle>
+            </horizontal>
+            <vertical>
+              <samples>16</samples>
+              <resolution>1</resolution>
+              <min_angle>-0.261799</min_angle>
+              <max_angle>0.261799</max_angle>
+            </vertical>
+          </scan>
+          <range>
+            <min>0.3</min>
+            <max>100.0</max>
+            <resolution>0.001</resolution>
+          </range>
+          <noise type="gaussian">
+            <mean>0.0</mean>
+            <stddev>0.02</stddev>
+          </noise>
+        </lidar>
+        <topic>model/orne_box/rfans</topic>
+      </sensor>
+    </gazebo>
+  </xacro:if>
   <xacro:include filename="$(find orne_box_description)/urdf/sensors/gnss.urdf.xacro"/>
   <xacro:include filename="$(find orne_box_description)/urdf/sensors/camera.urdf.xacro"/>

Commit message: support new caster wheel link

File: orne_box_description/urdf/orne_box.gazebo.xacro (robot description, xacro)
@@ -6,7 +6,15 @@
   <xacro:arg name="ignition_gazebo" default="false"/>
   <xacro:arg name="enable_camera" default="false"/>
-  <gazebo reference="caster_front_link">
-    <mu1>0.0001</mu1>
-    <mu2>0.0001</mu2>
+  <gazebo reference="left_caster_wheel_link">
+    <mu1>0.75</mu1>
+    <mu2>0.75</mu2>
+    <kp>1000000.0</kp>
+    <kd>100.0</kd>
+    <minDepth>0.001</minDepth>
+    <maxVel>1.0</maxVel>
+  </gazebo>
+  <gazebo reference="right_caster_wheel_link">
+    <mu1>0.75</mu1>
+    <mu2>0.75</mu2>
     <kp>1000000.0</kp>
     <kd>100.0</kd>
@@ -15,6 +23,6 @@
   </gazebo>
   <gazebo reference="left_wheel">
-    <mu1>0.95</mu1>
-    <mu2>0.95</mu2>
+    <mu1>0.85</mu1>
+    <mu2>0.85</mu2>
     <kp>1000000.0</kp>
     <kd>100.0</kd>
@@ -24,6 +32,6 @@
   </gazebo>
   <gazebo reference="right_wheel">
-    <mu1>0.95</mu1>
-    <mu2>0.95</mu2>
+    <mu1>0.85</mu1>
+    <mu2>0.85</mu2>
     <kp>1000000.0</kp>
     <kd>100.0</kd>
@@ -113,4 +121,16 @@
       </plugin>
       <plugin filename="libignition-gazebo-wheel-slip-system.so" name="ignition::gazebo::systems::WheelSlip">
+        <wheel link_name="left_caster_wheel_link">
+          <slip_compliance_lateral>0.6</slip_compliance_lateral>
+          <slip_compliance_longitudinal>0.45</slip_compliance_longitudinal>
+          <wheel_normal_force>80.6</wheel_normal_force>
+          <wheel_radius>0.04</wheel_radius>
+        </wheel>
+        <wheel link_name="right_caster_wheel_link">
+          <slip_compliance_lateral>0.6</slip_compliance_lateral>
+          <slip_compliance_longitudinal>0.45</slip_compliance_longitudinal>
+          <wheel_normal_force>80.6</wheel_normal_force>
+          <wheel_radius>0.04</wheel_radius>
+        </wheel>
         <wheel link_name="wheel_left_link">
           <slip_compliance_lateral>0.6</slip_compliance_lateral>

File: orne_box_description/urdf/orne_box.urdf.xacro (robot description, xacro)
@@ -5,9 +5,7 @@
   <xacro:include filename="$(find orne_box_description)/urdf/orne_box.gazebo.xacro"/>
   <xacro:include filename="$(find orne_box_description)/urdf/links/base_link.urdf.xacro"/>
-  <xacro:include filename="$(find orne_box_description)/urdf/links/caster_link.urdf.xacro"/>
   <xacro:include filename="$(find orne_box_description)/urdf/links/caster_wheel_link.urdf.xacro"/>
   <xacro:include filename="$(find orne_box_description)/urdf/links/caster_swivel_link.urdf.xacro"/>
   <xacro:include filename="$(find orne_box_description)/urdf/links/wheel_link.urdf.xacro"/>
-  <xacro:include filename="$(find orne_box_description)/urdf/joints/caster_joint.urdf.xacro"/>
   <xacro:include filename="$(find orne_box_description)/urdf/joints/caster_wheel_joint.urdf.xacro"/>
   <xacro:include filename="$(find orne_box_description)/urdf/joints/caster_swivel_joint.urdf.xacro"/>
@@ -18,10 +16,4 @@
   <xacro:base_link/>
   <!-- Setting for caster -->
-  <!--
-  <xacro:caster_joint parent="base_link">
-    <origin xyz="0.362 0.0 0.050" rpy="0 0 0"/>
-  </xacro:caster_joint>
-  <xacro:caster_link/>
-  -->
   <xacro:caster_wheel_link prefix="left"/>
   <xacro:caster_swivel_link prefix="left"/>
