Commit message: add simulation models

File: orne_box_description/urdf/orne_box.gazebo.xacro (robot description, xacro)
@@ -99,4 +99,109 @@
       <material>Gazebo/Black</material>
     </gazebo>
+<gazebo reference="lidar_with_mirror_center_link">
+    <sensor type="ray" name="lidar_with_mirror_center_sensor">
+      <pose>0 0 0 0 0 0</pose>
+      <visualize>$(arg laser_visual)</visualize>
+      <update_rate>10</update_rate>
+      <ray>
+        <scan>
+          <horizontal>
+            <samples>341</samples>
+            <resolution>1</resolution>
+            <min_angle>${-PI/180*60}</min_angle>
+            <max_angle>${ PI/180*60}</max_angle>
+          </horizontal>
+        </scan>
+        <range>
+          <min>0.10</min>
+          <max>5.60</max>
+          <resolution>0.001</resolution>
+        </range>
+        <noise>
+          <type>gaussian</type>
+          <!-- Noise parameters based on published spec for Hokuyo laser
+               achieving "+-30mm" accuracy at range < 10m.  A mean of 0.0m and
+               stddev of 0.01m will put 99.7% of samples within 0.03m of the true
+               reading. -->
+          <mean>0.0</mean>
+          <stddev>0.01</stddev>
+        </noise>
+      </ray>
+      <plugin name="gazebo_ros_head_hokuyo_controller" filename="libgazebo_ros_laser.so">
+        <topicName>/lidar_with_mirror_scan_center</topicName>
+        <frameName>lidar_with_mirror_center_link</frameName>
+      </plugin>
+    </sensor>
+  </gazebo>
+  <gazebo reference="lidar_with_mirror_left_link">
+    <sensor type="ray" name="lidar_with_mirror_left_sensor">
+      <pose>0 0 0 0 0 0</pose>
+      <visualize>$(arg laser_visual)</visualize>
+      <update_rate>10</update_rate>
+      <ray>
+        <scan>
+          <horizontal>
+            <samples>170</samples>
+            <resolution>1</resolution>
+            <min_angle>${PI/180*60}</min_angle>
+            <max_angle>${PI/180*120}</max_angle>
+          </horizontal>
+        </scan>
+        <range>
+          <min>0.10</min>
+          <max>5.60</max>
+          <resolution>0.001</resolution>
+        </range>
+        <noise>
+          <type>gaussian</type>
+          <!-- Noise parameters based on published spec for Hokuyo laser
+               achieving "+-30mm" accuracy at range < 10m.  A mean of 0.0m and
+               stddev of 0.01m will put 99.7% of samples within 0.03m of the true
+               reading. -->
+          <mean>0.0</mean>
+          <stddev>0.01</stddev>
+        </noise>
+      </ray>
+      <plugin name="gazebo_ros_head_hokuyo_controller" filename="libgazebo_ros_laser.so">
+        <topicName>/lidar_with_mirror_scan_left</topicName>
+        <frameName>lidar_with_mirror_left_link</frameName>
+      </plugin>
+    </sensor>
+  </gazebo>
+  <gazebo reference="lidar_with_mirror_right_link">
+    <sensor type="ray" name="lidar_with_mirror_right_sensor">
+      <pose>0 0 0 0 0 0</pose>
+      <visualize>$(arg laser_visual)</visualize>
+      <update_rate>10</update_rate>
+      <ray>
+        <scan>
+          <horizontal>
+            <samples>170</samples>
+            <resolution>1</resolution>
+            <min_angle>${-PI/180*120}</min_angle>
+            <max_angle>${-PI/180*60}</max_angle>
+          </horizontal>
+        </scan>
+        <range>
+          <min>0.10</min>
+          <max>5.60</max>
+          <resolution>0.001</resolution>
+        </range>
+        <noise>
+          <type>gaussian</type>
+          <!-- Noise parameters based on published spec for Hokuyo laser
+               achieving "+-30mm" accuracy at range < 10m.  A mean of 0.0m and
+               stddev of 0.01m will put 99.7% of samples within 0.03m of the true
+               reading. -->
+          <mean>0.0</mean>
+          <stddev>0.01</stddev>
+        </noise>
+      </ray>
+      <plugin name="gazebo_ros_head_hokuyo_controller" filename="libgazebo_ros_laser.so">
+        <topicName>/lidar_with_mirror_scan_right</topicName>
+        <frameName>lidar_with_mirror_right_link</frameName>
+      </plugin>
+    </sensor>
+  </gazebo>
   </xacro:if>
   <xacro:if value="$(arg ignition_gazebo)">

File: orne_box_description/urdf/orne_box.urdf.xacro (robot description, xacro)
@@ -52,3 +52,85 @@
     <origin xyz="0.374295 0 0.2185" rpy="${-PI} 0 0"/>
   </xacro:sensor_hokuyo>
+    <joint name="lidar_with_mirror_prismatic_joint" type="prismatic">
+    <parent link="base_link"/>
+    <child link="lidar_with_mirror_prismatic_link"/>
+    <origin xyz="1.0 0 0.3" rpy="0 0 0"/>
+    <axis xyz="0 0 1"/>
+    <limit effort="100" velocity="100.0" lower="-0.3" upper="1" />
+  </joint>
+  <link name="lidar_with_mirror_prismatic_link">
+    <inertial>
+      <origin xyz="0 0 0" />
+      <mass value="0.2" />
+      <inertia ixx="0.1" ixy="0.0" ixz="0.0" iyy="0.1" iyz="0.0" izz="0.1" />
+    </inertial>
+  </link>
+  <joint name="lidar_with_mirror_pitch_joint" type="revolute">
+    <parent link="lidar_with_mirror_prismatic_link"/>
+    <child link="lidar_with_mirror_pitch_link"/>
+    <origin xyz="0 0 0" rpy="0 ${PI/9} 0"/>
+    <axis xyz="0 1 0"/>
+    <limit effort="100" velocity="100.0" lower="${-PI}" upper="${PI}" />
+  </joint>
+  <link name="lidar_with_mirror_pitch_link">
+    <inertial>
+      <origin xyz="0 0 0" />
+      <mass value="0.2" />
+      <inertia ixx="0.1" ixy="0.0" ixz="0.0" iyy="0.1" iyz="0.0" izz="0.1" />
+    </inertial>
+  </link>
+  <joint name="lidar_with_mirror_roll_joint" type="revolute">
+    <parent link="lidar_with_mirror_pitch_link"/>
+    <child link="lidar_with_mirror_roll_link"/>
+    <origin xyz="0 0 0" rpy="0 0 0"/>
+    <axis xyz="1 0 0"/>
+    <limit effort="100" velocity="100.0" lower="${-PI}" upper="${PI}" />
+  </joint>
+  <link name="lidar_with_mirror_roll_link">
+    <inertial>
+      <origin xyz="0 0 0" />
+      <mass value="0.2" />
+      <inertia ixx="0.1" ixy="0.0" ixz="0.0" iyy="0.1" iyz="0.0" izz="0.1" />
+    </inertial>
+  </link>
+  <xacro:property name="len" value="0.1" />
+  <xacro:property name="front" value="0" />
+  <xacro:property name="height" value="0" />
+  <xacro:sensor_hokuyo name="lidar_with_mirror_center" parent="lidar_with_mirror_roll_link" size="0.05 0.05 0.05">
+    <origin xyz="${front} 0 ${height}" rpy="0 0 0"/>
+  </xacro:sensor_hokuyo>
+  <joint name="lidar_with_mirror_mirror1_roll_joint" type="revolute">
+    <parent link="lidar_with_mirror_center_link"/>
+    <child link="lidar_with_mirror_mirror1_roll_link"/>
+    <origin xyz="0 ${len} 0" rpy="${-PI/4} 0 0"/>
+    <axis xyz="-1 0 0"/>
+    <limit effort="100" velocity="100.0" lower="${-PI}" upper="${PI}" />
+  </joint>
+  <link name="lidar_with_mirror_mirror1_roll_link">
+    <inertial>
+      <origin xyz="0 0 0" />
+      <mass value="0.2" />
+      <inertia ixx="0.1" ixy="0.0" ixz="0.0" iyy="0.1" iyz="0.0" izz="0.1" />
+    </inertial>
+  </link>
+  <xacro:sensor_hokuyo name="lidar_with_mirror_left" parent="lidar_with_mirror_mirror1_roll_link" size="0.05 0.05 0.05">
+    <origin xyz="0 ${-len} 0" rpy="0 0 0"/>
+  </xacro:sensor_hokuyo>
+  <joint name="lidar_with_mirror_mirror2_roll_joint" type="revolute">
+    <parent link="lidar_with_mirror_center_link"/>
+    <child link="lidar_with_mirror_mirror2_roll_link"/>
+    <origin xyz="0 ${-len} 0" rpy="${PI/4} 0 0"/>
+    <axis xyz="1 0 0"/>
+    <limit effort="100" velocity="100.0" lower="${-PI}" upper="${PI}" />
+  </joint>
+  <link name="lidar_with_mirror_mirror2_roll_link">
+    <inertial>
+      <origin xyz="0 0 0" />
+      <mass value="0.2" />
+      <inertia ixx="0.1" ixy="0.0" ixz="0.0" iyy="0.1" iyz="0.0" izz="0.1" />
+    </inertial>
+  </link>
+  <xacro:sensor_hokuyo name="lidar_with_mirror_right" parent="lidar_with_mirror_mirror2_roll_link" size="0.05 0.05 0.05">
+    <origin xyz="0 ${len} 0" rpy="0 0 0"/>
+  </xacro:sensor_hokuyo>
 </robot>

Commit message: add mirror_lidar simulation

File: orne_box_description/urdf/orne_box.gazebo.xacro (robot description, xacro)
@@ -99,5 +99,5 @@
       <material>Gazebo/Black</material>
     </gazebo>
-<gazebo reference="lidar_with_mirror_center_link">
+  <gazebo reference="lidar_with_mirror_center_link">
     <sensor type="ray" name="lidar_with_mirror_center_sensor">
       <pose>0 0 0 0 0 0</pose>
@@ -116,5 +116,5 @@
           <min>0.10</min>
           <max>5.60</max>
-          <resolution>0.001</resolution>
+          <resolution>0.01</resolution>
         </range>
         <noise>

File: orne_box_description/urdf/orne_box.urdf.xacro (robot description, xacro)
@@ -52,5 +52,5 @@
     <origin xyz="0.374295 0 0.2185" rpy="${-PI} 0 0"/>
   </xacro:sensor_hokuyo>
-    <joint name="lidar_with_mirror_prismatic_joint" type="prismatic">
+  <joint name="lidar_with_mirror_prismatic_joint" type="prismatic">
     <parent link="base_link"/>
     <child link="lidar_with_mirror_prismatic_link"/>

Commit message: gnss simulator

File: orne_box_description/urdf/orne_box.gazebo.xacro (robot description, xacro)
@@ -78,3 +78,18 @@
     </sensor>
   </gazebo>
+  <link name="gps_link" />
+  <joint name="gps_joint" type="fixed">
+    <parent link="base_link" />
+    <child link="gps_link" />
+  </joint>
+  <gazebo>
+    <plugin name="gps" filename="libhector_gazebo_ros_gps.so">
+      <updateRate>10.0</updateRate>
+      <topicName>gps/fix</topicName>
+      <gaussianNoise>0.0 0.0 0.0</gaussianNoise>
+      <offset>0 0 0</offset>
+      <velocityGaussianNoise>0 0 0</velocityGaussianNoise>
+      <frameId>gps_link</frameId>
+    </plugin>
+  </gazebo>
 </robot>

Commit message: rm sensors

File: orne_box_description/urdf/orne_box.gazebo.xacro (robot description, xacro)
@@ -2,7 +2,6 @@
 <robot xmlns:xacro="http://ros.org/wiki/xacro" name="orne_box">
   <xacro:property name="PI" value="3.1415926535897931"/>
-  <xacro:arg name="laser_visual" default="true"/>
+  <!-- <xacro:arg name="laser_visual" default="true"/> -->
   <xacro:arg name="imu_visual" default="false"/>
-  <xacro:arg name="enable_camera" default="false"/>
   <gazebo reference="left_caster_wheel_link">
     <mu1>0.75</mu1>
@@ -145,5 +144,5 @@
     </gazebo>
     <!-- hokuyo -->
-    <gazebo reference="hokuyo_link">
+    <!-- <gazebo reference="hokuyo_link">
       <sensor type="ray" name="head_hokuyo_sensor">
         <pose>0 0 0 0 0 0</pose>
@@ -170,8 +169,4 @@
           <noise>
             <type>gaussian</type>
-            <!-- Noise parameters based on published spec for Hokuyo laser
-                 achieving "+-30mm" accuracy at range < 10m.  A mean of 0.0m and
-                 stddev of 0.01m will put 99.7% of samples within 0.03m of the true
-                 reading. -->
             <mean>0.0</mean>
             <stddev>0.01</stddev>
@@ -187,4 +182,4 @@
       </sensor>
       <material>Gazebo/Black</material>
-    </gazebo>
+    </gazebo> -->
 </robot>

File: orne_box_description/urdf/orne_box.urdf.xacro (robot description, xacro)
@@ -12,5 +12,5 @@
   <xacro:include filename="$(find orne_box_description)/urdf/joints/wheel_joint.urdf.xacro"/>
   <xacro:include filename="$(find orne_box_description)/urdf/sensors/imu.urdf.xacro"/>
-  <xacro:include filename="$(find orne_box_description)/urdf/sensors/hokuyo.urdf.xacro"/>
+  <!-- <xacro:include filename="$(find orne_box_description)/urdf/sensors/hokuyo.urdf.xacro"/> -->
   <!-- Setting for base -->
   <xacro:base_link/>
@@ -53,7 +53,7 @@
   </xacro:sensor_imu>
   <!-- Setting for 2D-LiDAR -->
-  <xacro:sensor_hokuyo name="hokuyo" parent="base_link" size="0.05 0.05 0.05">
-    <origin xyz="0.364295 0 0.185" rpy="3.14 0 0"/>
-  </xacro:sensor_hokuyo>
+  <!-- <xacro:sensor_hokuyo name="hokuyo" parent="base_link" size="0.05 0.05 0.05"> -->
+    <!-- <origin xyz="0.364295 0 0.185" rpy="3.14 0 0"/>
+  </xacro:sensor_hokuyo> -->
   <!-- <xacro:sensor_hokuyo name="mirror_lidar" parent="base_link" size="0.05 0.05 0.05">
     <origin xyz="0.43 0.0 0.34" rpy="0 0.314 0"/>

File: orne_box_description/urdf/orne_box_3d_lidar_rfans.urdf.xacro (robot description, xacro)
@@ -73,5 +73,5 @@
     </gazebo>
   </xacro:if>
-  <xacro:include filename="$(find orne_box_description)/urdf/sensors/gnss.urdf.xacro"/>
+  <!-- <xacro:include filename="$(find orne_box_description)/urdf/sensors/gnss.urdf.xacro"/>
   <xacro:include filename="$(find orne_box_description)/urdf/sensors/camera.urdf.xacro"/>
   <xacro:sensor_gnss name="gnss" parent="base_link">
@@ -80,4 +80,4 @@
   <xacro:sensor_camera name="camera" parent="base_link">
     <origin xyz="-0.08 0.0 0.8" rpy="0 0.38 0"/>
-  </xacro:sensor_camera>
+  </xacro:sensor_camera> -->
 </robot>
