Commit message: add 2D lidar for low obstacle detection in gazebo classic
- restore hokuyo.urdf.xacro and mount it at the old hokuyo position
- publish the ray sensor as /low_scan without visualization

Co-Authored-By: Claude Opus 5.5 <noreply@anthropic.com>

File: orne_box_description/urdf/orne_box.gazebo.xacro (robot description, xacro)
@@ -2,5 +2,5 @@
 <robot xmlns:xacro="http://ros.org/wiki/xacro" name="orne_box">
   <xacro:property name="PI" value="3.1415926535897931"/>
-  <xacro:arg name="laser_visual" default="true"/>
+  <xacro:arg name="laser_visual" default="false"/>
   <!--<xacro:arg name="imu_visual" default="false"/> -->
   <!--<xacro:arg name="enable_camera" default="false"/>-->
@@ -151,5 +151,5 @@
     </gazebo>
     <!-- hokuyo -->
-    <!--<gazebo reference="hokuyo_link">
+    <gazebo reference="hokuyo_link">
       <sensor type="ray" name="head_hokuyo_sensor">
         <pose>0 0 0 0 0 0</pose>
@@ -182,5 +182,5 @@
         <plugin name="gazebo_ros_head_hokuyo_controller" filename="libgazebo_ros_ray_sensor.so">
           <ros>
-            <remapping>~/out:=hokuyo_scan</remapping>
+            <remapping>~/out:=low_scan</remapping>
           </ros>
           <frame_name>hokuyo_link</frame_name>
@@ -189,4 +189,4 @@
       </sensor>
       <material>Gazebo/Black</material>
-    </gazebo> -->
+    </gazebo>
 </robot>

File: orne_box_description/urdf/orne_box_3d_lidar_rfans.urdf.xacro (robot description, xacro)
@@ -12,4 +12,9 @@
       <origin xyz="-0.12 0 0.60" rpy="0 0 0"/>
     </xacro:VLP-16>
+    <!-- Setting for 2D-LiDAR (低層障害物認識用, /low_scan) -->
+    <xacro:include filename="$(find orne_box_description)/urdf/sensors/hokuyo.urdf.xacro"/>
+    <xacro:sensor_hokuyo name="hokuyo" parent="base_link" size="0.05 0.05 0.05">
+      <origin xyz="0.364295 0 0.185" rpy="3.14 0 0"/>
+    </xacro:sensor_hokuyo>
   </xacro:if>
   <!-- @Ignition gazebo -->
