Commit message: edit xml and fix indentation in orne_box_description

File: orne_box_description/urdf/joints/caster_joint.urdf.xacro (robot description, xacro)
@@ -1,10 +1,10 @@
-<?xml version="1.0" ?>
+<?xml version="1.0"?>
 <robot xmlns:xacro="http://www.ros.org/wiki/xacro">
-	<xacro:macro name="caster_joint" params="parent *origin">
-		<joint name="caster_joint" type="fixed">
-			<parent link="${parent}"/>
-	    <child link="caster_front_link"/>
-			<xacro:insert_block name="origin"/>
-		</joint>
-	</xacro:macro>
+  <xacro:macro name="caster_joint" params="parent *origin">
+    <joint name="caster_joint" type="fixed">
+      <parent link="${parent}"/>
+      <child link="caster_front_link"/>
+      <xacro:insert_block name="origin"/>
+    </joint>
+  </xacro:macro>
 </robot>

File: orne_box_description/urdf/joints/wheel_joint.urdf.xacro (robot description, xacro)
@@ -1,22 +1,22 @@
-<?xml version="1.0" ?>
+<?xml version="1.0"?>
 <robot xmlns:xacro="http://www.ros.org/wiki/xacro">
-	<xacro:macro name="wheel_joint" params="prefix parent *origin *axis">
-		<joint name="${prefix}_wheel_hinge" type="revolute">
-			<parent link="${parent}"/>
-	    <child link="wheel_${prefix}_link"/>
-			<xacro:insert_block name="origin"/>
-			<xacro:insert_block name="axis"/>
-	    <limit effort="100" velocity="100.0"  lower="-5000" upper="5000" />
-		</joint>
-		<transmission name="transmission_${prefix}">
-		  <type>transmission_interface/SimpleTransmission</type>
-		  <joint name="${prefix}_wheel_hinge">
-		    <hardwareInterface>VelocityJointInterface</hardwareInterface>
-		  </joint>
-		<actuator name="${prefix}_motor">
-		    <hardwareInterface>VelocityJointInterface</hardwareInterface>
-		    <mechanicalReduction>1</mechanicalReduction>
-		  </actuator>
-		</transmission>
-	</xacro:macro>
+  <xacro:macro name="wheel_joint" params="prefix parent *origin *axis">
+    <joint name="${prefix}_wheel_hinge" type="revolute">
+      <parent link="${parent}"/>
+      <child link="wheel_${prefix}_link"/>
+      <xacro:insert_block name="origin"/>
+      <xacro:insert_block name="axis"/>
+      <limit effort="100" velocity="100.0" lower="-5000" upper="5000"/>
+    </joint>
+    <transmission name="transmission_${prefix}">
+      <type>transmission_interface/SimpleTransmission</type>
+      <joint name="${prefix}_wheel_hinge">
+        <hardwareInterface>VelocityJointInterface</hardwareInterface>
+      </joint>
+      <actuator name="${prefix}_motor">
+        <hardwareInterface>VelocityJointInterface</hardwareInterface>
+        <mechanicalReduction>1</mechanicalReduction>
+      </actuator>
+    </transmission>
+  </xacro:macro>
 </robot>

File: orne_box_description/urdf/links/base_link.urdf.xacro (robot description, xacro)
@@ -1,64 +1,64 @@
-<?xml version="1.0" ?>
+<?xml version="1.0"?>
 <robot xmlns:xacro="http://www.ros.org/wiki/xacro">
-	<xacro:macro name="base_link">
-	  <link name="base_link">
-		  <visual>
-		    <origin xyz="0.090 0 0.1715" rpy="0 0 0"/>
-		    <geometry>
-		      <box size="0.400 0.404 0.202"/>
-		    </geometry>
-		    <material name="orange"/>
-		  </visual>
-		  <visual>
-		    <origin xyz="0.36125 0 0.2625" rpy="0 0 0"/>
-		    <geometry>
-		      <box size="0.1425 0.404 0.020"/>
-		    </geometry>
-		    <material name="orange"/>
-		  </visual>
-		  <visual>
-		    <origin xyz="0.35625 0 0.156" rpy="0 0 0"/>
-		    <geometry>
-		      <box size="0.1325 0.404 0.020"/>
-		    </geometry>
-		    <material name="orange"/>
-		  </visual>
-		  <visual>
-		    <origin xyz="-0.120 0 0.4815" rpy="0 0 0"/>
-		    <geometry>
-		      <box size="0.020 0.404 0.822"/>
-		    </geometry>
-		    <material name="orange"/>
-		  </visual>
-		  <collision>
-		    <origin xyz="0.090 0 0.1715" rpy="0 0 0"/>
-		    <geometry>
-		      <box size="0.400 0.404 0.202"/>
-		    </geometry>
-		  </collision>
-		  <collision>
-		    <origin xyz="0.36125 0 0.2625" rpy="0 0 0"/>
-		    <geometry>
-		      <box size="0.1425 0.404 0.020"/>
-		    </geometry>
-		  </collision>
-		  <collision>
-		    <origin xyz="0.35625 0 0.156" rpy="0 0 0"/>
-		    <geometry>
-		      <box size="0.1325 0.404 0.020"/>
-		    </geometry>
-		  </collision>
-		  <collision>
-		    <origin xyz="-0.120 0 0.4815" rpy="0 0 0"/>
-		    <geometry>
-		      <box size="0.020 0.404 0.822"/>
-		    </geometry>
-		  </collision>
-		  <inertial>
-		    <origin xyz="0.090 0 0.1715" rpy="0 0 0"/>
-		    <mass value="25.0"/>
-		    <inertia ixx="1.0" ixy="0.0" ixz="0.0" iyy="1.0" iyz="0.0" izz="1.0" />
-		  </inertial>
-		</link>
-	</xacro:macro>
+  <xacro:macro name="base_link">
+    <link name="base_link">
+      <visual>
+        <origin xyz="0.090 0 0.1715" rpy="0 0 0"/>
+        <geometry>
+          <box size="0.400 0.404 0.202"/>
+        </geometry>
+        <material name="orange"/>
+      </visual>
+      <visual>
+        <origin xyz="0.36125 0 0.2625" rpy="0 0 0"/>
+        <geometry>
+          <box size="0.1425 0.404 0.020"/>
+        </geometry>
+        <material name="orange"/>
+      </visual>
+      <visual>
+        <origin xyz="0.35625 0 0.156" rpy="0 0 0"/>
+        <geometry>
+          <box size="0.1325 0.404 0.020"/>
+        </geometry>
+        <material name="orange"/>
+      </visual>
+      <visual>
+        <origin xyz="-0.120 0 0.4815" rpy="0 0 0"/>
+        <geometry>
+          <box size="0.020 0.404 0.822"/>
+        </geometry>
+        <material name="orange"/>
+      </visual>
+      <collision>
+        <origin xyz="0.090 0 0.1715" rpy="0 0 0"/>
+        <geometry>
+          <box size="0.400 0.404 0.202"/>
+        </geometry>
+      </collision>
+      <collision>
+        <origin xyz="0.36125 0 0.2625" rpy="0 0 0"/>
+        <geometry>
+          <box size="0.1425 0.404 0.020"/>
+        </geometry>
+      </collision>
+      <collision>
+        <origin xyz="0.35625 0 0.156" rpy="0 0 0"/>
+        <geometry>
+          <box size="0.1325 0.404 0.020"/>
+        </geometry>
+      </collision>
+      <collision>
+        <origin xyz="-0.120 0 0.4815" rpy="0 0 0"/>
+        <geometry>
+          <box size="0.020 0.404 0.822"/>
+        </geometry>
+      </collision>
+      <inertial>
+        <origin xyz="0.090 0 0.1715" rpy="0 0 0"/>
+        <mass value="25.0"/>
+        <inertia ixx="1.0" ixy="0.0" ixz="0.0" iyy="1.0" iyz="0.0" izz="1.0"/>
+      </inertial>
+    </link>
+  </xacro:macro>
 </robot>

File: orne_box_description/urdf/links/caster_link.urdf.xacro (robot description, xacro)
@@ -1,38 +1,38 @@
-<?xml version="1.0" ?>
+<?xml version="1.0"?>
 <robot xmlns:xacro="http://www.ros.org/wiki/xacro">
-	<xacro:macro name="caster_link">
-		<link name="caster_front_link">
-		  <visual>
-		    <origin xyz="0 0.150 0" rpy="${PI/2} 0 0"/>
-		    <geometry>
-		      <cylinder length="0.025" radius="0.050"/>
-		    </geometry>
-		    <material name="purple"/>
-		  </visual>
-		  <visual>
-		    <origin xyz="0 -0.150 0" rpy="${PI/2} 0 0"/>
-		    <geometry>
-		      <cylinder length="0.025" radius="0.050"/>
-		    </geometry>
-		    <material name="purple"/>
-		  </visual>
-		  <collision>
-		    <origin xyz="0 0.150 0" rpy="${PI/2} 0 0"/>
-		    <geometry>
-		      <cylinder length="0.025" radius="0.050"/>
-		    </geometry>
-		  </collision>
-		  <collision>
-		    <origin xyz="0 -0.150 0" rpy="${PI/2} 0 0"/>
-		    <geometry>
-		      <cylinder length="0.025" radius="0.050"/>
-		    </geometry>
-		  </collision>
-		  <inertial>
-		    <origin xyz="0 0 0" />
-		    <mass value="0.2" />
-		    <inertia ixx="0.1" ixy="0.0" ixz="0.0" iyy="0.1" iyz="0.0" izz="0.1" />
-		  </inertial>
-		</link>
-	</xacro:macro>
+  <xacro:macro name="caster_link">
+    <link name="caster_front_link">
+      <visual>
+        <origin xyz="0 0.150 0" rpy="${PI/2} 0 0"/>
+        <geometry>
+          <cylinder length="0.025" radius="0.050"/>
+        </geometry>
+        <material name="purple"/>
+      </visual>
+      <visual>
+        <origin xyz="0 -0.150 0" rpy="${PI/2} 0 0"/>
+        <geometry>
+          <cylinder length="0.025" radius="0.050"/>
+        </geometry>
+        <material name="purple"/>
+      </visual>
+      <collision>
+        <origin xyz="0 0.150 0" rpy="${PI/2} 0 0"/>
+        <geometry>
+          <cylinder length="0.025" radius="0.050"/>
+        </geometry>
+      </collision>
+      <collision>
+        <origin xyz="0 -0.150 0" rpy="${PI/2} 0 0"/>
+        <geometry>
+          <cylinder length="0.025" radius="0.050"/>
+        </geometry>
+      </collision>
+      <inertial>
+        <origin xyz="0 0 0"/>
+        <mass value="0.2"/>
+        <inertia ixx="0.1" ixy="0.0" ixz="0.0" iyy="0.1" iyz="0.0" izz="0.1"/>
+      </inertial>
+    </link>
+  </xacro:macro>
 </robot>

File: orne_box_description/urdf/links/wheel_link.urdf.xacro (robot description, xacro)
@@ -1,25 +1,25 @@
-<?xml version="1.0" ?>
+<?xml version="1.0"?>
 <robot xmlns:xacro="http://www.ros.org/wiki/xacro">
-	<xacro:macro name="wheel_link" params="prefix *origin width radius">
-	  <link name="wheel_${prefix}_link">
-			<visual>
-				<xacro:insert_block name="origin"/>
-	 	    <geometry>
-  	 	    <cylinder length="${width}" radius="${radius}"/>
-				</geometry>
-				<material name="white"/>
-			</visual>
-			<collision>
-				<xacro:insert_block name="origin"/>
-				<geometry>
-					<cylinder length="${width}" radius="${radius}"/>
-				</geometry>
-			</collision>
-	    <inertial>
-	      <origin xyz="0 0 0" />
-    	  <mass value="0.2" />
-  	    <inertia ixx="0.1" ixy="0.0" ixz="0.0" iyy="0.1" iyz="0.0" izz="0.1" />
-	    </inertial>
-	  </link>
-	</xacro:macro>
+  <xacro:macro name="wheel_link" params="prefix *origin width radius">
+    <link name="wheel_${prefix}_link">
+      <visual>
+        <xacro:insert_block name="origin"/>
+        <geometry>
+          <cylinder length="${width}" radius="${radius}"/>
+        </geometry>
+        <material name="white"/>
+      </visual>
+      <collision>
+        <xacro:insert_block name="origin"/>
+        <geometry>
+          <cylinder length="${width}" radius="${radius}"/>
+        </geometry>
+      </collision>
+      <inertial>
+        <origin xyz="0 0 0"/>
+        <mass value="0.2"/>
+        <inertia ixx="0.1" ixy="0.0" ixz="0.0" iyy="0.1" iyz="0.0" izz="0.1"/>
+      </inertial>
+    </link>
+  </xacro:macro>
 </robot>

File: orne_box_description/urdf/material_colors.xacro (robot description, xacro)
@@ -1,36 +1,36 @@
 <?xml version="1.0"?>
 <robot>
-	<material name="black">
-		<color rgba="0.0 0.0 0.0 1.0"/>
-	</material>
-	<material name="brown">
-		<color rgba="${222/255} ${207/255} ${195/255} 1.0"/>
-	</material>
-	<material name="red">
-		<color rgba="0.8 0.0 0.0 1.0"/>
-	</material>
-	<material name="orange">
-		<color rgba="${255/255} ${108/255} ${10/255} 1.0"/>
-	</material>
-	<material name="yellow">
-		<color rgba="0.8 0.8 0.0 1.0"/>
-	</material>
-	<material name="green">
-		<color rgba="0.0 0.8 0.0 1.0"/>
-	</material>
-	<material name="cyan">
-		<color rgba="0.0 0.8 0.8 1.0"/>
-	</material>
-	<material name="bule">
-		<color rgba="0.0 0.0 0.8 1.0"/>
-	</material>
-	<material name="purple">
-		<color rgba="0.8 0.0 0.8 1.0"/>
-	</material>
-	<material name="gray">
-		<color rgba="0.5 0.5 0.5 1.0"/>
-	</material>
-	<material name="white">
-		<color rgba="1.0 1.0 1.0 1.0"/>
-	</material>
+  <material name="black">
+    <color rgba="0.0 0.0 0.0 1.0"/>
+  </material>
+  <material name="brown">
+    <color rgba="${222/255} ${207/255} ${195/255} 1.0"/>
+  </material>
+  <material name="red">
+    <color rgba="0.8 0.0 0.0 1.0"/>
+  </material>
+  <material name="orange">
+    <color rgba="${255/255} ${108/255} ${10/255} 1.0"/>
+  </material>
+  <material name="yellow">
+    <color rgba="0.8 0.8 0.0 1.0"/>
+  </material>
+  <material name="green">
+    <color rgba="0.0 0.8 0.0 1.0"/>
+  </material>
+  <material name="cyan">
+    <color rgba="0.0 0.8 0.8 1.0"/>
+  </material>
+  <material name="bule">
+    <color rgba="0.0 0.0 0.8 1.0"/>
+  </material>
+  <material name="purple">
+    <color rgba="0.8 0.0 0.8 1.0"/>
+  </material>
+  <material name="gray">
+    <color rgba="0.5 0.5 0.5 1.0"/>
+  </material>
+  <material name="white">
+    <color rgba="1.0 1.0 1.0 1.0"/>
+  </material>
 </robot>

File: orne_box_description/urdf/orne_box.urdf.xacro (robot description, xacro)
@@ -12,10 +12,10 @@
   <xacro:include filename="$(find orne_box_description)/urdf/sensors/hokuyo.urdf.xacro"/>
   <!-- Setting for base -->
-	<xacro:base_link/>
+  <xacro:base_link/>
   <!-- Setting for caster -->
   <xacro:caster_joint parent="base_link">
     <origin xyz="0.362 0.0 0.050" rpy="0 0 0"/>
   </xacro:caster_joint>
-	<xacro:caster_link/>
+  <xacro:caster_link/>
   <!-- Setting for left wheel -->
   <xacro:wheel_joint prefix="left" parent="base_link">

File: orne_box_description/urdf/sensors/camera.urdf.xacro (robot description, xacro)
@@ -1,6 +1,6 @@
 <?xml version="1.0"?>
 <robot name="sensor_camera" xmlns:xacro="http://ros.org/wiki/xacro"
-                        xmlns:controller="http://playerstage.sourceforge.net/gazebo/xmlschema/#controller"
-                        xmlns:interface="http://playerstage.sourceforge.net/gazebo/xmlschema/#interface">
+                            xmlns:controller="http://playerstage.sourceforge.net/gazebo/xmlschema/#controller"
+                            xmlns:interface="http://playerstage.sourceforge.net/gazebo/xmlschema/#interface">
   <xacro:macro name="sensor_camera" params="name parent *origin">
     <joint name="${name}_joint" type="fixed">
@@ -13,8 +13,8 @@
       <visual>
         <origin rpy="0 0 0" xyz="0 0 0"/>
-				<geometry>
-	 	 			<box size="0.033 0.175 0.03"/>
-    	  </geometry>
-				<material name="bule"/>
+        <geometry>
+          <box size="0.033 0.175 0.03"/>
+        </geometry>
+        <material name="bule"/>
       </visual>
     </link>

File: orne_box_description/urdf/sensors/gnss.urdf.xacro (robot description, xacro)
@@ -1,6 +1,6 @@
 <?xml version="1.0"?>
 <robot name="sensor_gnss" xmlns:xacro="http://ros.org/wiki/xacro"
-                        xmlns:controller="http://playerstage.sourceforge.net/gazebo/xmlschema/#controller"
-                        xmlns:interface="http://playerstage.sourceforge.net/gazebo/xmlschema/#interface">
+                          xmlns:controller="http://playerstage.sourceforge.net/gazebo/xmlschema/#controller"
+                          xmlns:interface="http://playerstage.sourceforge.net/gazebo/xmlschema/#interface">
   <xacro:macro name="sensor_gnss" params="name parent *origin">
     <joint name="${name}_joint" type="fixed">
@@ -13,8 +13,8 @@
       <visual>
         <origin rpy="0 0 0" xyz="0 0 0"/>
-				<geometry>
+        <geometry>
           <cylinder  length="0.025" radius="0.05"/>
         </geometry>
-				<material name="red"/>
+        <material name="red"/>
       </visual>
     </link>

File: orne_box_description/urdf/sensors/hokuyo.urdf.xacro (robot description, xacro)
@@ -1,6 +1,6 @@
 <?xml version="1.0"?>
 <robot name="sensor_hokuyo" xmlns:xacro="http://ros.org/wiki/xacro"
-                        xmlns:controller="http://playerstage.sourceforge.net/gazebo/xmlschema/#controller"
-                        xmlns:interface="http://playerstage.sourceforge.net/gazebo/xmlschema/#interface">
+                            xmlns:controller="http://playerstage.sourceforge.net/gazebo/xmlschema/#controller"
+                            xmlns:interface="http://playerstage.sourceforge.net/gazebo/xmlschema/#interface">
   <xacro:macro name="sensor_hokuyo" params="name parent *origin size">
     <joint name="${name}_joint" type="fixed">
@@ -16,5 +16,5 @@
           <box size="${size}"/>
         </geometry>
-				<material name="black"/>
+        <material name="black"/>
       </visual>
     </link>

File: orne_box_description/urdf/sensors/imu.urdf.xacro (robot description, xacro)
@@ -1,6 +1,6 @@
 <?xml version="1.0"?>
 <robot name="sensor_imu" xmlns:xacro="http://ros.org/wiki/xacro"
-                        xmlns:controller="http://playerstage.sourceforge.net/gazebo/xmlschema/#controller"
-                        xmlns:interface="http://playerstage.sourceforge.net/gazebo/xmlschema/#interface">
+                         xmlns:controller="http://playerstage.sourceforge.net/gazebo/xmlschema/#controller"
+                         xmlns:interface="http://playerstage.sourceforge.net/gazebo/xmlschema/#interface">
   <xacro:macro name="sensor_imu" params="name parent *origin size">
     <joint name="${name}_joint" type="fixed">
@@ -16,5 +16,5 @@
           <box size="${size}"/>
         </geometry>
-				<material name="green"/>
+        <material name="green"/>
       </visual>
     </link>
