Commit message: Additional launch and configuration files for model visualization and simulation

File: orne_box_description/urdf/joints/wheel_joint.urdf.xacro (robot description, xacro)
@@ -2,5 +2,5 @@
 <robot xmlns:xacro="http://www.ros.org/wiki/xacro">
   <xacro:macro name="wheel_joint" params="prefix parent *origin *axis">
-    <joint name="${prefix}_wheel_hinge" type="revolute">
+    <joint name="${prefix}_wheel_joint" type="continuous">
       <parent link="${parent}"/>
       <child link="wheel_${prefix}_link"/>
@@ -11,9 +11,9 @@
     <transmission name="transmission_${prefix}">
       <type>transmission_interface/SimpleTransmission</type>
-      <joint name="${prefix}_wheel_hinge">
-        <hardwareInterface>VelocityJointInterface</hardwareInterface>
+      <joint name="${prefix}_wheel_joint">
+        <hardwareInterface>hardware_interface/VelocityJointInterface</hardwareInterface>
       </joint>
       <actuator name="${prefix}_motor">
-        <hardwareInterface>VelocityJointInterface</hardwareInterface>
+        <hardwareInterface>hardware_interface/VelocityJointInterface</hardwareInterface>
         <mechanicalReduction>1</mechanicalReduction>
       </actuator>

File: orne_box_description/urdf/orne_box.gazebo.xacro (robot description, xacro)
@@ -6,5 +6,5 @@
   <gazebo>
     <plugin name="gazebo_ros_control" filename="libgazebo_ros_control.so">
-      <robotNamespace>/orne-box</robotNamespace>
+      <robotNamespace>orne_box</robotNamespace>
       <robotSimType>gazebo_ros_control/DefaultRobotHWSim</robotSimType>
     </plugin>
@@ -13,5 +13,5 @@
     <material>Gazebo/Orange</material>
   </gazebo>
-  <gazebo reference="wheel_left_link">
+  <gazebo reference="left_wheel">
     <mu1>1.0</mu1>
     <mu2>1.0</mu2>
@@ -22,5 +22,5 @@
     <material>Gazebo/White</material>
   </gazebo>
-  <gazebo reference="wheel_right_link">
+  <gazebo reference="right_wheel">
     <mu1>1.0</mu1>
     <mu2>1.0</mu2>

Commit message: fix dynamics parameters

File: orne_box_description/urdf/joints/wheel_joint.urdf.xacro (robot description, xacro)
@@ -7,5 +7,6 @@
       <xacro:insert_block name="origin"/>
       <xacro:insert_block name="axis"/>
-      <limit effort="100" velocity="100.0" lower="-5000" upper="5000"/>
+      <limit effort="100.5" velocity="8.0" lower="-1e15" upper="1e15"/>
+      <dynamics damping="0.05"/>
     </joint>
     <transmission name="transmission_${prefix}">

File: orne_box_description/urdf/links/base_link.urdf.xacro (robot description, xacro)
@@ -58,5 +58,5 @@
         <origin xyz="0.090 0 0.1715" rpy="0 0 0"/>
         <mass value="25.0"/>
-        <inertia ixx="1.0" ixy="0.0" ixz="0.0" iyy="1.0" iyz="0.0" izz="1.0"/>
+        <inertia ixx="1.12" ixy="0.0" ixz="0.0" iyy="3.46" iyz="0.0" izz="3.9"/>
       </inertial>
     </link>

File: orne_box_description/urdf/links/caster_link.urdf.xacro (robot description, xacro)
@@ -32,5 +32,5 @@
         <origin xyz="0 0 0"/>
         <mass value="0.2"/>
-        <inertia ixx="0.1" ixy="0.0" ixz="0.0" iyy="0.1" iyz="0.0" izz="0.1"/>
+        <inertia ixx="0.001" ixy="0.0" ixz="0.0" iyy="0.001" iyz="0.0" izz="0.001"/>
       </inertial>
     </link>

File: orne_box_description/urdf/links/wheel_link.urdf.xacro (robot description, xacro)
@@ -18,6 +18,6 @@
       <inertial>
         <origin xyz="0 0 0"/>
-        <mass value="0.2"/>
-        <inertia ixx="0.1" ixy="0.0" ixz="0.0" iyy="0.1" iyz="0.0" izz="0.1"/>
+        <mass value="0.5"/>
+        <inertia ixx="0.005" ixy="0.0" ixz="0.0" iyy="0.005" iyz="0.0" izz="0.01"/>
       </inertial>
     </link>

File: orne_box_description/urdf/orne_box.gazebo.xacro (robot description, xacro)
@@ -5,4 +5,31 @@
   <xacro:arg name="imu_visual"   default="false"/>
   <xacro:arg name="ignition_gazebo" default="false"/>
+  <xacro:arg name="enable_camera" default="false"/>
+  <gazebo reference="caster_front_link">
+    <mu1>0.0001</mu1>
+    <mu2>0.0001</mu2>
+    <kp>1000000.0</kp>
+    <kd>100.0</kd>
+    <minDepth>0.001</minDepth>
+    <maxVel>1.0</maxVel>
+  </gazebo>
+  <gazebo reference="left_wheel">
+    <mu1>0.95</mu1>
+    <mu2>0.95</mu2>
+    <kp>1000000.0</kp>
+    <kd>100.0</kd>
+    <minDepth>0.001</minDepth>
+    <maxVel>1.0</maxVel>
+    <material>Gazebo/White</material>
+  </gazebo>
+  <gazebo reference="right_wheel">
+    <mu1>0.95</mu1>
+    <mu2>0.95</mu2>
+    <kp>1000000.0</kp>
+    <kd>100.0</kd>
+    <minDepth>0.001</minDepth>
+    <maxVel>1.0</maxVel>
+    <material>Gazebo/White</material>
+  </gazebo>
   <!-- @TODO More clear boolean operation -->
   <xacro:if value="${'$(arg ignition_gazebo)' == 'false'}">
@@ -15,27 +42,4 @@
     <gazebo reference="base_link">
       <material>Gazebo/Orange</material>
-    </gazebo>
-    <gazebo reference="left_wheel">
-      <mu1>1.0</mu1>
-      <mu2>1.0</mu2>
-      <kp>1000000.0</kp>
-      <kd>100.0</kd>
-      <minDepth>0.001</minDepth>
-      <maxVel>1.0</maxVel>
-      <material>Gazebo/White</material>
-    </gazebo>
-    <gazebo reference="right_wheel">
-      <mu1>1.0</mu1>
-      <mu2>1.0</mu2>
-      <kp>1000000.0</kp>
-      <kd>100.0</kd>
-      <minDepth>0.001</minDepth>
-      <maxVel>1.0</maxVel>
-      <material>Gazebo/White</material>
-    </gazebo>
-    <gazebo reference="caster_front_link">
-      <mu1>0.0</mu1>
-      <mu2>0.0</mu2>
-      <material>Gazebo/Red</material>
     </gazebo>
     <gazebo reference="imu_link">
@@ -86,4 +90,6 @@
   <xacro:if value="$(arg ignition_gazebo)">
     <gazebo>
+      <static>false</static>
+      <selfCollide>true</selfCollide>
       <plugin filename="ignition-gazebo-joint-state-publisher-system" name="ignition::gazebo::systems::JointStatePublisher">
         <topic>model/orne_box/joint_states</topic>
@@ -98,16 +104,25 @@
         <left_joint>left_wheel_joint</left_joint>
         <right_joint>right_wheel_joint</right_joint>
-        <wheel_separation>1.25</wheel_separation>
+        <wheel_separation>0.38</wheel_separation>
         <wheel_radius>0.3</wheel_radius>
-        <odom_publish_frequency>10</odom_publish_frequency>
-        <max_linear_acceleration>1</max_linear_acceleration>
-        <min_linear_acceleration>-1</min_linear_acceleration>
-        <max_angular_acceleration>2</max_angular_acceleration>
-        <min_angular_acceleration>-2</min_angular_acceleration>
-        <max_linear_velocity>0.5</max_linear_velocity>
-        <min_linear_velocity>-0.5</min_linear_velocity>
-        <max_angular_velocity>1</max_angular_velocity>
-        <min_angular_velocity>-1</min_angular_velocity>
-        <topic>cmd_vel</topic>
+        <odom_publish_frequency>30</odom_publish_frequency>
+        <max_angular_acceleration>3.14</max_angular_acceleration>
+        <min_angular_acceleration>-3.14</min_angular_acceleration>
+        <max_angular_velocity>1.57</max_angular_velocity>
+        <min_angular_velocity>-1.57</min_angular_velocity>
+      </plugin>
+      <plugin filename="libignition-gazebo-wheel-slip-system.so" name="ignition::gazebo::systems::WheelSlip">
+        <wheel link_name="wheel_left_link">
+          <slip_compliance_lateral>0.6</slip_compliance_lateral>
+          <slip_compliance_longitudinal>0.45</slip_compliance_longitudinal>
+          <wheel_normal_force>294.6</wheel_normal_force>
+          <wheel_radius>0.15</wheel_radius>
+        </wheel>
+        <wheel link_name="wheel_right_link">
+          <slip_compliance_lateral>0.6</slip_compliance_lateral>
+          <slip_compliance_longitudinal>0.45</slip_compliance_longitudinal>
+          <wheel_normal_force>294.6</wheel_normal_force>
+          <wheel_radius>0.15</wheel_radius>
+        </wheel>
       </plugin>
     </gazebo>
@@ -190,49 +205,51 @@
       </sensor>
     </gazebo>
-    <gazebo reference="zed_camera_center">
-      <sensor name="zed_camera_center" type="camera">
-        <always_on>1</always_on>
-        <update_rate>15</update_rate>
-        <visualize>false</visualize>
-        <topic>model/orne_box/zed_node/image</topic>
-        <camera>
-          <horizontal_fov>1.919805</horizontal_fov>
-          <image>
-            <width>1920</width>
-            <height>1080</height>
-          </image>
-          <clip>
-            <near>0.01</near>
-            <far>50</far>
-          </clip>
-          <noise type="gaussian">
-            <mean>0.0</mean>
-            <stddev>0.025</stddev>
-          </noise>
-        </camera>
-      </sensor>
-      <sensor name="zed_depth_camera_center" type="depth_camera">
-        <pose>0 0 -0.8 3.14 -0.38 0</pose>
-        <always_on>1</always_on>
-        <update_rate>15</update_rate>
-        <visualize>false</visualize>
-        <topic>model/orne_box/zed_node/depth_image</topic>
-        <camera>
-          <horizontal_fov>1.919805</horizontal_fov>
-          <image>
-            <width>1280</width>
-            <height>720</height>
-          </image>
-          <clip>
-            <near>0.4</near>
-            <far>6</far>
-          </clip>
-          <noise type="gaussian">
-            <mean>0.0</mean>
-            <stddev>0.1</stddev>
-          </noise>
-        </camera>
-      </sensor>
-    </gazebo>
+    <xacro:if value="$(arg enable_camera)">
+      <gazebo reference="zed_camera_center">
+        <sensor name="zed_camera_center" type="camera">
+          <always_on>1</always_on>
+          <update_rate>15</update_rate>
+          <visualize>false</visualize>
+          <topic>model/orne_box/zed_node/image</topic>
+          <camera>
+            <horizontal_fov>1.919805</horizontal_fov>
+            <image>
+              <width>1920</width>
+              <height>1080</height>
+            </image>
+            <clip>
+              <near>0.01</near>
+              <far>50</far>
+            </clip>
+            <noise type="gaussian">
+              <mean>0.0</mean>
+              <stddev>0.025</stddev>
+            </noise>
+          </camera>
+        </sensor>
+        <sensor name="zed_depth_camera_center" type="depth_camera">
+          <pose>0 0 -0.8 3.14 -0.38 0</pose>
+          <always_on>1</always_on>
+          <update_rate>15</update_rate>
+          <visualize>false</visualize>
+          <topic>model/orne_box/zed_node/depth_image</topic>
+          <camera>
+            <horizontal_fov>1.919805</horizontal_fov>
+            <image>
+              <width>1280</width>
+              <height>720</height>
+            </image>
+            <clip>
+              <near>0.4</near>
+              <far>6</far>
+            </clip>
+            <noise type="gaussian">
+              <mean>0.0</mean>
+              <stddev>0.1</stddev>
+            </noise>
+          </camera>
+        </sensor>
+      </gazebo>
+    </xacro:if>
   </xacro:if>
 </robot>

File: orne_box_description/urdf/orne_box_3d_lidar.urdf.xacro (robot description, xacro)
@@ -16,16 +16,14 @@
         <origin xyz="0.0 0.0 0.0" rpy="0.0 0.0 0.0"/>
         <mass value="0.3"/>
-        <inertia ixx="0.0" ixy="0.0" ixz="0.0" iyy="0.0" iyz="0.0" izz="0.0"/>
+        <inertia ixx="0.01" ixy="0.0" ixz="0.0" iyy="0.01" iyz="0.0" izz="0.01"/>
       </inertial>
-      <visual name="">
+      <visual name="surestar_visual">
         <origin xyz="0.0 0.0 0.0" rpy="0.0 0.0 0.0"/>
         <geometry>
           <cylinder radius="0.06" length="0.1"/>
         </geometry>
-        <material name="">
-          <color rgba="0.0 1.0 0.0 1.0"/>
-        </material>
+        <material name="green"/>
       </visual>
-      <collision>
+      <collision name="surestar_collision">
         <origin xyz="0.0 0.0 0.0" rpy="0.0 0.0 0.0"/>
         <geometry>

File: orne_box_description/urdf/sensors/camera.urdf.xacro (robot description, xacro)
@@ -11,4 +11,9 @@
     </joint>
     <link name="zed_camera_center">
+      <inertial>
+        <origin xyz="0.0 0.0 0.0" rpy="0.0 0.0 0.0"/>
+        <mass value="0.1"/>
+        <inertia ixx="0.005" ixy="0.0" ixz="0.0" iyy="0.005" iyz="0.0" izz="0.005"/>
+      </inertial>
       <visual>
         <origin rpy="0 0 0" xyz="0 0 0"/>

File: orne_box_description/urdf/sensors/gnss.urdf.xacro (robot description, xacro)
@@ -11,4 +11,9 @@
     </joint>
     <link name="${name}_link">
+      <inertial>
+        <origin xyz="0.0 0.0 0.0" rpy="0.0 0.0 0.0"/>
+        <mass value="0.1"/>
+        <inertia ixx="0.001" ixy="0.0" ixz="0.0" iyy="0.001" iyz="0.0" izz="0.001"/>
+      </inertial>
       <visual>
         <origin rpy="0 0 0" xyz="0 0 0"/>

File: orne_box_description/urdf/sensors/hokuyo.urdf.xacro (robot description, xacro)
@@ -11,4 +11,9 @@
     </joint>
     <link name="${name}_link">
+      <inertial>
+        <origin xyz="0.0 0.0 0.0" rpy="0.0 0.0 0.0"/>
+        <mass value="0.2"/>
+        <inertia ixx="0.005" ixy="0.0" ixz="0.0" iyy="0.005" iyz="0.0" izz="0.005"/>
+      </inertial>
       <visual>
         <origin rpy="0 0 0" xyz="0 0 0"/>

File: orne_box_description/urdf/sensors/imu.urdf.xacro (robot description, xacro)
@@ -12,4 +12,9 @@
     </joint>
     <link name="${name}_link">
+      <inertial>
+        <origin xyz="0.0 0.0 0.0" rpy="0.0 0.0 0.0"/>
+        <mass value="0.005"/>
+        <inertia ixx="0.001" ixy="0.0" ixz="0.0" iyy="0.001" iyz="0.0" izz="0.001"/>
+      </inertial>
       <visual>
         <origin rpy="0 0 0" xyz="0 0 0"/>

Commit message: lint

File: orne_box_description/urdf/joints/wheel_joint.urdf.xacro (robot description, xacro)
@@ -7,5 +7,5 @@
       <xacro:insert_block name="origin"/>
       <xacro:insert_block name="axis"/>
-      <limit effort="100.5" velocity="8.0" lower="-1e15" upper="1e15"/>
+      <limit effort="100.5" velocity="10.0" lower="-1e15" upper="1e15"/>
       <dynamics damping="0.05"/>
     </joint>

File: orne_box_description/urdf/links/wheel_link.urdf.xacro (robot description, xacro)
@@ -18,5 +18,5 @@
       <inertial>
         <origin xyz="0 0 0"/>
-        <mass value="0.5"/>
+        <mass value="0.15"/>
         <inertia ixx="0.005" ixy="0.0" ixz="0.0" iyy="0.005" iyz="0.0" izz="0.01"/>
       </inertial>

File: orne_box_description/urdf/orne_box.gazebo.xacro (robot description, xacro)
@@ -1,7 +1,7 @@
 <?xml version="1.0"?>
-<robot name="orne_box" xmlns:xacro="http://ros.org/wiki/xacro">
+<robot xmlns:xacro="http://ros.org/wiki/xacro" name="orne_box">
   <xacro:property name="PI" value="3.1415926535897931"/>
   <xacro:arg name="laser_visual" default="true"/>
-  <xacro:arg name="imu_visual"   default="false"/>
+  <xacro:arg name="imu_visual" default="false"/>
   <xacro:arg name="ignition_gazebo" default="false"/>
   <xacro:arg name="enable_camera" default="false"/>

File: orne_box_description/urdf/orne_box.urdf.xacro (robot description, xacro)
@@ -1,6 +1,6 @@
-<?xml version="1.0" ?>
-<robot name="orne_box" xmlns:xacro="http://www.ros.org/wiki/xacro">
+<?xml version="1.0"?>
+<robot xmlns:xacro="http://www.ros.org/wiki/xacro" name="orne_box">
   <xacro:property name="PI" value="3.1415926535897931"/>
-  <xacro:include filename="$(find orne_box_description)/urdf/material_colors.xacro" />
+  <xacro:include filename="$(find orne_box_description)/urdf/material_colors.xacro"/>
   <xacro:include filename="$(find orne_box_description)/urdf/orne_box.gazebo.xacro"/>
   <xacro:include filename="$(find orne_box_description)/urdf/links/base_link.urdf.xacro"/>
@@ -20,5 +20,5 @@
   <xacro:caster_wheel_joint prefix="left"/>
   <xacro:caster_swivel_joint prefix="left" parent="base_link">
-    <origin xyz="0.362 0.150 0.12" rpy="0 0 0"/>
+    <origin xyz="0.362 0.150 0.115" rpy="0 0 0"/>
   </xacro:caster_swivel_joint>
   <xacro:caster_wheel_link prefix="right"/>
@@ -26,5 +26,5 @@
   <xacro:caster_wheel_joint prefix="right"/>
   <xacro:caster_swivel_joint prefix="right" parent="base_link">
-    <origin xyz="0.362 -0.150 0.12" rpy="0 0 0"/>
+    <origin xyz="0.362 -0.150 0.115" rpy="0 0 0"/>
   </xacro:caster_swivel_joint>
   <!-- Setting for left wheel -->

File: orne_box_description/urdf/orne_box_3d_lidar.urdf.xacro (robot description, xacro)
@@ -1,4 +1,4 @@
-<?xml version="1.0" ?>
-<robot name="orne_box" xmlns:xacro="http://www.ros.org/wiki/xacro">
+<?xml version="1.0"?>
+<robot xmlns:xacro="http://www.ros.org/wiki/xacro" name="orne_box">
   <xacro:arg name="ignition_gazebo" default="false"/>
   <xacro:include filename="$(find orne_box_description)/urdf/orne_box.urdf.xacro"/>
@@ -8,5 +8,5 @@
     <!-- Setting for 3D-LiDAR -->
     <xacro:VLP-16 parent="base_link" name="surestar" topic="/rfans_points" organize_cloud="false" hz="10" samples="440" gpu="false">
-      <origin xyz="0.23 0 0.40" rpy="0 0 0" />
+      <origin xyz="0.23 0 0.40" rpy="0 0 0"/>
     </xacro:VLP-16>
   </xacro:if>

File: orne_box_description/urdf/sensors/camera.urdf.xacro (robot description, xacro)
@@ -1,6 +1,4 @@
 <?xml version="1.0"?>
-<robot name="sensor_camera" xmlns:xacro="http://ros.org/wiki/xacro"
-                            xmlns:controller="http://playerstage.sourceforge.net/gazebo/xmlschema/#controller"
-                            xmlns:interface="http://playerstage.sourceforge.net/gazebo/xmlschema/#interface">
+<robot xmlns:xacro="http://ros.org/wiki/xacro" xmlns:controller="http://playerstage.sourceforge.net/gazebo/xmlschema/#controller" xmlns:interface="http://playerstage.sourceforge.net/gazebo/xmlschema/#interface" name="sensor_camera">
   <xacro:macro name="sensor_camera" params="name parent *origin">
     <joint name="${name}_joint" type="fixed">

File: orne_box_description/urdf/sensors/gnss.urdf.xacro (robot description, xacro)
@@ -1,6 +1,4 @@
 <?xml version="1.0"?>
-<robot name="sensor_gnss" xmlns:xacro="http://ros.org/wiki/xacro"
-                          xmlns:controller="http://playerstage.sourceforge.net/gazebo/xmlschema/#controller"
-                          xmlns:interface="http://playerstage.sourceforge.net/gazebo/xmlschema/#interface">
+<robot xmlns:xacro="http://ros.org/wiki/xacro" xmlns:controller="http://playerstage.sourceforge.net/gazebo/xmlschema/#controller" xmlns:interface="http://playerstage.sourceforge.net/gazebo/xmlschema/#interface" name="sensor_gnss">
   <xacro:macro name="sensor_gnss" params="name parent *origin">
     <joint name="${name}_joint" type="fixed">
@@ -19,5 +17,5 @@
         <origin rpy="0 0 0" xyz="0 0 0"/>
         <geometry>
-          <cylinder  length="0.025" radius="0.05"/>
+          <cylinder length="0.025" radius="0.05"/>
         </geometry>
         <material name="red"/>

File: orne_box_description/urdf/sensors/hokuyo.urdf.xacro (robot description, xacro)
@@ -1,6 +1,4 @@
 <?xml version="1.0"?>
-<robot name="sensor_hokuyo" xmlns:xacro="http://ros.org/wiki/xacro"
-                            xmlns:controller="http://playerstage.sourceforge.net/gazebo/xmlschema/#controller"
-                            xmlns:interface="http://playerstage.sourceforge.net/gazebo/xmlschema/#interface">
+<robot xmlns:xacro="http://ros.org/wiki/xacro" xmlns:controller="http://playerstage.sourceforge.net/gazebo/xmlschema/#controller" xmlns:interface="http://playerstage.sourceforge.net/gazebo/xmlschema/#interface" name="sensor_hokuyo">
   <xacro:macro name="sensor_hokuyo" params="name parent *origin size">
     <joint name="${name}_joint" type="fixed">

File: orne_box_description/urdf/sensors/imu.urdf.xacro (robot description, xacro)
@@ -1,6 +1,4 @@
 <?xml version="1.0"?>
-<robot name="sensor_imu" xmlns:xacro="http://ros.org/wiki/xacro"
-                         xmlns:controller="http://playerstage.sourceforge.net/gazebo/xmlschema/#controller"
-                         xmlns:interface="http://playerstage.sourceforge.net/gazebo/xmlschema/#interface">
+<robot xmlns:xacro="http://ros.org/wiki/xacro" xmlns:controller="http://playerstage.sourceforge.net/gazebo/xmlschema/#controller" xmlns:interface="http://playerstage.sourceforge.net/gazebo/xmlschema/#interface" name="sensor_imu">
   <xacro:arg name="ignition_gazebo" default="false"/>
   <xacro:macro name="sensor_imu" params="name parent *origin size">
@@ -29,5 +27,6 @@
       <gazebo>
         <plugin name="ros_imu" filename="libgazebo_ros_imu.so">
-          <bodyName>imu_link</bodyName> <!-- bodyName always set base_link by URDF parser -->
+          <bodyName>imu_link</bodyName>
+          <!-- bodyName always set base_link by URDF parser -->
           <topicName>imu_data</topicName>
           <serviceName>imu_service</serviceName>
