Commit message: fix incorrect dynamics parameter

File: orne_box_description/urdf/joints/caster_wheel_joint.urdf.xacro (robot description, xacro)
@@ -5,5 +5,5 @@
       <parent link="${prefix}_caster_swivel_link"/>
       <child link="${prefix}_caster_wheel_link"/>
-      <origin xyz="0.01 0.0 -0.065" rpy="${-PI/2} 0 0"/>
+      <origin xyz="0.03 0.0 -0.065" rpy="${-PI/2} 0 0"/>
       <axis xyz="0 0 1"/>
       <limit effort="0.0" velocity="0.0" lower="-1e15" upper="1e15"/>

File: orne_box_description/urdf/joints/wheel_joint.urdf.xacro (robot description, xacro)
@@ -7,5 +7,5 @@
       <xacro:insert_block name="origin"/>
       <xacro:insert_block name="axis"/>
-      <limit effort="100.5" velocity="10.0" lower="-1e15" upper="1e15"/>
+      <limit effort="10.5" velocity="10.0" lower="-1e15" upper="1e15"/>
       <dynamics damping="0.05"/>
     </joint>

File: orne_box_description/urdf/orne_box.gazebo.xacro (robot description, xacro)
@@ -113,5 +113,5 @@
         <right_joint>right_wheel_joint</right_joint>
         <wheel_separation>0.38</wheel_separation>
-        <wheel_radius>0.3</wheel_radius>
+        <wheel_radius>0.152</wheel_radius>
         <odom_publish_frequency>30</odom_publish_frequency>
         <max_angular_acceleration>3.14</max_angular_acceleration>
@@ -122,24 +122,24 @@
       <plugin filename="libignition-gazebo-wheel-slip-system.so" name="ignition::gazebo::systems::WheelSlip">
         <wheel link_name="left_caster_wheel_link">
-          <slip_compliance_lateral>0.6</slip_compliance_lateral>
-          <slip_compliance_longitudinal>0.45</slip_compliance_longitudinal>
-          <wheel_normal_force>80.6</wheel_normal_force>
+          <slip_compliance_lateral>0.2</slip_compliance_lateral>
+          <slip_compliance_longitudinal>0.15</slip_compliance_longitudinal>
+          <wheel_normal_force>20.6</wheel_normal_force>
           <wheel_radius>0.04</wheel_radius>
         </wheel>
         <wheel link_name="right_caster_wheel_link">
-          <slip_compliance_lateral>0.6</slip_compliance_lateral>
-          <slip_compliance_longitudinal>0.45</slip_compliance_longitudinal>
-          <wheel_normal_force>80.6</wheel_normal_force>
+          <slip_compliance_lateral>0.2</slip_compliance_lateral>
+          <slip_compliance_longitudinal>0.15</slip_compliance_longitudinal>
+          <wheel_normal_force>20.6</wheel_normal_force>
           <wheel_radius>0.04</wheel_radius>
         </wheel>
         <wheel link_name="wheel_left_link">
-          <slip_compliance_lateral>0.6</slip_compliance_lateral>
-          <slip_compliance_longitudinal>0.45</slip_compliance_longitudinal>
+          <slip_compliance_lateral>0.7</slip_compliance_lateral>
+          <slip_compliance_longitudinal>0.55</slip_compliance_longitudinal>
           <wheel_normal_force>294.6</wheel_normal_force>
           <wheel_radius>0.15</wheel_radius>
         </wheel>
         <wheel link_name="wheel_right_link">
-          <slip_compliance_lateral>0.6</slip_compliance_lateral>
-          <slip_compliance_longitudinal>0.45</slip_compliance_longitudinal>
+          <slip_compliance_lateral>0.7</slip_compliance_lateral>
+          <slip_compliance_longitudinal>0.55</slip_compliance_longitudinal>
           <wheel_normal_force>294.6</wheel_normal_force>
           <wheel_radius>0.15</wheel_radius>

Commit message: repair simulation

File: orne_box_description/urdf/joints/caster_wheel_joint.urdf.xacro (robot description, xacro)
@@ -5,5 +5,5 @@
       <parent link="${prefix}_caster_swivel_link"/>
       <child link="${prefix}_caster_wheel_link"/>
-      <origin xyz="0.03 0.0 -0.065" rpy="${-PI/2} 0 0"/>
+      <origin xyz="0.03 0.0 -0.058" rpy="${-PI/2} 0 0"/>
       <axis xyz="0 0 1"/>
       <limit effort="0.0" velocity="0.0" lower="-1e15" upper="1e15"/>

File: orne_box_description/urdf/orne_box.gazebo.xacro (robot description, xacro)
@@ -2,6 +2,7 @@
 <robot xmlns:xacro="http://ros.org/wiki/xacro" name="orne_box">
   <xacro:property name="PI" value="3.1415926535897931"/>
-  <!-- <xacro:arg name="laser_visual" default="true"/> -->
-  <xacro:arg name="imu_visual" default="false"/>
+  <xacro:arg name="laser_visual" default="true"/>
+  <!--<xacro:arg name="imu_visual" default="false"/> -->
+  <!--<xacro:arg name="enable_camera" default="false"/>-->
   <gazebo reference="left_caster_wheel_link">
     <mu1>0.75</mu1>
@@ -54,5 +55,5 @@
         <odometry_frame>odom</odometry_frame>
         <!-- <odometrySource>world</odometrySource> -->
-        <robot_base_frame>base_footprint</robot_base_frame>
+        <robot_base_frame>base_link</robot_base_frame>
         <update_rate>30</update_rate>
         <!-- wheels -->
@@ -67,5 +68,5 @@
         <!-- output -->
         <publish_odom>true</publish_odom>
-        <publish_odom_tf>true</publish_odom_tf>
+        <publish_odom_tf>false</publish_odom_tf>
         <publish_wheel_tf>false</publish_wheel_tf>
       </plugin>
@@ -91,7 +92,7 @@
             <noise type="gaussian">
                 <mean>0.0</mean>
-                <stddev>2e-4</stddev>
-                <bias_mean>0.0000075</bias_mean>
-                <bias_stddev>0.0000008</bias_stddev>
+                <stddev>0.0</stddev>
+                <bias_mean>0.0</bias_mean>
+                <bias_stddev>0.0</bias_stddev>
               </noise>
             </x>
@@ -99,7 +100,7 @@
               <noise type="gaussian">
                 <mean>0.0</mean>
-                <stddev>2e-4</stddev>
-                <bias_mean>0.0000075</bias_mean>
-                <bias_stddev>0.0000008</bias_stddev>
+                <stddev>0.0</stddev>
+                <bias_mean>0.0</bias_mean>
+                <bias_stddev>0.0</bias_stddev>
               </noise>
             </y>
@@ -107,7 +108,7 @@
               <noise type="gaussian">
                 <mean>0.0</mean>
-                <stddev>2e-4</stddev>
-                <bias_mean>0.0000075</bias_mean>
-                <bias_stddev>0.0000008</bias_stddev>
+                <stddev>0.0</stddev>
+                <bias_mean>0.0</bias_mean>
+                <bias_stddev>0.0</bias_stddev>
               </noise>
             </z>
@@ -117,7 +118,7 @@
               <noise type="gaussian">
                 <mean>0.0</mean>
-                <stddev>1.7e-2</stddev>
-                <bias_mean>0.1</bias_mean>
-                <bias_stddev>0.001</bias_stddev>
+                <stddev>0.0</stddev>
+                <bias_mean>0.0</bias_mean>
+		<bias_stddev>0.0</bias_stddev>
               </noise>
             </x>
@@ -125,7 +126,7 @@
               <noise type="gaussian">
                 <mean>0.0</mean>
-                <stddev>1.7e-2</stddev>
-                <bias_mean>0.1</bias_mean>
-                <bias_stddev>0.001</bias_stddev>
+                <stddev>0.0</stddev>
+                <bias_mean>0.0</bias_mean>
+                <bias_stddev>0.0</bias_stddev>
               </noise>
             </y>
@@ -133,7 +134,7 @@
               <noise type="gaussian">
                 <mean>0.0</mean>
-                <stddev>1.7e-2</stddev>
-                <bias_mean>0.1</bias_mean>
-                <bias_stddev>0.001</bias_stddev>
+                <stddev>0.0</stddev>
+                <bias_mean>0.0</bias_mean>
+                <bias_stddev>0.0</bias_stddev>
               </noise>
             </z>
@@ -144,5 +145,5 @@
     </gazebo>
     <!-- hokuyo -->
-    <!-- <gazebo reference="hokuyo_link">
+    <!--<gazebo reference="hokuyo_link">
       <sensor type="ray" name="head_hokuyo_sensor">
         <pose>0 0 0 0 0 0</pose>
@@ -175,5 +176,5 @@
         <plugin name="gazebo_ros_head_hokuyo_controller" filename="libgazebo_ros_ray_sensor.so">
           <ros>
-            <remapping>~/out:=scan</remapping>
+            <remapping>~/out:=hokuyo_scan</remapping>
           </ros>
           <frame_name>hokuyo_link</frame_name>

File: orne_box_description/urdf/orne_box.urdf.xacro (robot description, xacro)
@@ -12,5 +12,5 @@
   <xacro:include filename="$(find orne_box_description)/urdf/joints/wheel_joint.urdf.xacro"/>
   <xacro:include filename="$(find orne_box_description)/urdf/sensors/imu.urdf.xacro"/>
-  <!-- <xacro:include filename="$(find orne_box_description)/urdf/sensors/hokuyo.urdf.xacro"/> -->
+  <xacro:include filename="$(find orne_box_description)/urdf/sensors/hokuyo.urdf.xacro"/>
   <!-- Setting for base -->
   <xacro:base_link/>
@@ -20,5 +20,5 @@
   <xacro:caster_wheel_joint prefix="left"/>
   <xacro:caster_swivel_joint prefix="left" parent="base_link">
-    <origin xyz="0.362 0.150 0.115" rpy="0 0 0"/>
+    <origin xyz="0.362 0.150 0.108" rpy="0 0 0"/>
   </xacro:caster_swivel_joint>
   <xacro:caster_wheel_link prefix="right"/>
@@ -26,20 +26,20 @@
   <xacro:caster_wheel_joint prefix="right"/>
   <xacro:caster_swivel_joint prefix="right" parent="base_link">
-    <origin xyz="0.362 -0.150 0.115" rpy="0 0 0"/>
+    <origin xyz="0.362 -0.150 0.108" rpy="0 0 0"/>
   </xacro:caster_swivel_joint>
   <!-- Setting for left wheel -->
   <xacro:wheel_joint prefix="left" parent="base_link">
-    <origin xyz="0.0 0.23075 0.152" rpy="${-PI/2} 0 0"/>
+    <origin xyz="0.0 0.23075 0.145" rpy="${-PI/2} 0 0"/>
     <axis xyz="0 0 1"/>
   </xacro:wheel_joint>
-  <xacro:wheel_link prefix="left" width="0.045" radius="0.152">
+  <xacro:wheel_link prefix="left" width="0.045" radius="0.145">
     <origin xyz="0.0 0.0 0.0" rpy="0 0 0"/>
   </xacro:wheel_link>
   <!-- Setting for right wheel -->
   <xacro:wheel_joint prefix="right" parent="base_link">
-    <origin xyz="0.0 -0.23075 0.152" rpy="${-PI/2} 0 0"/>
+    <origin xyz="0.0 -0.23075 0.145" rpy="${-PI/2} 0 0"/>
     <axis xyz="0 0 1"/>
   </xacro:wheel_joint>
-  <xacro:wheel_link prefix="right" width="0.045" radius="0.152">
+  <xacro:wheel_link prefix="right" width="0.045" radius="0.145">
     <origin xyz="0.0 0.0 0.0" rpy="0 0 0"/>
   </xacro:wheel_link>
@@ -53,7 +53,7 @@
   </xacro:sensor_imu>
   <!-- Setting for 2D-LiDAR -->
-  <!-- <xacro:sensor_hokuyo name="hokuyo" parent="base_link" size="0.05 0.05 0.05"> -->
-    <!-- <origin xyz="0.364295 0 0.185" rpy="3.14 0 0"/>
-  </xacro:sensor_hokuyo> -->
+  <!--<xacro:sensor_hokuyo name="hokuyo" parent="base_link" size="0.05 0.05 0.05">
+    <origin xyz="0.364295 0 0.185" rpy="3.14 0 0"/>
+  </xacro:sensor_hokuyo>-->
   <!-- <xacro:sensor_hokuyo name="mirror_lidar" parent="base_link" size="0.05 0.05 0.05">
     <origin xyz="0.43 0.0 0.34" rpy="0 0.314 0"/>
