Commit message: fix rfans driver

File: orne_box_description/urdf/sensors/imu.urdf.xacro (robot description, xacro)
@@ -8,5 +8,26 @@
       <child link="${name}_link"/>
     </joint>
+    <!-- <link name="${name}_link"> -->
     <link name="${name}_link">
+      <inertial>
+        <origin xyz="0.0 0.0 0.0" rpy="0.0 0.0 0.0"/>
+        <mass value="0.005"/>
+        <inertia ixx="0.001" ixy="0.0" ixz="0.0" iyy="0.001" iyz="0.0" izz="0.001"/>
+      </inertial>
+      <visual>
+        <origin rpy="0 0 0" xyz="0 0 0"/>
+        <geometry>
+          <box size="${size}"/>
+        </geometry>
+        <material name="green"/>
+      </visual>
+    </link>
+    <joint name="${name}_base_joint" type="fixed">
+      <axis xyz="1 0 0"/>
+      <xacro:insert_block name="origin"/>
+      <parent link="${name}_link"/>
+      <child link="${name}"/>
+    </joint>
+    <link name="${name}">
       <inertial>
         <origin xyz="0.0 0.0 0.0" rpy="0.0 0.0 0.0"/>
